File: ZX-Spectrum-Pentagon/CPU.sch (KiCad schematic (older format))
At the start: 0 parts

Commit message: improve schema
Parts:
- added R5: 330, symbol Device:R
- added RN1: 10k, Resistor_THT:R_Array_SIP9, symbol Device:R_Network08_Split
- added U15: Z80CPU, Package_DIP:DIP-40_W15.24mm, symbol Zilog:Z80CPU
- added U16: 74HC245, symbol 74IEC:74HC245
- added U17: 74HC244, Package_DIP:DIP-20_W7.62mm, symbol 74IEC:74HC244
- added U2: 74HC14, Package_DIP:DIP-14_W7.62mm, symbol 74IEC:74HC14
Connections:
- net labels added: C25, VCC, xA0, xA1, xA10, xA11, xA12, xA13, xA14, xA15, xA2, xA3, xA4, xA5, xA6, xA7, xA8, xA9, xD0, xD1, xD2, xD3, xD4, xD5, xD6, xD7, ~xBUSACK, ~xBUSRQ, ~xHALT, ~xINT, ~xIORQ, ~xM1, ~xMREQ, ~xNMI, ~xRD, ~xRESET, ~xRFSH, ~xWAIT, ~xWR
- wire segments 0 -> 59

Commit message: improve schema
Parts:
- added 1N4148: D2, symbol Device:D
- added C4: 47u/6.3V, symbol Device:CP
- added R7: 680, Resistor_SMD:R_0805_2012Metric, symbol Device:R
- added R8: 330, Resistor_SMD:R_0805_2012Metric, symbol Device:R
- added R9: 10k, Resistor_SMD:R_0805_2012Metric, symbol Device:R
- added RN2, RN? (x2): 10k, Resistor_THT:R_Array_SIP5, symbol Device:R_Network04_Split
- added SW1: RESET, symbol Switch:SW_Push
- added U18, U19: 74HC541, Package_DIP:DIP-20_W7.62mm, symbol 74IEC:74HC541
- added U9: 74HC00, symbol 74IEC:74HC00
- R5: footprint (none) -> Resistor_SMD:R_0805_2012Metric
Connections:
- net labels added: A0, A1, A10, A11, A12, A13, A14, A15, A2, A3, A4, A5, A6, A7, A8, A9, BUSACK, BUSRQ, C8, D0, D1, D2, D3, D4, D5, D6, D7, DIR, GND, xMREQ, ~BUSACK, ~BUSRQ, ~C25, ~HALT, ~INT, ~IORQ, ~M1, ~MREQ, ~NMI, ~RD, ~RESET, ~RESH, ~RFSH, ~ROMCS, ~RST, ~WAIT, ~WR
- net labels removed: ~xINT, ~xNMI, ~xRESET, ~xWAIT
- wire segments 59 -> 205
Other:
- moved on the sheet: R5, U2C, U2D, U2E, U2F

Commit message: improve schema
Connections:
- wire segments 205 -> 207
Changed lines of the file:
@@
 	1400 3300 1500 3200
 Entry Wire Line
-	1400 3400 1500 3300
+	1300 3950 1400 3850
 Wire Wire Line
 	1500 1250 1900 1250
@@
 Wire Wire Line
 	1500 3200 1900 3200
-Wire Wire Line
-	1500 3300 1900 3300
 Wire Wire Line
 	1900 3000 1400 3000
@@
 ~WAIT
 Text Label 1400 3000 0    50   ~ 0
-~RESET
+~RST
 Text Label 3250 3350 0    50   ~ 0
 ~xRFSH
@@
 Text Label 1500 3200 0    50   ~ 0
 ~xBUSACK
-Text Label 1500 3300 0    50   ~ 0
+Text Label 1400 3850 0    50   ~ 0
 ~xBUSRQ
 Wire Wire Line
@@
 Wire Wire Line
 	3100 3250 3500 3250
-Text GLabel 850  2200 0    50   Input ~ 0
+Text GLabel 850  2200 0    50   Input ~ 10
 C25
 $Comp
@@
 	0    1    1    0
 $EndComp
-Text GLabel 800  2600 0    50   Input ~ 0
+Text GLabel 800  2600 0    50   Input ~ 10
 C8
 Wire Wire Line
@@
 U 1 1 6374CB2D
 P 1550 4800
-F 0 "SW1" V 1700 4950 50  0000 C CNN
-F 1 "RESET" V 1400 4950 50  0000 C CNN
+F 0 "SW1" V 1650 4650 50  0000 C CNN
+F 1 "RESET" V 1450 4650 50  0000 C CNN
 F 2 "" H 1550 5000 50  0001 C CNN
 F 3 "~" H 1550 5000 50  0001 C CNN
@@
 Text GLabel 10850 4500 2    50   Output ~ 10
 ~RFSH
-Text GLabel 10050 1100 0    50   Input ~ 10
+Text GLabel 850  3550 0    50   Input ~ 10
 ~WAIT
-Text GLabel 10050 1250 0    50   Input ~ 10
+Text GLabel 850  3700 0    50   Input ~ 10
 ~INT
-Text GLabel 10050 1400 0    50   Input ~ 10
+Text GLabel 850  3850 0    50   Input ~ 10
 ~NMI
-Text GLabel 10050 1550 0    50   Input ~ 10
+Text GLabel 850  4000 0    50   Input ~ 10
 ~BUSRQ
-Text GLabel 10050 1700 0    50   Input ~ 10
+Text GLabel 850  4150 0    50   Input ~ 10
 ~RST
-Text GLabel 10050 1850 0    50   Input ~ 10
+Text GLabel 850  4300 0    50   Input ~ 10
 ~C25
 Wire Wire Line
-	10050 1100 10400 1100
-Entry Wire Line
-	10400 1100 10500 1200
-Entry Wire Line
-	10400 1250 10500 1350
-Entry Wire Line
-	10400 1400 10500 1500
-Entry Wire Line
-	10400 1550 10500 1650
-Entry Wire Line
-	10400 1700 10500 1800
-Entry Wire Line
-	10400 1850 10500 1950
-Entry Wire Line
-	10400 2000 10500 2100
-Text GLabel 10050 2000 0    50   Input ~ 10
+	850  3550 1200 3550
+Entry Wire Line
+	1200 3550 1300 3650
+Entry Wire Line
+	1200 3700 1300 3800
+Entry Wire Line
+	1200 3850 1300 3950
+Entry Wire Line
+	1200 4000 1300 4100
+Entry Wire Line
+	1200 4150 1300 4250
+Entry Wire Line
+	1200 4300 1300 4400
+Entry Wire Line
+	1200 4450 1300 4550
+Text GLabel 850  4450 0    50   Input ~ 10
 ~ROMCS
 Wire Wire Line
-	10050 1250 10400 1250
-Wire Wire Line
-	10050 1400 10400 1400
-Wire Wire Line
-	10050 1550 10400 1550
-Wire Wire Line
-	10050 1700 10400 1700
-Wire Wire Line
-	10050 1850 10400 1850
-Wire Wire Line
-	10050 2000 10400 2000
-Text Label 10250 1100 0    50   ~ 0
+	850  3700 1200 3700
+Wire Wire Line
+	850  3850 1200 3850
+Wire Wire Line
+	850  4000 1200 4000
+Wire Wire Line
+	850  4150 1200 4150
+Wire Wire Line
+	850  4300 1200 4300
+Wire Wire Line
+	850  4450 1200 4450
+Text Label 1050 3550 0    50   ~ 0
 ~WAIT
-Text Label 10300 1250 0    50   ~ 0
+Text Label 1100 3700 0    50   ~ 0
 ~INT
-Text Label 10250 1400 0    50   ~ 0
+Text Label 1050 3850 0    50   ~ 0
 ~NMI
-Text Label 10150 1550 0    50   ~ 0
+Text Label 950  4000 0    50   ~ 0
 ~BUSRQ
-Text Label 10250 1700 0    50   ~ 0
+Text Label 1050 4150 0    50   ~ 0
 ~RST
-Text Label 10250 1850 0    50   ~ 0
+Text Label 1050 4300 0    50   ~ 0
 ~C25
-Text Label 10150 2000 0    50   ~ 0
+Text Label 950  4450 0    50   ~ 0
 ~ROMCS
 Entry Wire Line
@@
 D7
 Wire Bus Line
+	1400 3300 1400 3650
+Wire Wire Line
+	1400 3850 1800 3850
+Wire Wire Line
+	1800 3300 1900 3300
+Wire Wire Line
+	1800 3850 1800 3300
+Wire Bus Line
 	6900 2500 6900 3200
 Wire Bus Line
-	1400 3300 1400 3650
-Wire Bus Line
-	1300 2700 1300 7300
-Wire Bus Line
 	6700 650  6700 1850
 Wire Bus Line
@@
 	1400 650  1400 1950
 Wire Bus Line
+	10500 600  10500 4650
+Wire Bus Line
+	1300 2800 1300 7300
+Wire Bus Line
 	5150 2500 5150 7300
 Wire Bus Line
-	10500 600  10500 4650
-Wire Bus Line
 	3600 650  3600 3650

Commit message: add footprint and symbol edge, update schema
Parts:
- added XM1: EDGE-28M5, zx_edge:EDGE_28M5-2.54, symbol edge_lib:EDGE-28M5
- U16: footprint (none) -> Package_DIP:DIP-20_W7.62mm
- gave numbers to parts that had none: 1
- renumbered C4 to C5
Connections:
- net labels added: +9V, DI_ULA, ROMCS
- net labels removed: ~ROMCS
- wire segments 207 -> 281
- no-connect marks 0 -> 9
Other:
- moved on the sheet: U2E, U2F

Commit message: update schema
Parts:
- removed RN1: 10k, Resistor_THT:R_Array_SIP9, symbol Device:R_Network08_Split
- removed RN2: 10k, Resistor_THT:R_Array_SIP5, symbol Device:R_Network04_Split
- added RS1: 8x10k, Resistor_THT:R_Array_SIP9, symbol zx_custom_symbol:Resistor_Set_8
- added RS2: 4x10k, Resistor_THT:R_Array_SIP5, symbol zx_custom_symbol:Resistor_Set_4
- added U20: GAL16V8, symbol Gal:GAL16V8
- SW1: footprint (none) -> Button_Switch_THT:SW_Tactile_SPST_Angled_PTS645Vx39-2LFS
Connections:
- net labels added: BC1, BDIR, CLK-REG-32765, DI-PORT-32765, DO-PORT-32765, IN-254, OUT-254, ~A5
- net labels removed: BUSRQ
- wire segments 281 -> 284
Other:
- note added: "BOTTOM"
- note added: "TOP"
- moved on the sheet: R8, R9

Commit message: improve schema for CPU, Generator, Power_Sources units
Parts:
- renumbered 1N4148 to 1N1, R7 to R6, R9 to R7, U16 to U15, U18 to U16, U19 to U17, U15 to U18, U17 to U19, U9 to U8
Changed lines of the file:
@@
 $Descr A4 11693 8268
 encoding utf-8
-Sheet 3 4
+Sheet 3 5
 Title "CPU unit"
 Date "28.05.2022"
@@
 $EndDescr
 $Comp
-L Zilog:Z80CPU U15
+L Zilog:Z80CPU U18
 U 1 1 62937C30
 P 2500 2200
-F 0 "U15" H 2500 3450 50  0000 C CNN
+F 0 "U18" H 2500 3450 50  0000 C CNN
 F 1 "Z80CPU" H 2500 950 50  0000 C CNN
 F 2 "Package_DIP:DIP-40_W15.24mm" H 1550 4550 50  0001 C CNN
@@
 $EndComp
 $Comp
-L 74IEC:74HC245 U16
+L 74IEC:74HC245 U15
 U 1 1 6293D735
 P 4400 1500
-F 0 "U16" H 4400 2050 50  0000 C CNN
+F 0 "U15" H 4400 2050 50  0000 C CNN
 F 1 "74HC245" H 4400 950 50  0000 C CNN
 F 2 "Package_DIP:DIP-20_W7.62mm" H 4400 1050 50  0001 C CNN
@@
 $EndComp
 $Comp
-L 74IEC:74HC244 U17
+L 74IEC:74HC244 U19
 U 1 1 62942C60
 P 4400 2650
-F 0 "U17" H 4400 2950 50  0000 C CNN
+F 0 "U19" H 4400 2950 50  0000 C CNN
 F 1 "74HC244" H 4400 2350 50  0000 C CNN
 F 2 "Package_DIP:DIP-20_W7.62mm" H 4400 2350 50  0001 C CNN
@@
 $EndComp
 $Comp
-L 74IEC:74HC244 U17
+L 74IEC:74HC244 U19
 U 2 1 6294532D
 P 4400 3450
-F 0 "U17" H 4400 3750 50  0000 C CNN
+F 0 "U19" H 4400 3750 50  0000 C CNN
 F 1 "74HC244" H 4400 3150 50  0000 C CNN
 F 2 "Package_DIP:DIP-20_W7.62mm" H 4400 3150 50  0001 C CNN
@@
 $Comp
 L 74IEC:74HC14 U2
-U 3 1 6294A0A1
+U 4 1 6294A0A1
 P 6300 3100
 F 0 "U2" H 6300 3250 50  0000 C CNN
@@
 F 2 "Package_DIP:DIP-14_W7.62mm" H 6300 3310 50  0001 C CNN
 F 3 "https://www.ti.com/lit/ug/scyd013b/scyd013b.pdf" H 6300 3310 50  0001 C CNN
-	3    6300 3100
+	4    6300 3100
 	1    0    0    -1
 $EndComp
 $Comp
 L 74IEC:74HC14 U2
-U 4 1 6294B2DD
+U 3 1 6294B2DD
 P 5800 2700
 F 0 "U2" H 5800 2850 50  0000 C CNN
@@
 F 2 "Package_DIP:DIP-14_W7.62mm" H 5800 2910 50  0001 C CNN
 F 3 "https://www.ti.com/lit/ug/scyd013b/scyd013b.pdf" H 5800 2910 50  0001 C CNN
-	4    5800 2700
+	3    5800 2700
 	1    0    0    -1
 $EndComp
@@
 $EndComp
 $Comp
-L power:VCC #PWR0115
+L power:VCC #PWR0110
 U 1 1 62C7E0CF
 P 1050 1700
-F 0 "#PWR0115" H 1050 1550 50  0001 C CNN
+F 0 "#PWR0110" H 1050 1550 50  0001 C CNN
 F 1 "VCC" H 1065 1873 50  0000 C CNN
 F 2 "" H 1050 1700 50  0001 C CNN
@@
 xD0
 $Comp
-L 74IEC:74HC541 U18
+L 74IEC:74HC541 U16
 U 1 1 6295A588
 P 6050 1500
-F 0 "U18" H 6050 2050 50  0000 C CNN
+F 0 "U16" H 6050 2050 50  0000 C CNN
 F 1 "74HC541" H 6050 850 50  0000 C CNN
 F 2 "Package_DIP:DIP-20_W7.62mm" H 6050 2050 50  0001 C CNN
@@
 $EndComp
 $Comp
-L 74IEC:74HC541 U19
+L 74IEC:74HC541 U17
 U 1 1 62977052
 P 7350 1500
-F 0 "U19" H 7350 2050 50  0000 C CNN
+F 0 "U17" H 7350 2050 50  0000 C CNN
 F 1 "74HC541" H 7350 850 50  0000 C CNN
 F 2 "Package_DIP:DIP-20_W7.62mm" H 7350 2050 50  0001 C CNN
@@
 BUSACK
 $Comp
-L power:GND #PWR0116
+L power:GND #PWR0111
 U 1 1 6312142A
 P 4000 3750
-F 0 "#PWR0116" H 4000 3500 50  0001 C CNN
+F 0 "#PWR0111" H 4000 3500 50  0001 C CNN
 F 1 "GND" H 4005 3577 50  0000 C CNN
 F 2 "" H 4000 3750 50  0001 C CNN
@@
 	3900 1850 4100 1850
 $Comp
-L 74IEC:74HC00 U9
+L 74IEC:74HC00 U8
 U 2 1 63258955
 P 5800 3100
-F 0 "U9" H 5800 3250 50  0000 C CNN
+F 0 "U8" H 5800 3250 50  0000 C CNN
 F 1 "74HC00" H 5800 2950 50  0000 C CNN
 F 2 "" H 5800 2850 50  0001 C CNN
@@
 D1
 $Comp
-L power:VCC #PWR0117
+L power:VCC #PWR0112
 U 1 1 633F9ACA
 P 6000 3500
-F 0 "#PWR0117" H 6000 3350 50  0001 C CNN
+F 0 "#PWR0112" H 6000 3350 50  0001 C CNN
 F 1 "VCC" H 6015 3673 50  0000 C CNN
 F 2 "" H 6000 3500 50  0001 C CNN
@@
 	1050 2200 1900 2200
 $Comp
-L Device:R R7
+L Device:R R6
 U 1 1 63686836
 P 1050 2600
-F 0 "R7" V 950 2650 50  0000 R CNN
+F 0 "R6" V 950 2650 50  0000 R CNN
 F 1 "680" V 1150 2650 50  0000 R CNN
 F 2 "Resistor_SMD:R_0805_2012Metric" V 980 2600 50  0001 C CNN
@@
 $EndComp
 $Comp
-L Device:R R9
+L Device:R R7
 U 1 1 637254A8
 P 3000 4200
-F 0 "R9" H 2950 4300 50  0000 R CNN
+F 0 "R7" H 2950 4300 50  0000 R CNN
 F 1 "10k" H 2950 4100 50  0000 R CNN
 F 2 "Resistor_SMD:R_0805_2012Metric" V 2930 4200 50  0001 C CNN
@@
 $EndComp
 $Comp
-L Device:D 1N4148
+L Device:D 1N1
 U 1 1 6373C550
 P 2550 4200
-F 0 "1N4148" V 2650 4050 50  0000 C CNN
+F 0 "1N1" V 2650 4050 50  0000 C CNN
 F 1 "D2" V 2450 4100 50  0000 C CNN
 F 2 "" H 2550 4200 50  0001 C CNN
@@
 $EndComp
 $Comp
-L power:GND #PWR0118
+L power:GND #PWR0113
 U 1 1 637DCF1B
 P 1950 5100
-F 0 "#PWR0118" H 1950 4850 50  0001 C CNN
+F 0 "#PWR0113" H 1950 4850 50  0001 C CNN
 F 1 "GND" H 1955 4927 50  0000 C CNN
 F 2 "" H 1950 5100 50  0001 C CNN
@@
 	3000 4000 3000 4050
 $Comp
-L power:VCC #PWR0119
+L power:VCC #PWR0114
 U 1 1 63832BA6
 P 2550 3950
-F 0 "#PWR0119" H 2550 3800 50  0001 C CNN
+F 0 "#PWR0114" H 2550 3800 50  0001 C CNN
 F 1 "VCC" H 2565 4123 50  0000 C CNN
 F 2 "" H 2550 3950 50  0001 C CNN
@@
 	9200 1550 9300 1550
 $Comp
-L power:GND #PWR0120
+L power:GND #PWR0115
 U 1 1 63964F32
 P 9200 1500
-F 0 "#PWR0120" H 9200 1250 50  0001 C CNN
+F 0 "#PWR0115" H 9200 1250 50  0001 C CNN
 F 1 "GND" V 9205 1372 50  0000 R CNN
 F 2 "" H 9200 1500 50  0001 C CNN
@@
 	9200 1500 9200 1550
 $Comp
-L power:VCC #PWR0121
+L power:VCC #PWR0116
 U 1 1 639DDDB7
 P 9300 1150
-F 0 "#PWR0121" H 9300 1000 50  0001 C CNN
+F 0 "#PWR0116" H 9300 1000 50  0001 C CNN
 F 1 "VCC" V 9315 1278 50  0000 L CNN
 F 2 "" H 9300 1150 50  0001 C CNN
@@
 $EndComp
 $Comp
-L power:+9V #PWR0122
+L power:+9V #PWR0117
 U 1 1 639DECDB
 P 9200 1250
-F 0 "#PWR0122" H 9200 1100 50  0001 C CNN
+F 0 "#PWR0117" H 9200 1100 50  0001 C CNN
 F 1 "+9V" V 9215 1378 50  0000 L CNN
 F 2 "" H 9200 1250 50  0001 C CNN
@@
 ~NMI
 $Comp
-L power:GND #PWR0123
+L power:GND #PWR0118
 U 1 1 63C54EB1
 P 9200 2250
-F 0 "#PWR0123" H 9200 2000 50  0001 C CNN
+F 0 "#PWR0118" H 9200 2000 50  0001 C CNN
 F 1 "GND" V 9205 2122 50  0000 R CNN
 F 2 "" H 9200 2250 50  0001 C CNN
@@
 $Comp
 L 74IEC:74HC14 U2
-U 6 1 6294DA85
+U 5 1 6294DA85
 P 3950 4500
 F 0 "U2" H 3950 4650 50  0000 C CNN
@@
 F 2 "Package_DIP:DIP-14_W7.62mm" H 3950 4710 50  0001 C CNN
 F 3 "https://www.ti.com/lit/ug/scyd013b/scyd013b.pdf" H 3950 4710 50  0001 C CNN
-	6    3950 4500
+	5    3950 4500
 	1    0    0    -1
 $EndComp
 $Comp
 L 74IEC:74HC14 U2
-U 5 1 6294C1A0
+U 6 1 6294C1A0
 P 4450 4500
 F 0 "U2" H 4450 4650 50  0000 C CNN
@@
 F 2 "Package_DIP:DIP-14_W7.62mm" H 4450 4710 50  0001 C CNN
 F 3 "https://www.ti.com/lit/ug/scyd013b/scyd013b.pdf" H 4450 4710 50  0001 C CNN
-	5    4450 4500
-	1    0    0    -1
-$EndComp
+	6    4450 4500
+	1    0    0    -1
+$EndComp
