File: ZX-Spectrum-Pentagon/Input_Output.sch (KiCad schematic (older format))
At the start: 0 parts

Commit message: Modefied Input_Output sheet add schema for AY-3-8910-8912-8913 modefied AY-3-8910-8912-8913 symbol add LM311 symbol
Parts:
- added CIO? (x2): 150nF, symbol Device:C
- added CIO?: 10uF/6v, symbol Device:CP
- added CIO?: 1nF, symbol Device:C
- added CIO? (x4): C, symbol Device:C
- added CIO?: 3.3nF, symbol Device:C
- added CIO? (x2): 10uF/6V, symbol Device:CP
- added CIO?: CP, symbol Device:CP
- added DIO? (x2): KZ140, symbol Device:D_Zener
- added DIO? (x9): 1N4148, symbol Device:D
- added JIO?: Conn_01x02_Female, Connector_PinSocket_2.54mm:PinSocket_1x02_P2.54mm_Vertical, symbol Connector:Conn_01x02_Female
- added JIOA?, JIOB?, JIOKB?: Conn_01x08_Female, Connector_PinSocket_2.54mm:PinSocket_1x08_P2.54mm_Vertical, symbol Connector:Conn_01x08_Female
- added JIOKB?: Conn_01x05_Female, Connector_PinSocket_2.54mm:PinSocket_1x05_P2.54mm_Vertical, symbol Connector:Conn_01x05_Female
- added LIO?: 100uH, symbol Device:L
- added RIO?: 1k, Resistor_SMD:R_0805_2012Metric, symbol Device:R
- added RIO?: 47k, Resistor_SMD:R_0805_2012Metric, symbol Device:R
- added RIO?: 2.2k, Resistor_SMD:R_0805_2012Metric, symbol Device:R
- added RIO? (x3): 330, Resistor_SMD:R_0805_2012Metric, symbol Device:R
- added RIO? (x4): R, Resistor_SMD:R_0805_2012Metric, symbol Device:R
- added RIO? (x3): 4.7k, Resistor_SMD:R_0805_2012Metric, symbol Device:R
- added RIO? (x2): 3.0k, Resistor_SMD:R_0805_2012Metric, symbol Device:R
- added RIO?: 160, Resistor_SMD:R_0805_2012Metric, symbol Device:R
- added RSI0?: 8x10k, Resistor_THT:R_Array_SIP9, symbol ZX-Spectrum-Pentagon-rescue:Resistor_Set_8-zx_custom_symbol-ZX-Spectrum-Pentago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
- added SWIO?: SW_Push_DPDT, symbol Switch:SW_Push_DPDT
- added U24: 74HC174, symbol 74IEC:74HC174
- added U25: 74HC244, symbol 74IEC:74HC244
- added U26: LM311, symbol ZX-Spectrum-Pentagon-rescue:LM311-zx_custom_symbol-ZX-Spectrum-Pentagon-rescue
- added U?: AY-3-8913_DUMMY, symbol zx_custom_symbol:AY-3-8913_DUMMY
- added U?: AY-3-8910, symbol zx_custom_symbol:AY-3-8910
- added U?: AY-3-8912_DUMMY, symbol zx_custom_symbol:AY-3-8912_DUMMY
Connections:
- net labels added: A10, A11, A12, A13, A14, A15, A8, A9, AY-CLK, AYA8, AY~A9, AY~CS, BC1, BC2, BDIR, CBRD0, CBRD1, CBRD2, CHA, CHB, CHC, D0, D1, D2, D3, D4, D5, D6, D7, GND, IN-254, IND5, IND7, IOA0, IOA1, IOA2, IOA3, IOA4, IOA5, IOA6, IOA7, IOB0, IOB1, IOB2, IOB3, IOB4, IOB5, IOB6, IOB7, KBA10, KBA11, KBA12, KBA13, KBA14, KBA15, KBA8, KBA9, KBD0, KBD1, KBD2, KBD3, KBD4, OUT-254, TapeIn, TapeOut, VCC, ~RST
- wire segments 0 -> 283
- no-connect marks 0 -> 7
Other:
- note added: "AY-mixing\nchanels ABC/ACB\n"

Commit message: restore library
Parts:
- removed RSI0?: 8x10k, Resistor_THT:R_Array_SIP9, symbol ZX-Spectrum-Pentagon-rescue:Resistor_Set_8-zx_custom_symbol-ZX-Spectrum-Pentago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
- removed U26: LM311, symbol ZX-Spectrum-Pentagon-rescue:LM311-zx_custom_symbol-ZX-Spectrum-Pentagon-rescue
- added RSIO?: 8x10k, symbol zx_custom_symbol:Resistor_Set_8
- added U?: LM311, symbol zx_custom_symbol:LM311
Changed lines of the file:
@@
-$EndComp
-$Comp
-L ZX-Spectrum-Pentagon-rescue:LM311-zx_custom_symbol-ZX-Spectrum-Pentagon-rescue U26
-U 1 1 62C2C360
-P 5100 3800
-F 0 "U26" H 5250 4000 50  0000 L CNN
-F 1 "LM311" H 5150 3650 50  0000 L CNN
-F 2 "" H 5100 3800 50  0001 C CNN
-F 3 "https://www.st.com/resource/en/datasheet/lm311.pdf" H 5100 3800 50  0001 C CNN
-	1    5100 3800
-	1    0    0    -1
-$EndComp
-$Comp
-L ZX-Spectrum-Pentagon-rescue:Resistor_Set_8-zx_custom_symbol-ZX-Spectrum-Pentagon-rescue RSI0?
-U 1 1 62C2EC5F
-P 2650 5400
-F 0 "RSI0?" V 2800 5600 50  0000 C CNN
-F 1 "8x10k" V 2800 5150 50  0000 C CNN
-F 2 "Resistor_THT:R_Array_SIP9" H 2670 5850 50  0001 C CNN
-F 3 "" H 2670 5850 50  0001 C CNN
-	1    2650 5400
-	0    -1   -1   0
 $EndComp
 $Comp
@@
 Wire Wire Line
 	3800 1900 3800 1750
+$Comp
+L zx_custom_symbol:LM311 U?
+U 1 1 63A0DC84
+P 5100 3800
+F 0 "U?" H 5444 3846 50  0000 L CNN
+F 1 "LM311" H 5444 3755 50  0000 L CNN
+F 2 "" H 5100 3800 50  0001 C CNN
+F 3 "https://www.st.com/resource/en/datasheet/lm311.pdf" H 5100 3800 50  0001 C CNN
+	1    5100 3800
+	1    0    0    -1
+$EndComp
 Wire Bus Line
 	11150 1200 11150 3500
@@
 Wire Bus Line
 	7650 1150 7650 3500
+$Comp
+L zx_custom_symbol:Resistor_Set_8 RSIO?
+U 1 1 62A48178
+P 2650 5400
+F 0 "RSIO?" V 2800 5600 50  0000 C CNN
+F 1 "8x10k" V 2800 5150 50  0000 C CNN
+F 2 "" H 2670 5850 50  0001 C CNN
+F 3 "" H 2670 5850 50  0001 C CNN
+	1    2650 5400
+	0    -1   -1   0
+$EndComp
 $EndSCHEMATC

Commit message: some updates
Parts:
- removed CIO?: C, symbol Device:C
- removed CIO?: CP, symbol Device:CP
- removed LIO?: 100uH, symbol Device:L
- removed U24: 74HC174, symbol 74IEC:74HC174
- added JIO? (x2): AudioJack, Connector_Audio:Jack_3.5mm_CUI_SJ1-3535NG_Horizontal, symbol zx_custom_symbol:AudioJack
- added JIO?: Conn_01x03_Female, Connector_PinSocket_2.54mm:PinSocket_1x03_P2.54mm_Vertical, symbol Connector:Conn_01x03_Female
- added U?: 74HC273, Package_DIP:DIP-20_W7.62mm, symbol 74IEC:74HC273
- CIO? (x2): value C -> 150nF
- CIO?: value C -> 100nF
- RIO?: value R -> 10k
- RIO? (x2): value R -> 47k
- RIO?: value R -> 100k
- RSIO?: footprint (none) -> Resistor_THT:R_Array_SIP9
- SWIO?: footprint (none) -> Button_Switch_THT:SW_E-Switch_EG2219_DPDT_Angled
- U?: footprint (none) -> Package_DIP:DIP-24_W15.24mm
- U? (x2): renamed from U25; footprint (none) -> Package_DIP:DIP-20_W7.62mm
- U?: footprint (none) -> Package_DIP:DIP-40_W15.24mm
- U?: footprint (none) -> Package_DIP:DIP-28_W15.24mm
- U?: footprint (none) -> Package_DIP:DIP-8_W7.62mm
Connections:
- net labels added: AY-POWER, AudioIntL, AudioIntR, OURD5, OURD6, OURD7
- wire segments 283 -> 335
Other:
- moved on the sheet: CIO?, RIO?

Commit message: add Memory sheet, some changes on CPU sheet
Parts:
- CIO? (x9): footprint (none) -> Capacitor_SMD:C_0805_2012Metric_Pad1.18x1.45mm_HandSolder
- CIO?: footprint (none) -> Capacitor_Tantalum_SMD:CP_EIA-3528-21_Kemet-B_Pad1.50x2.35mm_HandSolder
- DIO? (x11): footprint (none) -> Diode_SMD:D_SOD-323_HandSoldering
- RIO?: value 1k -> 1kOm; footprint Resistor_SMD:R_0805_2012Metric -> Resistor_SMD:R_0805_2012Metric_Pad1.20x1.40mm_HandSolder
- RIO? (x3): value 47k -> 47kOm; footprint Resistor_SMD:R_0805_2012Metric -> Resistor_SMD:R_0805_2012Metric_Pad1.20x1.40mm_HandSolder
- RIO?: value 2.2k -> 2.2kOm; footprint Resistor_SMD:R_0805_2012Metric -> Resistor_SMD:R_0805_2012Metric_Pad1.20x1.40mm_HandSolder
- RIO? (x4): footprint Resistor_SMD:R_0805_2012Metric -> Resistor_SMD:R_0805_2012Metric_Pad1.20x1.40mm_HandSolder
- RIO?: value 10k -> 10kOm; footprint Resistor_SMD:R_0805_2012Metric -> Resistor_SMD:R_0805_2012Metric_Pad1.20x1.40mm_HandSolder
- RIO? (x3): value 4.7k -> 4.7kOm; footprint Resistor_SMD:R_0805_2012Metric -> Resistor_SMD:R_0805_2012Metric_Pad1.20x1.40mm_HandSolder
- RIO? (x2): value 3.0k -> 3.0kOm; footprint Resistor_SMD:R_0805_2012Metric -> Resistor_SMD:R_0805_2012Metric_Pad1.20x1.40mm_HandSolder
- RIO?: value 100k -> 100kOm; footprint Resistor_SMD:R_0805_2012Metric -> Resistor_SMD:R_0805_2012Metric_Pad1.20x1.40mm_HandSolder
- RSIO?: value 8x10k -> 8x10kOm

Commit message: rename some signal
Connections:
- net labels added: CBRDB, CBRDG, CBRDR
- net labels removed: CBRD0, CBRD1, CBRD2
Changed lines of the file:
@@
 D5
 Text GLabel -4950 -12050 2    50   Output ~ 10
-CBRD0
+CBRDB
 Text GLabel 3000 1450 2    50   Output ~ 10
-CBRD0
+CBRDB
 Text GLabel 3000 1550 2    50   Output ~ 10
-CBRD1
+CBRDR
 Text GLabel 3000 1650 2    50   Output ~ 10
-CBRD2
+CBRDG
 Wire Wire Line
 	2550 1450 3000 1450
