File: ZX-Spectrum-Pentagon/Memory.sch (KiCad schematic (older format))
At the start: 9 parts

Commit message: improve memory sheet
Parts:
- removed U?: 74HC245, symbol 74IEC:74HC245
- added U?: HM628512, symbol GenericSRAM:HM628512
- added U?: 74HC32, symbol 74IEC:74HC32
- added U?: 74HC541, symbol 74IEC:74HC541
Connections:
- net labels added: GAP6, GAP7, GND, MA0, MA1, MA10, MA11, MA12, MA13, MA14, MA15, MA16, MA17, MA18, MA2, MA3, MA4, MA5, MA6, MA7, MA8, MA9, MD0, MD1, MD2, MD3, MD4, MD5, MD6, MD7, MX0, MX1, MX2, MX3, SCRSEL, VCC, ~CAS
- net labels removed: A, AM0, AM1, AM10, AM11, AM12, AM13, AM14, AM15, AM17, AM18, AM2, AM3, AM4, AM5, AM6, AM7, AM8, AM9, B, C33, C34, C35, C37, DM0, DM1, DM2, DM3, DM4, DM5, DM6, DM7, MX4
- wire segments 114 -> 199
Other:
- moved on the sheet: U?A

Commit message: cd cd c
Parts:
- U?: footprint (none) -> Package_DIP:DIP-32_W15.24mm
- U? (x4): footprint (none) -> Package_DIP:DIP-14_W7.62mm
- U? (x2): footprint (none) -> Package_DIP:DIP-20_W7.62mm
- U? (x4): footprint (none) -> Package_DIP:DIP-16_W7.62mm
Changed lines of the file:
@@
 $Descr A4 11693 8268
 encoding utf-8
-Sheet 8 8
+Sheet 8 9
 Title ""
 Date ""
@@
 F 0 "U?" H 2300 1850 50  0000 C CNN
 F 1 "74HC257" H 2300 750 50  0000 C CNN
-F 2 "" H 2850 1350 50  0001 C CNN
+F 2 "Package_DIP:DIP-16_W7.62mm" H 2850 1350 50  0001 C CNN
 F 3 "https://www.ti.com/lit/ug/scyd013b/scyd013b.pdf" H 2850 1350 50  0001 C CNN
 	1    2300 1300
@@
 F 0 "U?" H 2300 3350 50  0000 C CNN
 F 1 "74HC257" H 2300 2250 50  0000 C CNN
-F 2 "" H 2850 2850 50  0001 C CNN
+F 2 "Package_DIP:DIP-16_W7.62mm" H 2850 2850 50  0001 C CNN
 F 3 "https://www.ti.com/lit/ug/scyd013b/scyd013b.pdf" H 2850 2850 50  0001 C CNN
 	1    2300 2800
@@
 F 0 "U?" H 2300 4850 50  0000 C CNN
 F 1 "74HC257" H 2300 3750 50  0000 C CNN
-F 2 "" H 2850 4350 50  0001 C CNN
+F 2 "Package_DIP:DIP-16_W7.62mm" H 2850 4350 50  0001 C CNN
 F 3 "https://www.ti.com/lit/ug/scyd013b/scyd013b.pdf" H 2850 4350 50  0001 C CNN
 	1    2300 4300
@@
 F 0 "U?" H 2800 7100 50  0000 C CNN
 F 1 "74HC08" H 2800 6800 50  0000 C CNN
-F 2 "" H 2800 6650 50  0001 C CNN
+F 2 "Package_DIP:DIP-14_W7.62mm" H 2800 6650 50  0001 C CNN
 F 3 "https://www.ti.com/lit/ug/scyd013b/scyd013b.pdf" H 2800 7100 50  0001 C CNN
 	2    2800 6950
@@
 F 0 "U?" H 2800 7500 50  0000 C CNN
 F 1 "74HC08" H 2800 7200 50  0000 C CNN
-F 2 "" H 2800 7050 50  0001 C CNN
+F 2 "Package_DIP:DIP-14_W7.62mm" H 2800 7050 50  0001 C CNN
 F 3 "https://www.ti.com/lit/ug/scyd013b/scyd013b.pdf" H 2800 7500 50  0001 C CNN
 	4    2800 7350
@@
 F 0 "U?" H 2150 7050 50  0000 C CNN
 F 1 "74HC08" H 2150 6750 50  0000 C CNN
-F 2 "" H 2150 6600 50  0001 C CNN
+F 2 "Package_DIP:DIP-14_W7.62mm" H 2150 6600 50  0001 C CNN
 F 3 "https://www.ti.com/lit/ug/scyd013b/scyd013b.pdf" H 2150 7050 50  0001 C CNN
 	1    2150 6900
@@
 F 0 "U?" H 2300 6350 50  0000 C CNN
 F 1 "74HC257" H 2300 5250 50  0000 C CNN
-F 2 "" H 2850 5850 50  0001 C CNN
+F 2 "Package_DIP:DIP-16_W7.62mm" H 2850 5850 50  0001 C CNN
 F 3 "https://www.ti.com/lit/ug/scyd013b/scyd013b.pdf" H 2850 5850 50  0001 C CNN
 	1    2300 5800
@@
 F 0 "U?" H 5750 1900 50  0000 C CNN
 F 1 "74HC541" H 5750 700 50  0000 C CNN
-F 2 "" H 5750 1900 50  0001 C CNN
+F 2 "Package_DIP:DIP-20_W7.62mm" H 5750 1900 50  0001 C CNN
 F 3 "https://www.ti.com/lit/ug/scyd013b/scyd013b.pdf" H 5750 1900 50  0001 C CNN
 	1    5750 1350
@@
 F 0 "U?" H 4300 3050 50  0000 C CNN
 F 1 "HM628512" H 4300 750 50  0000 C CNN
-F 2 "" H 4300 3050 50  0001 C CNN
+F 2 "Package_DIP:DIP-32_W15.24mm" H 4300 3050 50  0001 C CNN
 F 3 "" H 4300 3050 50  0001 C CNN
 	1    4300 1900
@@
 F 0 "U?" H 2800 6700 50  0000 C CNN
 F 1 "74HC32" H 2800 6400 50  0000 C CNN
-F 2 "" H 2800 6250 50  0001 C CNN
+F 2 "Package_DIP:DIP-14_W7.62mm" H 2800 6250 50  0001 C CNN
 F 3 "https://www.ti.com/lit/ug/scyd013b/scyd013b.pdf" H 2800 6700 50  0001 C CNN
 	1    2800 6550
@@
 F 0 "U?" H 5750 3250 50  0000 C CNN
 F 1 "74HC574" H 5750 2150 50  0000 C CNN
-F 2 "" H 5750 2400 50  0001 C CNN
+F 2 "Package_DIP:DIP-20_W7.62mm" H 5750 2400 50  0001 C CNN
 F 3 "https://www.ti.com/lit/ug/scyd013b/scyd013b.pdf" H 5750 2400 50  0001 C CNN
 	1    5750 2700

Commit message: rename some signal
Changed lines of the file:
@@
 MD7
 Wire Bus Line
-	6450 700  6450 3450
+	6450 700  6450 2950
 Wire Bus Line
-	5000 700  5000 3700
+	5000 700  5000 3050
 Wire Bus Line
 	3400 700  3400 7700

Commit message: reset anatation
Changed lines of the file:
@@
 $Comp
 L 74IEC:74HC08 U?
-U 2 1 64281E3C
+U 4 1 64281E3C
 P 2800 6950
 F 0 "U?" H 2800 7100 50  0000 C CNN
@@
 F 2 "Package_DIP:DIP-14_W7.62mm" H 2800 6650 50  0001 C CNN
 F 3 "https://www.ti.com/lit/ug/scyd013b/scyd013b.pdf" H 2800 7100 50  0001 C CNN
-	2    2800 6950
+	4    2800 6950
 	1    0    0    -1
 $EndComp
 $Comp
 L 74IEC:74HC08 U?
-U 4 1 64284777
+U 1 1 64284777
 P 2800 7350
 F 0 "U?" H 2800 7500 50  0000 C CNN
@@
 F 2 "Package_DIP:DIP-14_W7.62mm" H 2800 7050 50  0001 C CNN
 F 3 "https://www.ti.com/lit/ug/scyd013b/scyd013b.pdf" H 2800 7500 50  0001 C CNN
-	4    2800 7350
+	1    2800 7350
 	1    0    0    -1
 $EndComp
 $Comp
 L 74IEC:74HC08 U?
-U 1 1 64285960
+U 3 1 64285960
 P 2150 6900
 F 0 "U?" H 2150 7050 50  0000 C CNN
@@
 F 2 "Package_DIP:DIP-14_W7.62mm" H 2150 6600 50  0001 C CNN
 F 3 "https://www.ti.com/lit/ug/scyd013b/scyd013b.pdf" H 2150 7050 50  0001 C CNN
-	1    2150 6900
+	3    2150 6900
 	1    0    0    -1
 $EndComp
@@
 $Comp
 L 74IEC:74HC32 U?
-U 1 1 62EC474A
+U 4 1 62EC474A
 P 2800 6550
 F 0 "U?" H 2800 6700 50  0000 C CNN
@@
 F 2 "Package_DIP:DIP-14_W7.62mm" H 2800 6250 50  0001 C CNN
 F 3 "https://www.ti.com/lit/ug/scyd013b/scyd013b.pdf" H 2800 6700 50  0001 C CNN
-	1    2800 6550
+	4    2800 6550
 	1    0    0    -1
 $EndComp

Commit message: fix ERC in Memory.sch
Parts:
- gave numbers to parts that had none: 10
Connections:
- net labels removed: CAS

Commit message: fix ERC in Memory_Signal.sch
Connections:
- net labels removed: ~RAS
- wire segments 199 -> 198
Changed lines of the file:
@@
 Text GLabel 1000 4500 0    50   Input ~ 10
 ~CAS
-Text GLabel 1000 4650 0    50   Input ~ 10
-~RAS
 Text Label 1600 1650 0    50   ~ 0
 B4
@@
 Text Label 1400 4500 2    50   ~ 0
 ~CAS
-Entry Wire Line
-	1500 4550 1400 4650
-Wire Wire Line
-	1400 4650 1000 4650
-Text Label 1400 4650 2    50   ~ 0
-~RAS
 Entry Wire Line
 	1500 850  1400 950
@@
 Wire Wire Line
 	1950 6850 1600 6850
-Wire Bus Line
-	3400 700  3400 7700
-Wire Bus Line
-	1500 700  1500 7300
-Wire Bus Line
-	5000 700  5000 3050
-Wire Bus Line
-	6450 700  6450 2950
 Text Label 1600 3150 0    50   ~ 0
 SCRSEL
@@
 	1    0    0    -1
 $EndComp
+Wire Bus Line
+	6450 700  6450 2950
+Wire Bus Line
+	5000 700  5000 3050
+Wire Bus Line
+	3400 700  3400 7700
+Wire Bus Line
+	1500 700  1500 7300
 $EndSCHEMATC
