File: ZX-Spectrum-Pentagon/Video_Formating.sch (KiCad schematic (older format))
At the start: 10 parts

Commit message: improve Video_Formating
Parts:
- added QVF? (x4): BC548, symbol zx_custom_symbol:NPN
- added RVF? (x4): 2.2kOm, symbol Device:R
- added RVF? (x3): 3.9kOm, symbol Device:R
- added RVF? (x6): 68, symbol Device:R
- added RVF? (x3): 75, symbol Device:R
- added RVF? (x3): 18kOm, symbol Device:R
- added RVF?: 330, symbol Device:R
- added RVF?: 680, symbol Device:R
Connections:
- net labels added: 512KMOD, BLUE_B, BLUE_CN, BLUE_EN, BLUE_P, BRIGHT, C7, FLASL_BIT, GREEN_B, GREEN_CN, GREEN_EN, GREEN_P, RED_B, RED_CN, RED_EN, RED_P, SERDATA, SYNC, SYNCOUT
- wire segments 172 -> 273
- no-connect marks 0 -> 5
Other:
- note added: "128K/512K"
- note removed: "128k/512k"
- moved on the sheet: RVF?

Commit message: rename some signal
Parts:
- added J?: Mini-DIN-8, symbol Connector:Mini-DIN-8
Connections:
- net labels added: BLUE_F, CBRDB, CBRDG, CBRDR, F25Hz, GREEN_F, RED_F
- net labels removed: BLUE_P, CBRD0, CBRD1, CBRD2, F-25Hz, GREEN_P, RED_P
- wire segments 273 -> 270
Other:
- moved on the sheet: RVF?

Commit message: reset anatation
Parts:
- RVF? (x21): footprint (none) -> Resistor_SMD:R_0805_2012Metric_Pad1.20x1.40mm_HandSolder
- gave numbers to parts that had none: 1
Connections:
- net labels added: SYNCO
- net labels removed: C7
Changed lines of the file:
@@
 $Descr A4 11693 8268
 encoding utf-8
-Sheet 8 9
+Sheet 7 9
 Title ""
 Date ""
@@
 C3
 Text Label 1400 3700 2    50   ~ 0
-C7
+SYNC
 Text Label 1400 3800 2    50   ~ 0
 C17
@@
 P 4500 6550
 AR Path="/62A08194/638D500F" Ref="SWIO?"  Part="1"
-AR Path="/62FD43AB/638D500F" Ref="SVF?"  Part="1"
-F 0 "SVF?" H 4500 6950 50  0000 C CNN
+AR Path="/62FD43AB/638D500F" Ref="SWIO?"  Part="1"
+F 0 "SWIO?" H 4500 6950 50  0000 C CNN
 F 1 "SW_Push_DPDT" H 4500 6944 50  0001 C CNN
 F 2 "Button_Switch_THT:SW_E-Switch_EG2219_DPDT_Angled" H 4500 6750 50  0001 C CNN
@@
 F 0 "RVF?" H 9070 3646 50  0000 L CNN
 F 1 "75" H 9070 3555 50  0000 L CNN
-F 2 "" V 8930 3600 50  0001 C CNN
+F 2 "Resistor_SMD:R_0805_2012Metric_Pad1.20x1.40mm_HandSolder" V 8930 3600 50  0001 C CNN
 F 3 "~" H 9000 3600 50  0001 C CNN
 	1    9000 3600
@@
 F 0 "RVF?" H 9570 3646 50  0000 L CNN
 F 1 "75" H 9570 3555 50  0000 L CNN
-F 2 "" V 9430 3600 50  0001 C CNN
+F 2 "Resistor_SMD:R_0805_2012Metric_Pad1.20x1.40mm_HandSolder" V 9430 3600 50  0001 C CNN
 F 3 "~" H 9500 3600 50  0001 C CNN
 	1    9500 3600
@@
 F 0 "RVF?" H 9070 3146 50  0000 L CNN
 F 1 "68" H 9070 3055 50  0000 L CNN
-F 2 "" V 8930 3100 50  0001 C CNN
+F 2 "Resistor_SMD:R_0805_2012Metric_Pad1.20x1.40mm_HandSolder" V 8930 3100 50  0001 C CNN
 F 3 "~" H 9000 3100 50  0001 C CNN
 	1    9000 3100
@@
 F 0 "RVF?" H 9570 3146 50  0000 L CNN
 F 1 "68" H 9570 3055 50  0000 L CNN
-F 2 "" V 9430 3100 50  0001 C CNN
+F 2 "Resistor_SMD:R_0805_2012Metric_Pad1.20x1.40mm_HandSolder" V 9430 3100 50  0001 C CNN
 F 3 "~" H 9500 3100 50  0001 C CNN
 	1    9500 3100
@@
 F 0 "RVF?" H 8670 2196 50  0000 L CNN
 F 1 "2.2kOm" H 8670 2105 50  0000 L CNN
-F 2 "" V 8530 2150 50  0001 C CNN
+F 2 "Resistor_SMD:R_0805_2012Metric_Pad1.20x1.40mm_HandSolder" V 8530 2150 50  0001 C CNN
 F 3 "~" H 8600 2150 50  0001 C CNN
 	1    8600 2150
@@
 F 0 "RVF?" H 8570 3646 50  0000 L CNN
 F 1 "75" H 8570 3555 50  0000 L CNN
-F 2 "" V 8430 3600 50  0001 C CNN
+F 2 "Resistor_SMD:R_0805_2012Metric_Pad1.20x1.40mm_HandSolder" V 8430 3600 50  0001 C CNN
 F 3 "~" H 8500 3600 50  0001 C CNN
 	1    8500 3600
@@
 F 0 "RVF?" H 8170 1696 50  0000 L CNN
 F 1 "2.2kOm" H 8170 1605 50  0000 L CNN
-F 2 "" V 8030 1650 50  0001 C CNN
+F 2 "Resistor_SMD:R_0805_2012Metric_Pad1.20x1.40mm_HandSolder" V 8030 1650 50  0001 C CNN
 F 3 "~" H 8100 1650 50  0001 C CNN
 	1    8100 1650
@@
 F 0 "RVF?" H 8570 3146 50  0000 L CNN
 F 1 "68" H 8570 3055 50  0000 L CNN
-F 2 "" V 8430 3100 50  0001 C CNN
+F 2 "Resistor_SMD:R_0805_2012Metric_Pad1.20x1.40mm_HandSolder" V 8430 3100 50  0001 C CNN
 F 3 "~" H 8500 3100 50  0001 C CNN
 	1    8500 3100
@@
 F 0 "RVF?" V 7550 1250 50  0000 C CNN
 F 1 "3.9kOm" V 7550 1550 50  0000 C CNN
-F 2 "" V 7580 1400 50  0001 C CNN
+F 2 "Resistor_SMD:R_0805_2012Metric_Pad1.20x1.40mm_HandSolder" V 7580 1400 50  0001 C CNN
 F 3 "~" H 7650 1400 50  0001 C CNN
 	1    7650 1400
@@
 F 0 "RVF?" H 9170 2696 50  0000 L CNN
 F 1 "2.2kOm" H 9170 2605 50  0000 L CNN
-F 2 "" V 9030 2650 50  0001 C CNN
+F 2 "Resistor_SMD:R_0805_2012Metric_Pad1.20x1.40mm_HandSolder" V 9030 2650 50  0001 C CNN
 F 3 "~" H 9100 2650 50  0001 C CNN
 	1    9100 2650
@@
 F 0 "RVF?" V 7550 1750 50  0000 C CNN
 F 1 "3.9kOm" V 7550 2100 50  0000 C CNN
-F 2 "" V 7580 1900 50  0001 C CNN
+F 2 "Resistor_SMD:R_0805_2012Metric_Pad1.20x1.40mm_HandSolder" V 7580 1900 50  0001 C CNN
 F 3 "~" H 7650 1900 50  0001 C CNN
 	1    7650 1900
@@
 F 0 "RVF?" V 7550 2250 50  0000 C CNN
 F 1 "3.9kOm" V 7550 2550 50  0000 C CNN
-F 2 "" V 7580 2400 50  0001 C CNN
+F 2 "Resistor_SMD:R_0805_2012Metric_Pad1.20x1.40mm_HandSolder" V 7580 2400 50  0001 C CNN
 F 3 "~" H 7650 2400 50  0001 C CNN
 	1    7650 2400
@@
 F 0 "RVF?" V 7550 1500 50  0000 C CNN
 F 1 "18kOm" V 7550 1750 50  0000 C CNN
-F 2 "" V 7580 1650 50  0001 C CNN
+F 2 "Resistor_SMD:R_0805_2012Metric_Pad1.20x1.40mm_HandSolder" V 7580 1650 50  0001 C CNN
 F 3 "~" H 7650 1650 50  0001 C CNN
 	1    7650 1650
@@
 F 0 "RVF?" V 7550 1950 50  0000 C CNN
 F 1 "18kOm" V 7550 2200 50  0000 C CNN
-F 2 "" V 7580 2100 50  0001 C CNN
+F 2 "Resistor_SMD:R_0805_2012Metric_Pad1.20x1.40mm_HandSolder" V 7580 2100 50  0001 C CNN
 F 3 "~" H 7650 2100 50  0001 C CNN
 	1    7650 2100
@@
 F 0 "RVF?" V 7550 2450 50  0000 C CNN
 F 1 "18kOm" V 7550 2700 50  0000 C CNN
-F 2 "" V 7580 2600 50  0001 C CNN
+F 2 "Resistor_SMD:R_0805_2012Metric_Pad1.20x1.40mm_HandSolder" V 7580 2600 50  0001 C CNN
 F 3 "~" H 7650 2600 50  0001 C CNN
 	1    7650 2600
@@
 F 0 "RVF?" V 10100 1650 50  0000 C CNN
 F 1 "68" V 9900 1650 50  0000 C CNN
-F 2 "" V 9930 1650 50  0001 C CNN
+F 2 "Resistor_SMD:R_0805_2012Metric_Pad1.20x1.40mm_HandSolder" V 9930 1650 50  0001 C CNN
 F 3 "~" H 10000 1650 50  0001 C CNN
 	1    10000 1650
@@
 F 0 "RVF?" V 10100 2150 50  0000 C CNN
 F 1 "68" V 9900 2150 50  0000 C CNN
-F 2 "" V 9930 2150 50  0001 C CNN
+F 2 "Resistor_SMD:R_0805_2012Metric_Pad1.20x1.40mm_HandSolder" V 9930 2150 50  0001 C CNN
 F 3 "~" H 10000 2150 50  0001 C CNN
 	1    10000 2150
@@
 F 0 "RVF?" V 10100 2650 50  0000 C CNN
 F 1 "68" V 9900 2650 50  0000 C CNN
-F 2 "" V 9930 2650 50  0001 C CNN
+F 2 "Resistor_SMD:R_0805_2012Metric_Pad1.20x1.40mm_HandSolder" V 9930 2650 50  0001 C CNN
 F 3 "~" H 10000 2650 50  0001 C CNN
 	1    10000 2650
@@
 F 0 "RVF?" H 8550 4350 50  0000 L CNN
 F 1 "330" H 8550 4150 50  0000 L CNN
-F 2 "" V 8430 4250 50  0001 C CNN
+F 2 "Resistor_SMD:R_0805_2012Metric_Pad1.20x1.40mm_HandSolder" V 8430 4250 50  0001 C CNN
 F 3 "~" H 8500 4250 50  0001 C CNN
 	1    8500 4250
@@
 F 0 "RVF?" V 7850 5100 50  0000 C CNN
 F 1 "2.2kOm" V 8050 5100 50  0000 C CNN
-F 2 "" V 7880 5100 50  0001 C CNN
+F 2 "Resistor_SMD:R_0805_2012Metric_Pad1.20x1.40mm_HandSolder" V 7880 5100 50  0001 C CNN
 F 3 "~" H 7950 5100 50  0001 C CNN
 	1    7950 5100
@@
 F 0 "RVF?" V 7850 4800 50  0000 C CNN
 F 1 "680" V 8050 4800 50  0000 C CNN
-F 2 "" V 7880 4800 50  0001 C CNN
+F 2 "Resistor_SMD:R_0805_2012Metric_Pad1.20x1.40mm_HandSolder" V 7880 4800 50  0001 C CNN
 F 3 "~" H 7950 4800 50  0001 C CNN
 	1    7950 4800
@@
 SYNCOUT
 Text GLabel 10500 5300 2    50   Output ~ 10
-SYNC
+SYNCO
 Wire Wire Line
 	8500 3850 8500 4100
@@
 C5
 Text GLabel 1000 3700 0    50   Input ~ 10
-C7
+SYNC
 Text GLabel 1000 3800 0    50   Input ~ 10
 C17
@@
 	1500 4750 1600 4850
 Text Label 1600 4850 0    50   ~ 0
-C7
+SYNC
 $Comp
 L power:VCC #PWR?

Commit message: rename some signals
Connections:
- net labels added: FSYNC, SYNCTTL
- net labels removed: SYNC, SYNCO
Changed lines of the file:
@@
 C3
 Text Label 1400 3700 2    50   ~ 0
-SYNC
+FSYNC
 Text Label 1400 3800 2    50   ~ 0
 C17
@@
 SYNCOUT
 Text GLabel 10500 5300 2    50   Output ~ 10
-SYNCO
+SYNCTTL
 Wire Wire Line
 	8500 3850 8500 4100
@@
 C5
 Text GLabel 1000 3700 0    50   Input ~ 10
-SYNC
+FSYNC
 Text GLabel 1000 3800 0    50   Input ~ 10
 C17
@@
 	1500 4750 1600 4850
 Text Label 1600 4850 0    50   ~ 0
-SYNC
+FSYNC
 $Comp
 L power:VCC #PWR?

Commit message: add VideoEncoder sheet
Parts:
- removed J?: Mini-DIN-8, symbol Connector:Mini-DIN-8
- removed QVF? (x4): BC548, symbol zx_custom_symbol:NPN
- removed RVF? (x4): 2.2kOm, Resistor_SMD:R_0805_2012Metric_Pad1.20x1.40mm_HandSolder, symbol Device:R
- removed RVF? (x3): 3.9kOm, Resistor_SMD:R_0805_2012Metric_Pad1.20x1.40mm_HandSolder, symbol Device:R
- removed RVF? (x6): 68, Resistor_SMD:R_0805_2012Metric_Pad1.20x1.40mm_HandSolder, symbol Device:R
- removed RVF? (x3): 75, Resistor_SMD:R_0805_2012Metric_Pad1.20x1.40mm_HandSolder, symbol Device:R
- removed RVF? (x3): 18kOm, Resistor_SMD:R_0805_2012Metric_Pad1.20x1.40mm_HandSolder, symbol Device:R
- removed RVF?: 330, Resistor_SMD:R_0805_2012Metric_Pad1.20x1.40mm_HandSolder, symbol Device:R
- removed RVF?: 680, Resistor_SMD:R_0805_2012Metric_Pad1.20x1.40mm_HandSolder, symbol Device:R
- gave numbers to parts that had none: 1
Connections:
- net labels added: TTLB, TTLG, TTLR, TTLSYNC, TTLY
- net labels removed: BLUE_CN, BLUE_EN, GREEN_CN, GREEN_EN, RED_CN, RED_EN, SYNCOUT, SYNCTTL
- wire segments 270 -> 185

Commit message: fix ERC in Video_Formating.sch
Parts:
- gave numbers to parts that had none: 10
Connections:
- net labels removed: С5
- no-connect marks 5 -> 7
Changed lines of the file:
@@
 	1400 1700 1500 1600
 $Comp
-L 74IEC:74HC574 U?
+L 74IEC:74HC574 U29
 U 1 1 632C89BD
 P 2200 1500
-F 0 "U?" H 2200 2050 50  0000 C CNN
+F 0 "U29" H 2200 2050 50  0000 C CNN
 F 1 "74HC574" H 2200 950 50  0000 C CNN
 F 2 "Package_DIP:DIP-20_W7.62mm" H 2200 1200 50  0001 C CNN
@@
 $EndComp
 $Comp
-L 74IEC:74HC574 U?
+L 74IEC:74HC574 U30
 U 1 1 632CEC67
 P 3100 1600
-F 0 "U?" H 3100 2150 50  0000 C CNN
+F 0 "U30" H 3100 2150 50  0000 C CNN
 F 1 "74HC574" H 3100 1050 50  0000 C CNN
 F 2 "Package_DIP:DIP-20_W7.62mm" H 3100 1300 50  0001 C CNN
@@
 	2700 2050 2700 2150
 $Comp
-L power:GND #PWR?
+L power:GND #PWR0141
 U 1 1 632E6C13
 P 2700 2250
-F 0 "#PWR?" H 2700 2000 50  0001 C CNN
+F 0 "#PWR0141" H 2700 2000 50  0001 C CNN
 F 1 "GND" H 2705 2077 50  0000 C CNN
 F 2 "" H 2700 2250 50  0001 C CNN
@@
 C3
 $Comp
-L 74IEC:74HC574 U?
+L 74IEC:74HC574 U34
 U 1 1 6330BD21
 P 2200 6600
-F 0 "U?" H 2200 7150 50  0000 C CNN
+F 0 "U34" H 2200 7150 50  0000 C CNN
 F 1 "74HC574" H 2200 6050 50  0000 C CNN
 F 2 "Package_DIP:DIP-20_W7.62mm" H 2200 6300 50  0001 C CNN
@@
 P 3250 6650
 AR Path="/6332DE4B" Ref="U?"  Part="1"
-AR Path="/62FD43AB/6332DE4B" Ref="U?"  Part="1"
-F 0 "U?" H 3250 7350 50  0000 C CNN
+AR Path="/62FD43AB/6332DE4B" Ref="U35"  Part="1"
+F 0 "U35" H 3250 7350 50  0000 C CNN
 F 1 "74HC166" H 3250 5950 50  0000 C CNN
 F 2 "Package_DIP:DIP-16_W7.62mm" H 3250 6050 50  0001 C CNN
@@
 	2700 7050 2900 7050
 $Comp
-L power:GND #PWR?
+L power:GND #PWR0142
 U 1 1 63470A69
 P 1900 7150
-F 0 "#PWR?" H 1900 6900 50  0001 C CNN
+F 0 "#PWR0142" H 1900 6900 50  0001 C CNN
 F 1 "GND" H 1905 6977 50  0000 C CNN
 F 2 "" H 1900 7150 50  0001 C CNN
@@
 $EndComp
 $Comp
-L 74IEC:74XX153 U?
+L 74IEC:74XX153 U31
 U 1 1 63481D4A
 P 5350 1700
-F 0 "U?" H 5350 2350 50  0000 C CNN
+F 0 "U31" H 5350 2350 50  0000 C CNN
 F 1 "74XX153" H 5350 1050 50  0000 C CNN
 F 2 "Package_DIP:DIP-16_W7.62mm" H 5350 1750 50  0001 C CNN
@@
 $EndComp
 $Comp
-L 74IEC:74XX153 U?
+L 74IEC:74XX153 U32
 U 1 1 63485DD9
 P 5350 3500
-F 0 "U?" H 5350 4150 50  0000 C CNN
+F 0 "U32" H 5350 4150 50  0000 C CNN
 F 1 "74XX153" H 5350 2850 50  0000 C CNN
 F 2 "Package_DIP:DIP-16_W7.62mm" H 5350 3550 50  0001 C CNN
@@
 Wire Wire Line
 	4800 2250 4800 2850
-Wire Wire Line
-	4800 4050 5000 4050
 Wire Wire Line
 	4800 2050 4600 2050
@@
 	4800 2850 4800 4050
 Text Label 1600 2850 0    50   ~ 0
-С5
+C5
 Wire Wire Line
 	5000 1150 4900 1150
@@
 P 4500 6550
 AR Path="/62A08194/638D500F" Ref="SWIO?"  Part="1"
-AR Path="/62FD43AB/638D500F" Ref="SWVF?"  Part="1"
-F 0 "SWVF?" H 4500 6950 50  0000 C CNN
+AR Path="/62FD43AB/638D500F" Ref="SWIO1"  Part="1"
+F 0 "SWIO1" H 4500 6950 50  0000 C CNN
 F 1 "SW_Push_DPDT" H 4500 6944 50  0001 C CNN
 F 2 "Button_Switch_THT:SW_E-Switch_EG2219_DPDT_Angled" H 4500 6750 50  0001 C CNN
@@
 	4850 6650 4700 6650
 $Comp
-L power:GND #PWR?
+L power:GND #PWR0143
 U 1 1 6397C066
 P 4850 6950
-F 0 "#PWR?" H 4850 6700 50  0001 C CNN
+F 0 "#PWR0143" H 4850 6700 50  0001 C CNN
 F 1 "GND" H 4855 6777 50  0000 C CNN
 F 2 "" H 4850 6950 50  0001 C CNN
@@
 Connection ~ 4850 6650
 $Comp
-L Device:R RVF?
+L Device:R RVF1
 U 1 1 639A492B
 P 4200 6050
-F 0 "RVF?" H 3900 6150 50  0000 L CNN
+F 0 "RVF1" H 3900 6150 50  0000 L CNN
 F 1 "4.7kOm" H 3850 5900 50  0000 L CNN
 F 2 "Resistor_SMD:R_0805_2012Metric_Pad1.20x1.40mm_HandSolder" V 4130 6050 50  0001 C CNN
@@
 $EndComp
 $Comp
-L power:VCC #PWR?
+L power:VCC #PWR0144
 U 1 1 639BDFE6
 P 4200 5700
-F 0 "#PWR?" H 4200 5550 50  0001 C CNN
+F 0 "#PWR0144" H 4200 5550 50  0001 C CNN
 F 1 "VCC" H 4215 5873 50  0000 C CNN
 F 2 "" H 4200 5700 50  0001 C CNN
@@
 128K/512K
 $Comp
-L 74IEC:74HC86 U?
+L 74IEC:74HC86 U20
 U 4 1 63A0E5BA
 P 5400 5400
-F 0 "U?" H 5400 5550 50  0000 C CNN
+F 0 "U20" H 5400 5550 50  0000 C CNN
 F 1 "74HC86" H 5400 5250 50  0000 C CNN
 F 2 "" H 5400 5100 50  0001 C CNN
@@
 512KMOD
 $Comp
-L power:GND #PWR?
+L power:GND #PWR0145
 U 1 1 6334F3AB
 P 2800 7350
-F 0 "#PWR?" H 2800 7100 50  0001 C CNN
+F 0 "#PWR0145" H 2800 7100 50  0001 C CNN
 F 1 "GND" H 2805 7177 50  0000 C CNN
 F 2 "" H 2800 7350 50  0001 C CNN
@@
 Connection ~ 4900 3850
 $Comp
-L power:GND #PWR?
+L power:GND #PWR0146
 U 1 1 635A9564
 P 4900 4950
-F 0 "#PWR?" H 4900 4700 50  0001 C CNN
+F 0 "#PWR0146" H 4900 4700 50  0001 C CNN
 F 1 "GND" H 4905 4777 50  0000 C CNN
 F 2 "" H 4900 4950 50  0001 C CNN
@@
 	2750 4050 2750 3100
 $Comp
-L Gal:GAL16V8 U?
+L Gal:GAL16V8 U33
 U 1 1 637AE6C9
 P 3300 4300
-F 0 "U?" H 3300 4850 50  0000 C CNN
+F 0 "U33" H 3300 4850 50  0000 C CNN
 F 1 "GAL16V8" H 3300 3750 50  0000 C CNN
 F 2 "Package_DIP:DIP-20_W7.62mm" H 3300 4850 50  0001 C CNN
@@
 512KMOD
 $Comp
-L power:VCC #PWR?
+L power:VCC #PWR0147
 U 1 1 64647478
 P 2650 4750
-F 0 "#PWR?" H 2650 4600 50  0001 C CNN
+F 0 "#PWR0147" H 2650 4600 50  0001 C CNN
 F 1 "VCC" H 2665 4923 50  0000 C CNN
 F 2 "" H 2650 4750 50  0001 C CNN
@@
 	4700 4450 4700 3950
 Connection ~ 4700 3950
-Wire Bus Line
-	1500 950  1500 7500
 Text GLabel 6000 4650 2    50   Output ~ 10
 GPA6
@@
 Text GLabel 6000 1400 2    50   Output ~ 10
 TTLB
+NoConn ~ 4700 6450
+NoConn ~ 4700 6850
+Wire Wire Line
+	5000 4050 4800 4050
+Wire Bus Line
+	1500 950  1500 7500
 $EndSCHEMATC
