File: ZX-Spectrum-Pentagon/InputOutput.sch (KiCad schematic (older format))
At the start: 57 parts

Commit message: Rename schama sheet
Connections:
- wire segments 352 -> 351
Changed lines of the file:
@@
 Wire Wire Line
 	5000 3500 5000 3800
-Wire Wire Line
-	5000 3800 5000 3850
-Connection ~ 5000 3800
 $Comp
 L zx_custom_symbol:LM311 U?

Commit message: add footprints. prepare pcb for edge connector
Parts:
- CIO?: footprint Capacitor_SMD:C_0805_2012Metric_Pad1.18x1.45mm_HandSolder -> Package_TO_SOT_SMD:SOT-23_Handsoldering
- CIO? (x2): footprint Capacitor_SMD:C_0805_2012Metric_Pad1.18x1.45mm_HandSolder -> Capacitor_Tantalum_SMD:CP_EIA-3528-21_Kemet-B_Pad1.50x2.35mm_HandSolder
Changed lines of the file:
@@
 F 0 "CIO?" V 8500 4200 50  0000 C CNN
 F 1 "10uF/6V" V 8200 4200 50  0000 C CNN
-F 2 "Capacitor_SMD:C_0805_2012Metric_Pad1.18x1.45mm_HandSolder" H 8388 4050 50  0001 C CNN
+F 2 "Capacitor_Tantalum_SMD:CP_EIA-3528-21_Kemet-B_Pad1.50x2.35mm_HandSolder" H 8388 4050 50  0001 C CNN
 F 3 "~" H 8350 4200 50  0001 C CNN
 	1    8350 4200
@@
 F 0 "CIO?" H 3250 3400 50  0000 C CNN
 F 1 "3.3nF" H 3250 3200 50  0000 C CNN
-F 2 "Capacitor_SMD:C_0805_2012Metric_Pad1.18x1.45mm_HandSolder" H 3438 3150 50  0001 C CNN
+F 2 "Package_TO_SOT_SMD:SOT-23_Handsoldering" H 3438 3150 50  0001 C CNN
 F 3 "~" H 3400 3300 50  0001 C CNN
 	1    3400 3300
@@
 F 0 "CIO?" V 8500 5100 50  0000 C CNN
 F 1 "10uF/6V" V 8200 5100 50  0000 C CNN
-F 2 "Capacitor_SMD:C_0805_2012Metric_Pad1.18x1.45mm_HandSolder" H 8388 4950 50  0001 C CNN
+F 2 "Capacitor_Tantalum_SMD:CP_EIA-3528-21_Kemet-B_Pad1.50x2.35mm_HandSolder" H 8388 4950 50  0001 C CNN
 F 3 "~" H 8350 5100 50  0001 C CNN
 	1    8350 5100

Commit message: set annotate
Parts:
- gave numbers to parts that had none: 56
