File: ZX-Spectrum-Pentagon/MemorySignal.sch (KiCad schematic (older format))
At the start: 5 parts, among them U11 74HC74, U12 74HC273, U13 74HC257, U7 74HC00

Commit message: reset annotate and update CPU for new symbol
Parts:
- renumbered CM1 to CM?, U12 to U?, U13 to U?, U7 to U?, U11 to U?
Changed lines of the file:
@@
 $EndDescr
 $Comp
-L 74IEC:74HC273 U12
+L 74IEC:74HC273 U?
 U 1 1 630C4800
 P 2200 4000
-F 0 "U12" H 2200 4550 50  0000 C CNN
+F 0 "U?" H 2200 4550 50  0000 C CNN
 F 1 "74HC273" H 2200 3450 50  0000 C CNN
 F 2 "Package_DIP:DIP-20_W7.62mm" H 2200 4100 50  0001 C CNN
@@
 Connection ~ 3750 4350
 $Comp
-L power:GND #PWR015
+L power:GND #PWR?
 U 1 1 630CEE03
 P 3750 4600
-F 0 "#PWR015" H 3750 4350 50  0001 C CNN
+F 0 "#PWR?" H 3750 4350 50  0001 C CNN
 F 1 "GND" H 3755 4427 50  0000 C CNN
 F 2 "" H 3750 4600 50  0001 C CNN
@@
 $EndComp
 $Comp
-L 74IEC:74HC00 U7
+L 74IEC:74HC00 U?
 U 2 1 630EDD14
 P 2200 5650
-F 0 "U7" H 2200 5800 50  0000 C CNN
+F 0 "U?" H 2200 5800 50  0000 C CNN
 F 1 "74HC00" H 2200 5500 50  0000 C CNN
 F 2 "Package_DIP:DIP-14_W7.62mm" H 2200 5400 50  0001 C CNN
@@
 	1600 4450 1900 4450
 $Comp
-L Device:C CM1
+L Device:C CM?
 U 1 1 6317FAB4
 P 1700 4750
-F 0 "CM1" H 1815 4796 50  0000 L CNN
+F 0 "CM?" H 1815 4796 50  0000 L CNN
 F 1 "1nF" H 1815 4705 50  0000 L CNN
 F 2 "Capacitor_SMD:C_0805_2012Metric_Pad1.18x1.45mm_HandSolder" H 1738 4600 50  0001 C CNN
@@
 	3300 4050 4200 4050
 $Comp
-L 74IEC:74HC257 U13
+L 74IEC:74HC257 U?
 U 1 1 630C909E
 P 4550 4000
-F 0 "U13" H 4550 4550 50  0000 C CNN
+F 0 "U?" H 4550 4550 50  0000 C CNN
 F 1 "74HC257" H 4550 3450 50  0000 C CNN
 F 2 "Package_DIP:DIP-16_W7.62mm" H 5100 4050 50  0001 C CNN
@@
 $EndComp
 $Comp
-L power:VCC #PWR014
+L power:VCC #PWR?
 U 1 1 631CE012
 P 3850 3100
-F 0 "#PWR014" H 3850 2950 50  0001 C CNN
+F 0 "#PWR?" H 3850 2950 50  0001 C CNN
 F 1 "VCC" H 3865 3273 50  0000 C CNN
 F 2 "" H 3850 3100 50  0001 C CNN
@@
 	4000 4450 4000 5650
 $Comp
-L power:GND #PWR016
+L power:GND #PWR?
 U 1 1 631FC597
 P 1700 5000
-F 0 "#PWR016" H 1700 4750 50  0001 C CNN
+F 0 "#PWR?" H 1700 4750 50  0001 C CNN
 F 1 "GND" H 1705 4827 50  0000 C CNN
 F 2 "" H 1700 5000 50  0001 C CNN
@@
 	1800 1550 1900 1550
 $Comp
-L power:VCC #PWR013
+L power:VCC #PWR?
 U 1 1 64D856C7
 P 1800 1450
-F 0 "#PWR013" H 1800 1300 50  0001 C CNN
+F 0 "#PWR?" H 1800 1300 50  0001 C CNN
 F 1 "VCC" H 1815 1623 50  0000 C CNN
 F 2 "" H 1800 1450 50  0001 C CNN
@@
 	3200 3950 3200 6200
 $Comp
-L 74IEC:74HC74 U11
+L 74IEC:74HC74 U?
 U 1 1 647AC379
 P 2200 1700
-F 0 "U11" H 2200 1950 50  0000 C CNN
+F 0 "U?" H 2200 1950 50  0000 C CNN
 F 1 "74HC74" H 2200 1450 50  0000 C CNN
 F 2 "Package_DIP:DIP-14_W7.62mm" H 2200 1950 50  0001 C CNN
@@
 $EndComp
 $Comp
-L 74IEC:74HC74 U11
+L 74IEC:74HC74 U?
 U 2 1 647AEFC0
 P 2200 2700
-F 0 "U11" H 2200 2950 50  0000 C CNN
+F 0 "U?" H 2200 2950 50  0000 C CNN
 F 1 "74HC74" H 2200 2450 50  0000 C CNN
 F 2 "Package_DIP:DIP-14_W7.62mm" H 2200 2950 50  0001 C CNN

Commit message: set annotate
Parts:
- gave numbers to parts that had none: 5
Changed lines of the file:
@@
 $EndDescr
 $Comp
-L 74IEC:74HC273 U?
+L 74IEC:74HC273 U12
 U 1 1 630C4800
 P 2200 4000
-F 0 "U?" H 2200 4550 50  0000 C CNN
+F 0 "U12" H 2200 4550 50  0000 C CNN
 F 1 "74HC273" H 2200 3450 50  0000 C CNN
 F 2 "Package_DIP:DIP-20_W7.62mm" H 2200 4100 50  0001 C CNN
@@
 Connection ~ 3750 4350
 $Comp
-L power:GND #PWR?
+L power:GND #PWR015
 U 1 1 630CEE03
 P 3750 4600
-F 0 "#PWR?" H 3750 4350 50  0001 C CNN
+F 0 "#PWR015" H 3750 4350 50  0001 C CNN
 F 1 "GND" H 3755 4427 50  0000 C CNN
 F 2 "" H 3750 4600 50  0001 C CNN
@@
 $EndComp
 $Comp
-L 74IEC:74HC00 U?
+L 74IEC:74HC00 U7
 U 2 1 630EDD14
 P 2200 5650
-F 0 "U?" H 2200 5800 50  0000 C CNN
+F 0 "U7" H 2200 5800 50  0000 C CNN
 F 1 "74HC00" H 2200 5500 50  0000 C CNN
 F 2 "Package_DIP:DIP-14_W7.62mm" H 2200 5400 50  0001 C CNN
@@
 	1600 4450 1900 4450
 $Comp
-L Device:C CM?
+L Device:C CM1
 U 1 1 6317FAB4
 P 1700 4750
-F 0 "CM?" H 1815 4796 50  0000 L CNN
+F 0 "CM1" H 1815 4796 50  0000 L CNN
 F 1 "1nF" H 1815 4705 50  0000 L CNN
 F 2 "Capacitor_SMD:C_0805_2012Metric_Pad1.18x1.45mm_HandSolder" H 1738 4600 50  0001 C CNN
@@
 	3300 4050 4200 4050
 $Comp
-L 74IEC:74HC257 U?
+L 74IEC:74HC257 U13
 U 1 1 630C909E
 P 4550 4000
-F 0 "U?" H 4550 4550 50  0000 C CNN
+F 0 "U13" H 4550 4550 50  0000 C CNN
 F 1 "74HC257" H 4550 3450 50  0000 C CNN
 F 2 "Package_DIP:DIP-16_W7.62mm" H 5100 4050 50  0001 C CNN
@@
 $EndComp
 $Comp
-L power:VCC #PWR?
+L power:VCC #PWR014
 U 1 1 631CE012
 P 3850 3100
-F 0 "#PWR?" H 3850 2950 50  0001 C CNN
+F 0 "#PWR014" H 3850 2950 50  0001 C CNN
 F 1 "VCC" H 3865 3273 50  0000 C CNN
 F 2 "" H 3850 3100 50  0001 C CNN
@@
 	4000 4450 4000 5650
 $Comp
-L power:GND #PWR?
+L power:GND #PWR016
 U 1 1 631FC597
 P 1700 5000
-F 0 "#PWR?" H 1700 4750 50  0001 C CNN
+F 0 "#PWR016" H 1700 4750 50  0001 C CNN
 F 1 "GND" H 1705 4827 50  0000 C CNN
 F 2 "" H 1700 5000 50  0001 C CNN
@@
 	1800 1550 1900 1550
 $Comp
-L power:VCC #PWR?
+L power:VCC #PWR013
 U 1 1 64D856C7
 P 1800 1450
-F 0 "#PWR?" H 1800 1300 50  0001 C CNN
+F 0 "#PWR013" H 1800 1300 50  0001 C CNN
 F 1 "VCC" H 1815 1623 50  0000 C CNN
 F 2 "" H 1800 1450 50  0001 C CNN
@@
 	3200 3950 3200 6200
 $Comp
-L 74IEC:74HC74 U?
+L 74IEC:74HC74 U11
 U 1 1 647AC379
 P 2200 1700
-F 0 "U?" H 2200 1950 50  0000 C CNN
+F 0 "U11" H 2200 1950 50  0000 C CNN
 F 1 "74HC74" H 2200 1450 50  0000 C CNN
 F 2 "Package_DIP:DIP-14_W7.62mm" H 2200 1950 50  0001 C CNN
@@
 $EndComp
 $Comp
-L 74IEC:74HC74 U?
+L 74IEC:74HC74 U11
 U 2 1 647AEFC0
 P 2200 2700
-F 0 "U?" H 2200 2950 50  0000 C CNN
+F 0 "U11" H 2200 2950 50  0000 C CNN
 F 1 "74HC74" H 2200 2450 50  0000 C CNN
 F 2 "Package_DIP:DIP-14_W7.62mm" H 2200 2950 50  0001 C CNN
