File: ZX-Spectrum-Pentagon/VideoEncoder.sch (KiCad schematic (older format))
At the start: 53 parts

Commit message: add footprints. prepare pcb for edge connector
Parts:
- CVE? (x6): footprint (none) -> Capacitor_SMD:C_0805_2012Metric_Pad1.18x1.45mm_HandSolder
- CVE? (x5): footprint (none) -> Capacitor_Tantalum_SMD:CP_EIA-3528-21_Kemet-B_Pad1.50x2.35mm_HandSolder
- CVE?: value 5pf -> 5pF
- DVE?: footprint (none) -> Diode_SMD:D_SOD-323_HandSoldering
- J?: footprint local footprint:CUI_MD-80SGK -> ZX-Spectrum-Pentagon:CUI_MD-80SGK
- JVE?: footprint (none) -> ZX-Spectrum-Pentagon:CUI_RCJ-013
- LVE?: footprint (none) -> Inductor_SMD:L_7.3x7.3_H4.5
- QVF? (x4): value BC548 -> BC848; footprint (none) -> Package_TO_SOT_SMD:SOT-23_Handsoldering
- U?: footprint (none) -> Package_SO:SOIC-16W_5.3x10.2mm_P1.27mm
- YVE?: value 3.579545 OR 14.318180 -> 3.579545MHz OR 14.318180MHz; footprint (none) -> Crystal:Crystal_HC49-U_Vertical
- YVE?: value 4.433619 or 17.734480 -> 4.433619MHz or 17.734480MHz; footprint (none) -> Crystal:Crystal_HC49-U_Vertical
Other:
- moved on the sheet: RVE?
Changed lines of the file:
@@
 P 3500 6450
 F 0 "YVE?" V 3350 6300 50  0000 C CNN
-F 1 "3.579545 OR 14.318180" V 3650 5950 50  0000 C CNN
-F 2 "" H 3500 6450 50  0001 C CNN
+F 1 "3.579545MHz OR 14.318180MHz" V 3650 5800 50  0000 C CNN
+F 2 "Crystal:Crystal_HC49-U_Vertical" H 3500 6450 50  0001 C CNN
 F 3 "~" H 3500 6450 50  0001 C CNN
 	1    3500 6450
@@
 F 0 "CVE?" V 6600 5300 50  0000 C CNN
 F 1 "0.1uF" V 6800 5350 50  0000 C CNN
-F 2 "" H 6738 5000 50  0001 C CNN
+F 2 "Capacitor_SMD:C_0805_2012Metric_Pad1.18x1.45mm_HandSolder" H 6738 5000 50  0001 C CNN
 F 3 "~" H 6700 5150 50  0001 C CNN
 	1    6700 5150
@@
 F 0 "CVE?" V 6550 4700 50  0000 C CNN
 F 1 "220uF/6.3v" V 6800 4550 50  0000 C CNN
-F 2 "" H 6738 4700 50  0001 C CNN
+F 2 "Capacitor_Tantalum_SMD:CP_EIA-3528-21_Kemet-B_Pad1.50x2.35mm_HandSolder" H 6738 4700 50  0001 C CNN
 F 3 "~" H 6700 4850 50  0001 C CNN
 	1    6700 4850
@@
 F 0 "JVE?" H 8250 4900 50  0000 L CNN
 F 1 "Conn_Coaxial" H 8250 4884 50  0001 L CNN
-F 2 "" H 8150 5000 50  0001 C CNN
+F 2 "ZX-Spectrum-Pentagon:CUI_RCJ-013" H 8150 5000 50  0001 C CNN
 F 3 " ~" H 8150 5000 50  0001 C CNN
 	1    8150 5000
@@
 F 0 "LVE?" V 5050 2300 50  0000 C CNN
 F 1 "100uH" V 5050 2050 50  0000 C CNN
-F 2 "" H 4950 2150 50  0001 C CNN
+F 2 "Inductor_SMD:L_7.3x7.3_H4.5" H 4950 2150 50  0001 C CNN
 F 3 "~" H 4950 2150 50  0001 C CNN
 	1    4950 2150
@@
 F 0 "CVE?" H 5350 2850 50  0000 C CNN
 F 1 "0.1uF" H 5350 2650 50  0000 C CNN
-F 2 "" H 5238 2600 50  0001 C CNN
+F 2 "Capacitor_SMD:C_0805_2012Metric_Pad1.18x1.45mm_HandSolder" H 5238 2600 50  0001 C CNN
 F 3 "~" H 5200 2750 50  0001 C CNN
 	1    5200 2750
@@
 F 0 "CVE?" H 5850 2850 50  0000 C CNN
 F 1 "47uF/6.3v" H 5950 2650 50  0000 C CNN
-F 2 "" H 5738 2600 50  0001 C CNN
+F 2 "Capacitor_Tantalum_SMD:CP_EIA-3528-21_Kemet-B_Pad1.50x2.35mm_HandSolder" H 5738 2600 50  0001 C CNN
 F 3 "~" H 5700 2750 50  0001 C CNN
 	1    5700 2750
@@
 F 0 "CVE?" V 4000 5750 50  0000 C CNN
 F 1 "0.1uF" V 4000 5450 50  0000 C CNN
-F 2 "" H 3888 5450 50  0001 C CNN
+F 2 "Capacitor_SMD:C_0805_2012Metric_Pad1.18x1.45mm_HandSolder" H 3888 5450 50  0001 C CNN
 F 3 "~" H 3850 5600 50  0001 C CNN
 	1    3850 5600
@@
 F 0 "CVE?" V 4000 5450 50  0000 C CNN
 F 1 "0.1uF" V 4000 5150 50  0000 C CNN
-F 2 "" H 3888 5150 50  0001 C CNN
+F 2 "Capacitor_SMD:C_0805_2012Metric_Pad1.18x1.45mm_HandSolder" H 3888 5150 50  0001 C CNN
 F 3 "~" H 3850 5300 50  0001 C CNN
 	1    3850 5300
@@
 F 0 "CVE?" V 4000 4850 50  0000 C CNN
 F 1 "0.1uF" V 4000 4550 50  0000 C CNN
-F 2 "" H 3888 4550 50  0001 C CNN
+F 2 "Capacitor_SMD:C_0805_2012Metric_Pad1.18x1.45mm_HandSolder" H 3888 4550 50  0001 C CNN
 F 3 "~" H 3850 4700 50  0001 C CNN
 	1    3850 4700
@@
 F 0 "U?" H 5400 5600 50  0000 C CNN
 F 1 "AD724" H 5400 4600 50  0000 C CNN
-F 2 "" H 5400 5800 50  0001 C CNN
+F 2 "Package_SO:SOIC-16W_5.3x10.2mm_P1.27mm" H 5400 5800 50  0001 C CNN
 F 3 "" H 5400 5800 50  0001 C CNN
 	1    5400 5100
@@
 F 0 "J?" H 5300 1650 50  0000 C CNN
 F 1 "Mini-DIN-8" H 5500 950 50  0001 C CNN
-F 2 "local footprint:CUI_MD-80SGK" V 5490 1340 50  0001 C CNN
+F 2 "ZX-Spectrum-Pentagon:CUI_MD-80SGK" V 5490 1340 50  0001 C CNN
 F 3 "http://service.powerdynamics.com/ec/Catalog17/Section%2011.pdf" V 5490 1340 50  0001 C CNN
 	1    5500 1350
@@
 $Comp
 L zx_custom_symbol:NPN QVF?
-U 1 1 62DD06E8
+U 2 1 62DD06E8
 P 2700 3250
 AR Path="/62FD43AB/62DD06E8" Ref="QVF?"  Part="1"
-AR Path="/62BF0F7B/62DD06E8" Ref="QVF?"  Part="1"
+AR Path="/62BF0F7B/62DD06E8" Ref="QVF?"  Part="2"
 F 0 "QVF?" H 2888 3296 50  0000 L CNN
-F 1 "BC548" H 2888 3205 50  0000 L CNN
-F 2 "" H 2750 3260 50  0001 C CNN
+F 1 "BC848" H 2888 3205 50  0000 L CNN
+F 2 "Package_TO_SOT_SMD:SOT-23_Handsoldering" H 2750 3260 50  0001 C CNN
 F 3 "" H 2750 3260 50  0001 C CNN
-	1    2700 3250
+	2    2700 3250
 	1    0    0    -1
 $EndComp
 $Comp
 L zx_custom_symbol:NPN QVF?
-U 1 1 62DD06E2
+U 2 1 62DD06E2
 P 3200 3750
 AR Path="/62FD43AB/62DD06E2" Ref="QVF?"  Part="1"
-AR Path="/62BF0F7B/62DD06E2" Ref="QVF?"  Part="1"
+AR Path="/62BF0F7B/62DD06E2" Ref="QVF?"  Part="2"
 F 0 "QVF?" H 3388 3796 50  0000 L CNN
-F 1 "BC548" H 3388 3705 50  0000 L CNN
-F 2 "" H 3250 3760 50  0001 C CNN
+F 1 "BC848" H 3388 3705 50  0000 L CNN
+F 2 "Package_TO_SOT_SMD:SOT-23_Handsoldering" H 3250 3760 50  0001 C CNN
 F 3 "" H 3250 3760 50  0001 C CNN
-	1    3200 3750
+	2    3200 3750
 	1    0    0    -1
 $EndComp
 $Comp
 L zx_custom_symbol:NPN QVF?
-U 1 1 62DD06DC
+U 2 1 62DD06DC
 P 2200 2750
 AR Path="/62FD43AB/62DD06DC" Ref="QVF?"  Part="1"
-AR Path="/62BF0F7B/62DD06DC" Ref="QVF?"  Part="1"
+AR Path="/62BF0F7B/62DD06DC" Ref="QVF?"  Part="2"
 F 0 "QVF?" H 2388 2796 50  0000 L CNN
-F 1 "BC548" H 2388 2705 50  0000 L CNN
-F 2 "" H 2250 2760 50  0001 C CNN
+F 1 "BC848" H 2388 2705 50  0000 L CNN
+F 2 "Package_TO_SOT_SMD:SOT-23_Handsoldering" H 2250 2760 50  0001 C CNN
 F 3 "" H 2250 2760 50  0001 C CNN
-	1    2200 2750
+	2    2200 2750
 	1    0    0    -1
 $EndComp
 $Comp
 L zx_custom_symbol:NPN QVF?
-U 1 1 62DD06D6
+U 2 1 62DD06D6
 P 2200 2050
 AR Path="/62FD43AB/62DD06D6" Ref="QVF?"  Part="1"
-AR Path="/62BF0F7B/62DD06D6" Ref="QVF?"  Part="1"
-F 0 "QVF?" H 2388 2096 50  0000 L CNN
-F 1 "BC548" H 2388 2005 50  0000 L CNN
-F 2 "" H 2250 2060 50  0001 C CNN
+AR Path="/62BF0F7B/62DD06D6" Ref="QVF?"  Part="2"
+F 0 "QVF?" H 2400 2050 50  0000 L CNN
+F 1 "BC848" H 2400 2150 50  0000 L CNN
+F 2 "Package_TO_SOT_SMD:SOT-23_Handsoldering" H 2250 2060 50  0001 C CNN
 F 3 "" H 2250 2060 50  0001 C CNN
-	1    2200 2050
+	2    2200 2050
 	1    0    0    1
 $EndComp
@@
 P 4500 6450
 F 0 "YVE?" V 4350 6600 50  0000 C CNN
-F 1 "4.433619 or 17.734480" V 4650 6950 50  0000 C CNN
-F 2 "" H 4500 6450 50  0001 C CNN
+F 1 "4.433619MHz or 17.734480MHz" V 4650 7100 50  0000 C CNN
+F 2 "Crystal:Crystal_HC49-U_Vertical" H 4500 6450 50  0001 C CNN
 F 3 "~" H 4500 6450 50  0001 C CNN
 	1    4500 6450
@@
 F 0 "DVE?" V 3650 7100 50  0000 C CNN
 F 1 "1N4148" V 3400 7300 50  0000 R CNN
-F 2 "" H 3500 6950 50  0001 C CNN
+F 2 "Diode_SMD:D_SOD-323_HandSoldering" H 3500 6950 50  0001 C CNN
 F 3 "~" H 3500 6950 50  0001 C CNN
 	1    3500 6950
@@
 P 4000 6450
 F 0 "CVE?" H 3850 6550 50  0000 C CNN
-F 1 "5pf" H 4150 6550 50  0000 C CNN
+F 1 "5pF" H 4150 6550 50  0000 C CNN
 F 2 "Capacitor_SMD:C_0805_2012Metric_Pad1.18x1.45mm_HandSolder" H 4038 6300 50  0001 C CNN
 F 3 "~" H 4000 6450 50  0001 C CNN
@@
 	4700 5400 4700 6100
 Wire Wire Line
-	2500 6100 2500 6800
+	2150 6100 2150 6800
 Wire Wire Line
 	4800 6200 4800 5500
@@
 L power:VCC #PWR?
 U 1 1 63AD0237
-P 2350 6300
+P 2000 6300
 AR Path="/62FD43AB/63AD0237" Ref="#PWR?"  Part="1"
 AR Path="/62BF0F7B/63AD0237" Ref="#PWR?"  Part="1"
-F 0 "#PWR?" H 2350 6150 50  0001 C CNN
-F 1 "VCC" H 2365 6473 50  0000 C CNN
-F 2 "" H 2350 6300 50  0001 C CNN
-F 3 "" H 2350 6300 50  0001 C CNN
-	1    2350 6300
+F 0 "#PWR?" H 2000 6150 50  0001 C CNN
+F 1 "VCC" H 2015 6473 50  0000 C CNN
+F 2 "" H 2000 6300 50  0001 C CNN
+F 3 "" H 2000 6300 50  0001 C CNN
+	1    2000 6300
 	1    0    0    -1
 $EndComp
@@
 L Device:R RVE?
 U 1 1 63AEB9D7
-P 2350 6550
+P 2000 6550
 AR Path="/62FD43AB/63AEB9D7" Ref="RVE?"  Part="1"
 AR Path="/62BF0F7B/63AEB9D7" Ref="RVE?"  Part="1"
-F 0 "RVE?" H 2200 6700 50  0000 C CNN
-F 1 "10kOm" H 2200 6400 50  0000 C CNN
-F 2 "Resistor_SMD:R_0805_2012Metric_Pad1.20x1.40mm_HandSolder" V 2280 6550 50  0001 C CNN
-F 3 "~" H 2350 6550 50  0001 C CNN
-	1    2350 6550
-	1    0    0    -1
-$EndComp
-Wire Wire Line
-	2350 6300 2350 6400
-Wire Wire Line
-	2350 6700 2350 6800
-Wire Wire Line
-	2350 6800 2500 6800
-Connection ~ 2500 6800
-Wire Wire Line
-	2500 7300 3900 7300
-Wire Wire Line
-	2500 6800 2500 7300
+F 0 "RVE?" H 1850 6700 50  0000 C CNN
+F 1 "10kOm" H 1850 6400 50  0000 C CNN
+F 2 "Resistor_SMD:R_0805_2012Metric_Pad1.20x1.40mm_HandSolder" V 1930 6550 50  0001 C CNN
+F 3 "~" H 2000 6550 50  0001 C CNN
+	1    2000 6550
+	1    0    0    -1
+$EndComp
+Wire Wire Line
+	2000 6300 2000 6400
+Wire Wire Line
+	2000 6700 2000 6800
+Wire Wire Line
+	2000 6800 2150 6800
+Connection ~ 2150 6800
+Wire Wire Line
+	2150 7300 3900 7300
+Wire Wire Line
+	2150 6800 2150 7300
 Connection ~ 3900 7300
 Wire Wire Line
 	3900 7300 3900 7400
 Wire Wire Line
-	4700 6100 2500 6100
+	4700 6100 2150 6100
 Wire Wire Line
 	5100 2150 5450 2150
@@
 F 0 "CVE?" H 7150 2800 50  0000 C CNN
 F 1 "220uF/6.3v" H 7250 2600 50  0000 C CNN
-F 2 "" H 7038 2550 50  0001 C CNN
+F 2 "Capacitor_Tantalum_SMD:CP_EIA-3528-21_Kemet-B_Pad1.50x2.35mm_HandSolder" H 7038 2550 50  0001 C CNN
 F 3 "~" H 7000 2700 50  0001 C CNN
 	1    7000 2700
@@
 F 0 "CVE?" H 7650 2800 50  0000 C CNN
 F 1 "220uF/6.3v" H 7750 2600 50  0000 C CNN
-F 2 "" H 7538 2550 50  0001 C CNN
+F 2 "Capacitor_Tantalum_SMD:CP_EIA-3528-21_Kemet-B_Pad1.50x2.35mm_HandSolder" H 7538 2550 50  0001 C CNN
 F 3 "~" H 7500 2700 50  0001 C CNN
 	1    7500 2700
@@
 F 0 "CVE?" H 5350 3850 50  0000 C CNN
 F 1 "0.1uF" H 5350 3650 50  0000 C CNN
-F 2 "" H 5238 3600 50  0001 C CNN
+F 2 "Capacitor_SMD:C_0805_2012Metric_Pad1.18x1.45mm_HandSolder" H 5238 3600 50  0001 C CNN
 F 3 "~" H 5200 3750 50  0001 C CNN
 	1    5200 3750
@@
 F 0 "CVE?" H 5850 3850 50  0000 C CNN
 F 1 "47uF/6.3v" H 5950 3650 50  0000 C CNN
-F 2 "" H 5738 3600 50  0001 C CNN
+F 2 "Capacitor_Tantalum_SMD:CP_EIA-3528-21_Kemet-B_Pad1.50x2.35mm_HandSolder" H 5738 3600 50  0001 C CNN
 F 3 "~" H 5700 3750 50  0001 C CNN
 	1    5700 3750

Commit message: change 74HC157 to 74HC257
Changed lines of the file:
@@
 	5900 5200 6300 5200
 Wire Wire Line
-	4050 1200 4000 1200
-Connection ~ 4050 1200
+	4100 1200 4000 1200
+Connection ~ 4100 1200
 Wire Wire Line
-	4050 1100 4000 1100
-Connection ~ 4050 1100
+	4100 1100 4000 1100
+Connection ~ 4100 1100
 Wire Wire Line
-	4050 1100 4050 1200
+	4100 1100 4100 1200
 Text Label 4400 1200 2    50   ~ 0
 LUMA
@@
 SYNC
 Wire Wire Line
-	4400 1200 4050 1200
+	4400 1200 4100 1200
 Wire Wire Line
-	4400 1100 4050 1100
+	4400 1100 4100 1100
 Wire Wire Line
 	4400 1000 4000 1000

Commit message: add companent list
Parts:
- YVE?: value 4.433619MHz or 17.734480MHz -> 4.433618MHz or 17.734480MHz
Changed lines of the file:
@@
 P 4500 6450
 F 0 "YVE?" V 4350 6600 50  0000 C CNN
-F 1 "4.433619MHz or 17.734480MHz" V 4650 7100 50  0000 C CNN
+F 1 "4.433618MHz or 17.734480MHz" V 4650 7100 50  0000 C CNN
 F 2 "Crystal:Crystal_HC49-U_Vertical" H 4500 6450 50  0001 C CNN
 F 3 "~" H 4500 6450 50  0001 C CNN

Commit message: fix video connector
Parts:
- JVE?: value Conn_Coaxial -> Video; symbol Connector:Conn_Coaxial -> zx_custom_symbol:Conn_Coaxial
Changed lines of the file:
@@
-$EndComp
-$Comp
-L Connector:Conn_Coaxial JVE?
-U 1 1 62EC1959
-P 8150 5000
-F 0 "JVE?" H 8250 4900 50  0000 L CNN
-F 1 "Conn_Coaxial" H 8250 4884 50  0001 L CNN
-F 2 "ZX-Spectrum-Pentagon:CUI_RCJ-013" H 8150 5000 50  0001 C CNN
-F 3 " ~" H 8150 5000 50  0001 C CNN
-	1    8150 5000
-	1    0    0    -1
 $EndComp
 $Comp
@@
 	5200 4000 5700 4000
 Wire Bus Line
-	1500 800  1500 1300
-Wire Bus Line
 	6500 800  6500 1950
 Wire Bus Line
 	4500 800  4500 4100
+Wire Bus Line
+	1500 800  1500 1300
+$Comp
+L zx_custom_symbol:Conn_Coaxial JVE?
+U 1 1 62EC1959
+P 8150 5000
+F 0 "JVE?" H 8150 5150 50  0000 C CNN
+F 1 "Video" H 8250 4884 50  0000 L CNN
+F 2 "ZX-Spectrum-Pentagon:CUI_RCJ-013" H 8150 5000 50  0001 C CNN
+F 3 " ~" H 8150 5000 50  0001 C CNN
+	1    8150 5000
+	1    0    0    -1
+$EndComp
 $EndSCHEMATC

Commit message: fix video standart switch
Connections:
- wire segments 212 -> 213
Changed lines of the file:
@@
 P 4000 7600
 F 0 "JVE?" V 4250 7450 50  0000 R CNN
-F 1 "PAL/NTSC" V 4100 7450 50  0000 R CNN
+F 1 "PAL/NTSC" V 4150 8000 50  0000 C CNN
 F 2 "Connector_PinSocket_2.54mm:PinSocket_1x03_P2.54mm_Vertical" H 4000 7600 50  0001 C CNN
 F 3 "~" H 4000 7600 50  0001 C CNN
@@
 Wire Wire Line
 	5200 4000 5700 4000
-Wire Bus Line
-	6500 800  6500 1950
-Wire Bus Line
-	4500 800  4500 4100
-Wire Bus Line
-	1500 800  1500 1300
 $Comp
 L zx_custom_symbol:Conn_Coaxial JVE?
@@
 	1    0    0    -1
 $EndComp
+$Comp
+L power:GND #PWR?
+U 1 1 62B90E90
+P 4500 7300
+F 0 "#PWR?" H 4500 7050 50  0001 C CNN
+F 1 "GND" H 4505 7127 50  0000 C CNN
+F 2 "" H 4500 7300 50  0001 C CNN
+F 3 "" H 4500 7300 50  0001 C CNN
+	1    4500 7300
+	1    0    0    -1
+$EndComp
+Wire Wire Line
+	4500 7200 4500 7300
+Connection ~ 4500 7200
+Wire Bus Line
+	1500 800  1500 1300
+Wire Bus Line
+	6500 800  6500 1950
+Wire Bus Line
+	4500 800  4500 4100
 $EndSCHEMATC

Commit message: update connectors for VideoEncoder.sch
Parts:
- removed J?: Mini-DIN-8, ZX-Spectrum-Pentagon:CUI_MD-80SGK, symbol Connector:Mini-DIN-8
- added JVE?: SVIDEO, ZX-Spectrum-Pentagon:CUI_MD-80SGK, symbol zx_custom_symbol:Mini-DIN-8
Connections:
- wire segments 213 -> 224
Changed lines of the file:
@@
 AudioIntR
 Connection ~ 2300 2450
-Text Label 6400 1250 2    50   ~ 0
+Text Label 6400 950  2    50   ~ 0
 RED
-Text Label 6400 950  2    50   ~ 0
+Text Label 6400 1850 2    50   ~ 0
 GREEN
 Text Label 4600 1250 0    50   ~ 0
@@
 Entry Wire Line
 	4400 4000 4500 4100
-Text Label 6400 1750 2    50   ~ 0
+Text Label 6400 1250 2    50   ~ 0
 VIDEO
 Wire Wire Line
@@
 	6500 1050 6400 950
 Wire Wire Line
-	5500 1650 5500 1750
-Wire Wire Line
-	6400 1750 5500 1750
+	5500 1650 5500 1850
+Wire Wire Line
+	6400 1850 5500 1850
 Entry Wire Line
-	6500 1850 6400 1750
+	6500 1950 6400 1850
 Wire Wire Line
 	6400 1350 5800 1350
@@
 L power:GND #PWR?
 U 1 1 631447CC
-P 5100 1550
-F 0 "#PWR?" H 5100 1300 50  0001 C CNN
-F 1 "GND" H 5105 1377 50  0000 C CNN
-F 2 "" H 5100 1550 50  0001 C CNN
-F 3 "" H 5100 1550 50  0001 C CNN
-	1    5100 1550
-	1    0    0    -1
+P 4850 1700
+F 0 "#PWR?" H 4850 1450 50  0001 C CNN
+F 1 "GND" H 4855 1527 50  0000 C CNN
+F 2 "" H 4850 1700 50  0001 C CNN
+F 3 "" H 4850 1700 50  0001 C CNN
+	1    4850 1700
+	0    1    1    0
 $EndComp
 Text GLabel 1000 5900 0    50   Input ~ 10
@@
 F 3 "" H 1900 5300 50  0001 C CNN
 	1    1900 5300
-	1    0    0    -1
-$EndComp
-$Comp
-L Connector:Mini-DIN-8 J?
-U 1 1 62DD07EE
-P 5500 1350
-AR Path="/62FD43AB/62DD07EE" Ref="J?"  Part="1"
-AR Path="/62BF0F7B/62DD07EE" Ref="J?"  Part="1"
-F 0 "J?" H 5300 1650 50  0000 C CNN
-F 1 "Mini-DIN-8" H 5500 950 50  0001 C CNN
-F 2 "ZX-Spectrum-Pentagon:CUI_MD-80SGK" V 5490 1340 50  0001 C CNN
-F 3 "http://service.powerdynamics.com/ec/Catalog17/Section%2011.pdf" V 5490 1340 50  0001 C CNN
-	1    5500 1350
 	1    0    0    -1
 $EndComp
@@
 $EndComp
 Wire Wire Line
-	5100 1450 5100 1550
-Wire Wire Line
 	4650 4700 4900 4700
 Wire Wire Line
@@
 U 1 1 62EC1959
 P 8150 5000
-F 0 "JVE?" H 8150 5150 50  0000 C CNN
-F 1 "Video" H 8250 4884 50  0000 L CNN
+AR Path="/62EC1959" Ref="JVE?"  Part="1"
+AR Path="/62BF0F7B/62EC1959" Ref="JVE?"  Part="1"
+F 0 "JVE?" H 8000 5100 50  0000 C CNN
+F 1 "Video" H 8250 5100 50  0000 L CNN
 F 2 "ZX-Spectrum-Pentagon:CUI_RCJ-013" H 8150 5000 50  0001 C CNN
 F 3 " ~" H 8150 5000 50  0001 C CNN
@@
 	4500 7200 4500 7300
 Connection ~ 4500 7200
+$Comp
+L zx_custom_symbol:Mini-DIN-8 JVE?
+U 1 1 62BAAD99
+P 5500 1350
+F 0 "JVE?" H 5700 1600 50  0000 C CNN
+F 1 "SVIDEO" H 5250 1600 50  0000 C CNN
+F 2 "ZX-Spectrum-Pentagon:CUI_MD-80SGK" V 5490 1340 50  0001 C CNN
+F 3 "http://service.powerdynamics.com/ec/Catalog17/Section%2011.pdf" V 5490 1340 50  0001 C CNN
+	1    5500 1350
+	1    0    0    -1
+$EndComp
+Wire Wire Line
+	5100 1450 5100 1600
+Wire Wire Line
+	4850 1700 5100 1700
+Wire Wire Line
+	5200 1600 5100 1600
+Connection ~ 5100 1600
+Wire Wire Line
+	5100 1600 5100 1700
+Wire Wire Line
+	5200 1700 5100 1700
+Connection ~ 5100 1700
+Connection ~ 5900 1700
+Wire Wire Line
+	5800 1700 5900 1700
+Wire Wire Line
+	5900 1600 5900 1700
+Wire Wire Line
+	5800 1600 5900 1600
+Wire Wire Line
+	6000 1700 5900 1700
+$Comp
+L power:GND #PWR?
+U 1 1 62C0F5F3
+P 6000 1700
+F 0 "#PWR?" H 6000 1450 50  0001 C CNN
+F 1 "GND" H 6005 1527 50  0000 C CNN
+F 2 "" H 6000 1700 50  0001 C CNN
+F 3 "" H 6000 1700 50  0001 C CNN
+	1    6000 1700
+	0    -1   1    0
+$EndComp
+Wire Wire Line
+	8050 5200 8050 5250
+Wire Wire Line
+	8050 5250 8250 5250
+Wire Wire Line
+	8250 5250 8250 5200
 Wire Bus Line
 	1500 800  1500 1300

Commit message: fix ground connection for video
Connections:
- wire segments 224 -> 226
Changed lines of the file:
@@
 L power:GND #PWR?
 U 1 1 62EA775C
-P 8150 5300
-F 0 "#PWR?" H 8150 5050 50  0001 C CNN
-F 1 "GND" H 8155 5127 50  0000 C CNN
-F 2 "" H 8150 5300 50  0001 C CNN
-F 3 "" H 8150 5300 50  0001 C CNN
-	1    8150 5300
+P 8150 5400
+F 0 "#PWR?" H 8150 5150 50  0001 C CNN
+F 1 "GND" H 8155 5227 50  0000 C CNN
+F 2 "" H 8150 5400 50  0001 C CNN
+F 3 "" H 8150 5400 50  0001 C CNN
+	1    8150 5400
 	1    0    0    -1
 $EndComp
@@
 $EndComp
 Wire Wire Line
-	8050 5200 8050 5250
-Wire Wire Line
-	8050 5250 8250 5250
-Wire Wire Line
-	8250 5250 8250 5200
+	8050 5200 8050 5300
+Wire Wire Line
+	8050 5300 8150 5300
+Wire Wire Line
+	8250 5300 8250 5200
 Wire Bus Line
 	1500 800  1500 1300
@@
 Wire Bus Line
 	4500 800  4500 4100
+Connection ~ 8150 5300
+Wire Wire Line
+	8150 5300 8150 5400
+Wire Wire Line
+	8150 5300 8250 5300
 $EndSCHEMATC

Commit message: Fix component value & footprint
Parts:
- CVE? (x6): value 0.1uF -> 100nF
- CVE? (x2): value 47uF/6.3v -> 47uF/16V
- CVE? (x3): value 220uF/6.3v -> 220uF/6V
Changed lines of the file:
@@
 P 6700 5150
 F 0 "CVE?" V 6600 5300 50  0000 C CNN
-F 1 "0.1uF" V 6800 5350 50  0000 C CNN
+F 1 "100nF" V 6800 5350 50  0000 C CNN
 F 2 "Capacitor_SMD:C_0805_2012Metric_Pad1.18x1.45mm_HandSolder" H 6738 5000 50  0001 C CNN
 F 3 "~" H 6700 5150 50  0001 C CNN
@@
 P 6700 4850
 F 0 "CVE?" V 6550 4700 50  0000 C CNN
-F 1 "220uF/6.3v" V 6800 4550 50  0000 C CNN
+F 1 "220uF/6V" V 6800 4550 50  0000 C CNN
 F 2 "Capacitor_Tantalum_SMD:CP_EIA-3528-21_Kemet-B_Pad1.50x2.35mm_HandSolder" H 6738 4700 50  0001 C CNN
 F 3 "~" H 6700 4850 50  0001 C CNN
@@
 P 5200 2750
 F 0 "CVE?" H 5350 2850 50  0000 C CNN
-F 1 "0.1uF" H 5350 2650 50  0000 C CNN
+F 1 "100nF" H 5350 2650 50  0000 C CNN
 F 2 "Capacitor_SMD:C_0805_2012Metric_Pad1.18x1.45mm_HandSolder" H 5238 2600 50  0001 C CNN
 F 3 "~" H 5200 2750 50  0001 C CNN
@@
 P 5700 2750
 F 0 "CVE?" H 5850 2850 50  0000 C CNN
-F 1 "47uF/6.3v" H 5950 2650 50  0000 C CNN
+F 1 "47uF/16V" H 5950 2650 50  0000 C CNN
 F 2 "Capacitor_Tantalum_SMD:CP_EIA-3528-21_Kemet-B_Pad1.50x2.35mm_HandSolder" H 5738 2600 50  0001 C CNN
 F 3 "~" H 5700 2750 50  0001 C CNN
@@
 P 3850 5600
 F 0 "CVE?" V 4000 5750 50  0000 C CNN
-F 1 "0.1uF" V 4000 5450 50  0000 C CNN
+F 1 "100nF" V 4000 5450 50  0000 C CNN
 F 2 "Capacitor_SMD:C_0805_2012Metric_Pad1.18x1.45mm_HandSolder" H 3888 5450 50  0001 C CNN
 F 3 "~" H 3850 5600 50  0001 C CNN
@@
 P 3850 5300
 F 0 "CVE?" V 4000 5450 50  0000 C CNN
-F 1 "0.1uF" V 4000 5150 50  0000 C CNN
+F 1 "100nF" V 4000 5150 50  0000 C CNN
 F 2 "Capacitor_SMD:C_0805_2012Metric_Pad1.18x1.45mm_HandSolder" H 3888 5150 50  0001 C CNN
 F 3 "~" H 3850 5300 50  0001 C CNN
@@
 P 3850 4700
 F 0 "CVE?" V 4000 4850 50  0000 C CNN
-F 1 "0.1uF" V 4000 4550 50  0000 C CNN
+F 1 "100nF" V 4000 4550 50  0000 C CNN
 F 2 "Capacitor_SMD:C_0805_2012Metric_Pad1.18x1.45mm_HandSolder" H 3888 4550 50  0001 C CNN
 F 3 "~" H 3850 4700 50  0001 C CNN
@@
 P 7000 2700
 F 0 "CVE?" H 7150 2800 50  0000 C CNN
-F 1 "220uF/6.3v" H 7250 2600 50  0000 C CNN
+F 1 "220uF/6V" H 7250 2600 50  0000 C CNN
 F 2 "Capacitor_Tantalum_SMD:CP_EIA-3528-21_Kemet-B_Pad1.50x2.35mm_HandSolder" H 7038 2550 50  0001 C CNN
 F 3 "~" H 7000 2700 50  0001 C CNN
@@
 P 7500 2700
 F 0 "CVE?" H 7650 2800 50  0000 C CNN
-F 1 "220uF/6.3v" H 7750 2600 50  0000 C CNN
+F 1 "220uF/6V" H 7750 2600 50  0000 C CNN
 F 2 "Capacitor_Tantalum_SMD:CP_EIA-3528-21_Kemet-B_Pad1.50x2.35mm_HandSolder" H 7538 2550 50  0001 C CNN
 F 3 "~" H 7500 2700 50  0001 C CNN
@@
 P 5200 3750
 F 0 "CVE?" H 5350 3850 50  0000 C CNN
-F 1 "0.1uF" H 5350 3650 50  0000 C CNN
+F 1 "100nF" H 5350 3650 50  0000 C CNN
 F 2 "Capacitor_SMD:C_0805_2012Metric_Pad1.18x1.45mm_HandSolder" H 5238 3600 50  0001 C CNN
 F 3 "~" H 5200 3750 50  0001 C CNN
@@
 P 5700 3750
 F 0 "CVE?" H 5850 3850 50  0000 C CNN
-F 1 "47uF/6.3v" H 5950 3650 50  0000 C CNN
+F 1 "47uF/16V" H 5950 3650 50  0000 C CNN
 F 2 "Capacitor_Tantalum_SMD:CP_EIA-3528-21_Kemet-B_Pad1.50x2.35mm_HandSolder" H 5738 3600 50  0001 C CNN
 F 3 "~" H 5700 3750 50  0001 C CNN
@@
 Wire Wire Line
 	8250 5300 8250 5200
+Connection ~ 8150 5300
+Wire Wire Line
+	8150 5300 8150 5400
+Wire Wire Line
+	8150 5300 8250 5300
 Wire Bus Line
 	1500 800  1500 1300
@@
 Wire Bus Line
 	4500 800  4500 4100
-Connection ~ 8150 5300
-Wire Wire Line
-	8150 5300 8150 5400
-Wire Wire Line
-	8150 5300 8250 5300
 $EndSCHEMATC
