File: ZX-Spectrum-Pentagon/Generator.sch (KiCad schematic (older format))
At the start: 50 parts

Commit message: clear all pcb
Changed lines of the file:
@@
 $Comp
 L 74IEC:74HC14 U?
-U 2 1 629C03DD
+U 4 1 629C03DD
 P 2900 1100
 F 0 "U?" H 2900 1250 50  0000 C CNN
@@
 F 2 "Package_DIP:DIP-14_W7.62mm" H 2900 1310 50  0001 C CNN
 F 3 "https://www.ti.com/lit/ug/scyd013b/scyd013b.pdf" H 2900 1310 50  0001 C CNN
-	2    2900 1100
+	4    2900 1100
 	1    0    0    -1
 $EndComp
 $Comp
 L 74IEC:74HC14 U?
-U 1 1 629BF100
+U 3 1 629BF100
 P 2400 1100
 F 0 "U?" H 2400 1250 50  0000 C CNN
@@
 F 2 "Package_DIP:DIP-14_W7.62mm" H 2400 1310 50  0001 C CNN
 F 3 "https://www.ti.com/lit/ug/scyd013b/scyd013b.pdf" H 2400 1310 50  0001 C CNN
-	1    2400 1100
+	3    2400 1100
 	1    0    0    -1
 $EndComp
@@
 $Comp
 L 74IEC:74HC14 U?
-U 4 1 6347B914
+U 6 1 6347B914
 P 9650 3700
 AR Path="/6296ED1F/6347B914" Ref="U?"  Part="4"
-AR Path="/6296E6C7/6347B914" Ref="U?"  Part="4"
+AR Path="/6296E6C7/6347B914" Ref="U?"  Part="6"
 F 0 "U?" H 9650 3850 50  0000 C CNN
 F 1 "74HC14" H 9650 3550 50  0000 C CNN
 F 2 "Package_DIP:DIP-14_W7.62mm" H 9650 3910 50  0001 C CNN
 F 3 "https://www.ti.com/lit/ug/scyd013b/scyd013b.pdf" H 9650 3910 50  0001 C CNN
-	4    9650 3700
+	6    9650 3700
 	1    0    0    -1
 $EndComp
 $Comp
 L 74IEC:74HC14 U?
-U 3 1 6347B91A
+U 5 1 6347B91A
 P 9150 3700
 AR Path="/6296ED1F/6347B91A" Ref="U?"  Part="3"
-AR Path="/6296E6C7/6347B91A" Ref="U?"  Part="3"
+AR Path="/6296E6C7/6347B91A" Ref="U?"  Part="5"
 F 0 "U?" H 9150 3850 50  0000 C CNN
 F 1 "74HC14" H 9150 3550 50  0000 C CNN
 F 2 "Package_DIP:DIP-14_W7.62mm" H 9150 3910 50  0001 C CNN
 F 3 "https://www.ti.com/lit/ug/scyd013b/scyd013b.pdf" H 9150 3910 50  0001 C CNN
-	3    9150 3700
+	5    9150 3700
 	1    0    0    -1
 $EndComp

Commit message: add footprints. prepare pcb for edge connector
Parts:
- CG?: value 100p -> 100pF
- CG?: value 1n2 -> 1nF; Spice_Model (none) -> 1n; Spice_Netlist_Enabled (none) -> Y; Spice_Primitive (none) -> R
- CG?: value 22n -> 22nF
- CG?: value 510p -> 510pF
- QG?: value 2N2369A -> BC848; footprint (none) -> Package_TO_SOT_SMD:SOT-23_Handsoldering
- U? (x2): footprint (none) -> Package_DIP:DIP-14_W7.62mm
Changed lines of the file:
@@
 P 5950 6000
 F 0 "CG?" V 5800 6000 50  0000 C CNN
-F 1 "22n" V 6100 6000 50  0000 C CNN
+F 1 "22nF" V 6100 6000 50  0000 C CNN
 F 2 "Capacitor_SMD:C_0805_2012Metric_Pad1.18x1.45mm_HandSolder" H 5988 5850 50  0001 C CNN
 F 3 "~" H 5950 6000 50  0001 C CNN
@@
 P 7300 6250
 F 0 "CG?" H 7200 6150 50  0000 C CNN
-F 1 "510p" H 7150 6350 50  0000 C CNN
+F 1 "510pF" H 7150 6350 50  0000 C CNN
 F 2 "Capacitor_SMD:C_0805_2012Metric_Pad1.18x1.45mm_HandSolder" H 7338 6100 50  0001 C CNN
 F 3 "~" H 7300 6250 50  0001 C CNN
@@
 P 5400 5050
 F 0 "CG?" H 5500 5150 50  0000 C CNN
-F 1 "1n2" H 5500 4950 50  0000 C CNN
+F 1 "1nF" H 5500 4950 50  0000 C CNN
 F 2 "Capacitor_SMD:C_0805_2012Metric_Pad1.18x1.45mm_HandSolder" H 5438 4900 50  0001 C CNN
 F 3 "~" H 5400 5050 50  0001 C CNN
+F 4 "R" H 5400 5050 50  0001 C CNN "Spice_Primitive"
+F 5 "1n" H 5400 5050 50  0001 C CNN "Spice_Model"
+F 6 "Y" H 5400 5050 50  0001 C CNN "Spice_Netlist_Enabled"
 	1    5400 5050
 	1    0    0    -1
@@
 $Comp
 L zx_custom_symbol:NPN QG?
-U 1 1 62B83B79
+U 2 1 62B83B79
 P 4950 4500
 F 0 "QG?" H 5138 4546 50  0000 L CNN
-F 1 "2N2369A" H 5138 4455 50  0000 L CNN
-F 2 "" H 5000 4510 50  0001 C CNN
+F 1 "BC848" H 5138 4455 50  0000 L CNN
+F 2 "Package_TO_SOT_SMD:SOT-23_Handsoldering" H 5000 4510 50  0001 C CNN
 F 3 "" H 5000 4510 50  0001 C CNN
-	1    4950 4500
+	2    4950 4500
 	1    0    0    -1
 $EndComp
@@
 F 0 "U?" H 3500 5500 50  0000 C CNN
 F 1 "74HC74" H 3500 5000 50  0000 C CNN
-F 2 "" H 3500 5500 50  0001 C CNN
+F 2 "Package_DIP:DIP-14_W7.62mm" H 3500 5500 50  0001 C CNN
 F 3 "https://www.ti.com/lit/ug/scyd013b/scyd013b.pdf" H 3500 5500 50  0001 C CNN
 	1    3500 5250
@@
 F 0 "U?" H 3500 6100 50  0000 C CNN
 F 1 "74HC74" H 3500 5600 50  0000 C CNN
-F 2 "" H 3500 6100 50  0001 C CNN
+F 2 "Package_DIP:DIP-14_W7.62mm" H 3500 6100 50  0001 C CNN
 F 3 "https://www.ti.com/lit/ug/scyd013b/scyd013b.pdf" H 3500 6100 50  0001 C CNN
 	2    3500 5850
@@
 P 1350 1100
 F 0 "CG?" V 1200 1100 50  0000 C CNN
-F 1 "100p" V 1500 1100 50  0000 C CNN
+F 1 "100pF" V 1500 1100 50  0000 C CNN
 F 2 "Capacitor_SMD:C_0805_2012Metric_Pad1.18x1.45mm_HandSolder" H 1388 950 50  0001 C CNN
 F 3 "~" H 1350 1100 50  0001 C CNN

Commit message: change 74HC157 to 74HC257
Parts:
- removed U?: 74HC157, Package_DIP:DIP-16_W7.62mm, symbol 74IEC:74HC157
- added U?: 74HC257, n, symbol 74IEC:74HC257
Connections:
- wire segments 281 -> 283
Changed lines of the file:
@@
-	1    0    0    -1
-$EndComp
-$Comp
-L 74IEC:74HC157 U?
-U 1 1 63A00742
-P 6950 3700
-F 0 "U?" H 6950 4250 50  0000 C CNN
-F 1 "74HC157" H 6950 3150 50  0000 C CNN
-F 2 "Package_DIP:DIP-16_W7.62mm" H 6950 3850 50  0001 C CNN
-F 3 "https://www.ti.com/lit/ug/scyd013b/scyd013b.pdf" H 6950 3850 50  0001 C CNN
-	1    6950 3700
 	1    0    0    -1
 $EndComp
@@
 	6100 5250 6450 5250
 Wire Wire Line
-	3800 5750 10500 5750
+	3800 5750 8800 5750
 Wire Wire Line
 	7200 6000 7300 6000
@@
 HSYNC
 Wire Wire Line
-	10500 5600 4000 5600
+	10500 5600 8150 5600
 Connection ~ 4000 5600
 Wire Wire Line
@@
 Wire Wire Line
 	2950 6750 5550 6750
+$Comp
+L 74IEC:74HC257 U?
+U 1 1 62B96FF4
+P 6950 3700
+F 0 "U?" H 6950 4250 50  0000 C CNN
+F 1 "74HC257" H 6950 3150 50  0000 C CNN
+F 2 " n" H 7500 3750 50  0001 C CNN
+F 3 "https://www.ti.com/lit/ug/scyd013b/scyd013b.pdf" H 7500 3750 50  0001 C CNN
+	1    6950 3700
+	1    0    0    -1
+$EndComp
+Connection ~ 8150 5600
+Wire Wire Line
+	8150 5600 4000 5600
+Connection ~ 8800 5750
+Wire Wire Line
+	8800 5750 10500 5750
 Wire Bus Line
 	7500 2850 7500 5300

Commit message: rename from 74XX152 to 74HC153
Connections:
- wire segments 283 -> 281
Changed lines of the file:
@@
 	6100 5250 6450 5250
-Wire Wire Line
-	3800 5750 8800 5750
 Wire Wire Line
 	7200 6000 7300 6000
@@
 Text GLabel 10500 5600 2    50   Output ~ 10
 HSYNC
-Wire Wire Line
-	10500 5600 8150 5600
 Connection ~ 4000 5600
 Wire Wire Line
@@
 	1    0    0    -1
 $EndComp
-Connection ~ 8150 5600
-Wire Wire Line
-	8150 5600 4000 5600
-Connection ~ 8800 5750
-Wire Wire Line
-	8800 5750 10500 5750
+Wire Wire Line
+	3800 5750 10500 5750
+Wire Wire Line
+	4000 5600 10500 5600
 Wire Bus Line
 	7500 2850 7500 5300

Commit message: add footprint for 74HC257
Parts:
- U?: footprint n -> Package_DIP:DIP-16_W7.62mm
Changed lines of the file:
@@
 F 0 "U?" H 6950 4250 50  0000 C CNN
 F 1 "74HC257" H 6950 3150 50  0000 C CNN
-F 2 " n" H 7500 3750 50  0001 C CNN
+F 2 "Package_DIP:DIP-16_W7.62mm" H 7500 3750 50  0001 C CNN
 F 3 "https://www.ti.com/lit/ug/scyd013b/scyd013b.pdf" H 7500 3750 50  0001 C CNN
 	1    6950 3700

Commit message: Fix component value & footprint
Parts:
- CG?: value 47uF/6.3V -> 47uF/16V
- CG?: Spice_Model 1n -> (none)
- DG?: value 1N1448 -> 1N4148
Changed lines of the file:
@@
 F 3 "~" H 5400 5050 50  0001 C CNN
 F 4 "R" H 5400 5050 50  0001 C CNN "Spice_Primitive"
-F 5 "1n" H 5400 5050 50  0001 C CNN "Spice_Model"
+F 5 "" H 5400 5050 50  0001 C CNN "Spice_Model"
 F 6 "Y" H 5400 5050 50  0001 C CNN "Spice_Netlist_Enabled"
 	1    5400 5050
@@
 P 6500 6250
 F 0 "DG?" V 6350 6350 50  0000 C CNN
-F 1 "1N1448" V 6600 6400 50  0000 C CNN
+F 1 "1N4148" V 6600 6400 50  0000 C CNN
 F 2 "Diode_SMD:D_SOD-323_HandSoldering" H 6500 6250 50  0001 C CNN
 F 3 "~" H 6500 6250 50  0001 C CNN
@@
 AR Path="/6296E6C7/6347B93C" Ref="CG?"  Part="1"
 F 0 "CG?" H 8400 4100 50  0000 C CNN
-F 1 "47uF/6.3V" H 8300 3850 50  0000 C CNN
+F 1 "47uF/16V" H 8300 3850 50  0000 C CNN
 F 2 "Capacitor_Tantalum_SMD:CP_EIA-3528-21_Kemet-B_Pad1.50x2.35mm_HandSolder" H 8588 3800 50  0001 C CNN
 F 3 "~" H 8550 3950 50  0001 C CNN

Commit message: move from globag label to hierarchical label. fix all warning
Parts:
- gave numbers to parts that had none: 31
Connections:
- net labels added: ZB1, ZB10, ZB11, ZB14, ZB15, ZB16, ZB17, ZB18, ZB2, ZB3, ZB4, ZB5, ZB9
- net labels removed: B1, B10, B11, B14, B15, B16, B17, B18, B2, B3, B4, B5, B9
- wire segments 281 -> 279
Other:
- moved on the sheet: U14F, U16A, U19B, U22B, U23A, U7C

Commit message: Rename screen address signal
Connections:
- net labels added: SA0, SA1, SA10, SA11, SA12, SA2, SA3, SA4, SA5, SA6, SA7, SA8, SA9
- net labels removed: ZB1, ZB10, ZB11, ZB14, ZB15, ZB16, ZB17, ZB18, ZB2, ZB3, ZB4, ZB5, ZB9
Changed lines of the file:
@@
 	2050 3550 2150 3650
 Text Label 2050 3550 2    50   ~ 0
-ZB1
+SA0
 Entry Wire Line
 	2050 3650 2150 3750
 Text Label 2050 3650 2    50   ~ 0
-ZB2
+SA1
 Entry Wire Line
 	2050 4350 2150 4450
@@
 	1750 4550 2050 4550
 Text Label 2050 4350 2    50   ~ 0
-ZB3
+SA2
 Text Label 2050 4450 2    50   ~ 0
-ZB4
+SA3
 Text Label 2050 4550 2    50   ~ 0
-ZB5
+SA4
 Wire Wire Line
 	750  3600 1050 3600
@@
 $EndComp
 Text Label 2250 4750 0    50   ~ 0
-ZB5
+SA4
 Entry Wire Line
 	2150 4850 2250 4750
@@
 	2250 4000 2450 4000
 Text Label 2250 4000 0    50   ~ 0
-ZB3
+SA2
 Wire Wire Line
 	2450 4450 2250 4450
 Text Label 2250 4450 0    50   ~ 0
-ZB4
+SA3
 Entry Wire Line
 	2050 4650 2150 4750
@@
 B12
 Text Label 2050 6050 2    50   ~ 0
-ZB11
+SA7
 Entry Wire Line
 	2050 6250 2150 6350
@@
 	1850 5850 1850 5700
 Text Label 2050 5600 2    50   ~ 0
-ZB9
+SA5
 Text Label 2050 5500 2    50   ~ 0
 B8
@@
 	2250 6300 2550 6300
 Text Label 2250 6300 0    50   ~ 0
-ZB10
+SA6
 Text Label 2250 6400 0    50   ~ 0
-ZB11
+SA7
 Wire Wire Line
 	2450 6700 2550 6700
@@
 	2150 5550 2250 5450
 Text Label 2250 5450 0    50   ~ 0
-ZB1
+SA0
 Wire Wire Line
 	3050 5100 3050 5000
@@
 	6100 3950 6500 3950
 Text HLabel 10500 3100 2    50   Output ~ 10
-ZB1
+SA0
 Text HLabel 10500 3200 2    50   Output ~ 10
-ZB2
+SA1
 Text HLabel 10500 3300 2    50   Output ~ 10
-ZB3
+SA2
 Text HLabel 10500 3400 2    50   Output ~ 10
-ZB4
+SA3
 Text HLabel 10500 3500 2    50   Output ~ 10
-ZB5
+SA4
 Text HLabel 10500 3600 2    50   Output ~ 10
-ZB9
+SA5
 Text HLabel 10500 3700 2    50   Output ~ 10
-ZB10
+SA6
 Text HLabel 10500 3800 2    50   Output ~ 10
-ZB11
+SA7
 Text HLabel 10500 3900 2    50   Output ~ 10
-ZB14
+SA8
 Text HLabel 10500 4000 2    50   Output ~ 10
-ZB15
+SA9
 Text HLabel 10500 4100 2    50   Output ~ 10
-ZB16
+SA10
 Text HLabel 10500 4200 2    50   Output ~ 10
-ZB17
+SA11
 Entry Wire Line
 	7400 3400 7500 3500
@@
 	7150 4000 7400 4000
 Text Label 7400 3400 2    50   ~ 0
-ZB14
+SA8
 Text Label 7400 3600 2    50   ~ 0
-ZB15
+SA9
 Text Label 7400 3800 2    50   ~ 0
-ZB16
+SA10
 Text Label 7400 4000 2    50   ~ 0
-ZB17
+SA11
 Entry Wire Line
 	10150 3000 10250 3100
@@
 	10150 3400 10250 3500
 Text Label 10250 3100 0    50   ~ 0
-ZB1
+SA0
 Text Label 10250 3200 0    50   ~ 0
-ZB2
+SA1
 Text Label 10250 3300 0    50   ~ 0
-ZB3
+SA2
 Text Label 10250 3400 0    50   ~ 0
-ZB4
+SA3
 Text Label 10250 3500 0    50   ~ 0
-ZB5
+SA4
 Text Label 10250 3600 0    50   ~ 0
-ZB9
+SA5
 Text Label 10250 3700 0    50   ~ 0
-ZB10
+SA6
 Text Label 10250 3800 0    50   ~ 0
-ZB11
+SA7
 Text Label 10250 3900 0    50   ~ 0
-ZB14
+SA8
 Text Label 10250 4000 0    50   ~ 0
-ZB15
+SA9
 Text Label 10250 4100 0    50   ~ 0
-ZB16
+SA10
 Text Label 10250 4200 0    50   ~ 0
-ZB17
+SA11
 Wire Wire Line
 	4550 4500 4750 4500
@@
 B13
 Text HLabel 10500 4300 2    50   Output ~ 10
-ZB18
+SA12
 Entry Wire Line
 	10150 4200 10250 4300
@@
 	7150 5200 7400 5200
 Text Label 7400 5200 2    50   ~ 0
-ZB18
+SA12
 Text HLabel 6100 4150 0    50   Input ~ 10
 C30
@@
 Connection ~ 850  5450
 Text Label 10250 4300 0    50   ~ 0
-ZB18
+SA12
 Wire Wire Line
 	6650 5200 6750 5200
@@
 	6250 5150 5750 5150
 Text Label 2050 5700 2    50   ~ 0
-ZB10
+SA6
 Wire Wire Line
 	2250 5150 2450 5150
