File: ZX-Spectrum-Pentagon/PowerSources.sch (KiCad schematic (older format))
At the start: 55 parts

Commit message: add footprints. prepare pcb for edge connector
Parts:
- CNPS?: footprint (none) -> Connector_BarrelJack:BarrelJack_Wuerth_6941xx301002
Changed lines of the file:
@@
 F 0 "CNPS?" H 1350 2100 50  0000 C CNN
 F 1 "Power_Jack" H 1300 1700 50  0000 C CNN
-F 2 "" H 1300 2100 50  0001 C CNN
+F 2 "Connector_BarrelJack:BarrelJack_Wuerth_6941xx301002" H 1300 2100 50  0001 C CNN
 F 3 "" H 1300 2100 50  0001 C CNN
 	1    1300 1900

Commit message: Add diode bridge model and datasheet
Parts:
- removed DPS?: D_Bridge_+-AA, Diode_SMD:Diode_Bridge_Vishay_DFS, symbol Device:D_Bridge_+-AA
- added DPS?: DF005S, Diode_SMD:Diode_Bridge_Vishay_DFS, symbol Device:D_Bridge_+A-A
Changed lines of the file:
@@
-	1    0    0    -1
-$EndComp
-$Comp
-L Device:D_Bridge_+-AA DPS?
-U 1 1 629DB190
-P 2300 1900
-F 0 "DPS?" H 2450 2100 50  0000 L CNN
-F 1 "D_Bridge_+-AA" H 2644 1855 50  0001 L CNN
-F 2 "Diode_SMD:Diode_Bridge_Vishay_DFS" H 2300 1900 50  0001 C CNN
-F 3 "~" H 2300 1900 50  0001 C CNN
-	1    2300 1900
 	1    0    0    -1
 $EndComp
@@
 	9500 900  10500 900
 Connection ~ 9500 1850
+$Comp
+L Device:D_Bridge_+A-A DPS?
+U 1 1 62BAF1DA
+P 2300 1900
+F 0 "DPS?" H 2450 2100 50  0000 L CNN
+F 1 "DF005S" H 2450 1650 50  0000 L CNN
+F 2 "Diode_SMD:Diode_Bridge_Vishay_DFS" H 2300 1900 50  0001 C CNN
+F 3 "https://www.vishay.com/docs/88573/dfs.pdf" H 2300 1900 50  0001 C CNN
+	1    2300 1900
+	1    0    0    -1
+$EndComp
 $EndSCHEMATC

Commit message: modefied bridge
Parts:
- removed DPS?: DF005S, Diode_SMD:Diode_Bridge_Vishay_DFS, symbol Device:D_Bridge_+A-A
- added DPS?: DF005S, Diode_SMD:Diode_Bridge_Vishay_DFS, symbol Device:D_Bridge_+-AA
Changed lines of the file:
@@
 Connection ~ 9500 1850
 $Comp
-L Device:D_Bridge_+A-A DPS?
-U 1 1 62BAF1DA
+L Device:D_Bridge_+-AA DPS?
+U 1 1 62BAF22D
 P 2300 1900
-F 0 "DPS?" H 2450 2100 50  0000 L CNN
-F 1 "DF005S" H 2450 1650 50  0000 L CNN
+F 0 "DPS?" H 2400 2100 50  0000 L CNN
+F 1 "DF005S" H 2500 1700 50  0000 C CNN
 F 2 "Diode_SMD:Diode_Bridge_Vishay_DFS" H 2300 1900 50  0001 C CNN
 F 3 "https://www.vishay.com/docs/88573/dfs.pdf" H 2300 1900 50  0001 C CNN

Commit message: Fix component value & footprint
Parts:
- CPS?: value 330uF/16v -> 330uF/16V
- CPS?: value 330uF/6V -> 330uF/16V
- CPS?: value 4,7uF/6V -> 4.7uF/16V
- CPS?: value 4,7uF/16V -> 4.7uF/16V
- gave numbers to parts that had none: 1
Changed lines of the file:
@@
 P 2900 2150
 F 0 "CPS?" H 3050 2250 50  0000 C CNN
-F 1 "330uF/16v" H 3150 2050 50  0000 C CNN
+F 1 "330uF/16V" H 3150 2050 50  0000 C CNN
 F 2 "Capacitor_Tantalum_SMD:CP_EIA-7343-31_Kemet-D_Pad2.25x2.55mm_HandSolder" H 2938 2000 50  0001 C CNN
 F 3 "~" H 2900 2150 50  0001 C CNN
@@
 P 5500 2150
 F 0 "CPS?" H 5650 2250 50  0000 C CNN
-F 1 "330uF/6V" H 5750 2050 50  0000 C CNN
+F 1 "330uF/16V" H 5750 2050 50  0000 C CNN
 F 2 "Capacitor_Tantalum_SMD:CP_EIA-7343-31_Kemet-D_Pad2.25x2.55mm_HandSolder" H 5538 2000 50  0001 C CNN
 F 3 "~" H 5500 2150 50  0001 C CNN
@@
 P 6500 2150
 F 0 "CPS?" H 6650 2250 50  0000 C CNN
-F 1 "4,7uF/6V" H 6700 2050 50  0000 C CNN
+F 1 "4.7uF/16V" H 6700 2050 50  0000 C CNN
 F 2 "Capacitor_Tantalum_SMD:CP_EIA-3528-21_Kemet-B_Pad1.50x2.35mm_HandSolder" H 6538 2000 50  0001 C CNN
 F 3 "~" H 6500 2150 50  0001 C CNN
@@
 P 9000 2100
 F 0 "CPS?" H 9050 2200 50  0000 L CNN
-F 1 "4,7uF/16V" H 9050 2000 50  0000 L CNN
+F 1 "4.7uF/16V" H 9050 2000 50  0000 L CNN
 F 2 "Capacitor_Tantalum_SMD:CP_EIA-3528-21_Kemet-B_Pad1.50x2.35mm_HandSolder" H 9038 1950 50  0001 C CNN
 F 3 "~" H 9000 2100 50  0001 C CNN
@@
 	6950 1950 6950 2000
 $Comp
-L zx_custom_symbol:Power_Jack CNPS?
+L zx_custom_symbol:Power_Jack JPS?
 U 1 1 62B64645
 P 1300 1900
-F 0 "CNPS?" H 1350 2100 50  0000 C CNN
+F 0 "JPS?" H 1350 2100 50  0000 C CNN
 F 1 "Power_Jack" H 1300 1700 50  0000 C CNN
 F 2 "Connector_BarrelJack:BarrelJack_Wuerth_6941xx301002" H 1300 2100 50  0001 C CNN

Commit message: update comanents
Parts:
- CPF? (x40): footprint Capacitor_SMD:C_1210_3225Metric_Pad1.33x2.70mm_HandSolder -> Capacitor_SMD:C_1206_3216Metric_Pad1.33x1.80mm_HandSolder

Commit message: fix erc
Parts:
- gave numbers to parts that had none: 55

Commit message: clear annotation
Parts:
- renumbered CPF1 to CPF?, CPF2 to CPF?, CPF3 to CPF?, CPF4 to CPF?, CPF5 to CPF?, CPF6 to CPF?, CPF7 to CPF?, CPF8 to CPF?, CPF9 to CPF?, CPF10 to CPF?, CPF11 to CPF?, CPF12 to CPF?, CPF13 to CPF?, CPF14 to CPF?, CPF15 to CPF?, CPF16 to CPF?, CPF17 to CPF?, CPF18 to CPF?, CPF21 to CPF?, CPF22 to CPF?, CPF23 to CPF?, CPF24 to CPF?, CPF25 to CPF?, CPF26 to CPF?, CPF27 to CPF?, CPF28 to CPF?, CPF29 to CPF?, CPF30 to CPF?, CPF31 to CPF?, CPF32 to CPF?, CPF33 to CPF?, CPF34 to CPF?, CPF35 to CPF?, CPF36 to CPF?, CPF37 to CPF?, CPF38 to CPF?, CPF19 to CPF?, CPF20 to CPF?, CPF39 to CPF?, CPF40 to CPF?, CPS3 to CPS?, CPS2 to CPS?, CPS4 to CPS?, CPS5 to CPS?, CPS6 to CPS?, CPS7 to CPS?, CPS8 to CPS?, CPS1 to CPS?, DPS2 to DPS?, DPS1 to DPS?, JPS1 to JPS?, LPS1 to LPS?, RPS1 to RPS?, UPS2 to UPS?, UPS1 to UPS?
