File: ZX-Spectrum-Pentagon/VideoFormating.sch (KiCad schematic (older format))
At the start: 10 parts

Commit message: add footprints. prepare pcb for edge connector
Parts:
- U?: footprint (none) -> Package_DIP:DIP-14_W7.62mm
Changed lines of the file:
@@
 F 0 "U?" H 5400 5550 50  0000 C CNN
 F 1 "74HC86" H 5400 5250 50  0000 C CNN
-F 2 "" H 5400 5100 50  0001 C CNN
+F 2 "Package_DIP:DIP-14_W7.62mm" H 5400 5100 50  0001 C CNN
 F 3 "https://www.ti.com/lit/ug/scyd013b/scyd013b.pdf" H 5400 5600 50  0001 C CNN
 	4    5400 5400

Commit message: set annotate
Parts:
- gave numbers to parts that had none: 10
Changed lines of the file:
@@
 	1400 1700 1500 1600
 $Comp
-L 74IEC:74HC574 U?
+L 74IEC:74HC574 U29
 U 1 1 632C89BD
 P 2200 1500
-F 0 "U?" H 2200 2050 50  0000 C CNN
+F 0 "U29" H 2200 2050 50  0000 C CNN
 F 1 "74HC574" H 2200 950 50  0000 C CNN
 F 2 "Package_DIP:DIP-20_W7.62mm" H 2200 1200 50  0001 C CNN
@@
 $EndComp
 $Comp
-L 74IEC:74HC574 U?
+L 74IEC:74HC574 U30
 U 1 1 632CEC67
 P 3100 1600
-F 0 "U?" H 3100 2150 50  0000 C CNN
+F 0 "U30" H 3100 2150 50  0000 C CNN
 F 1 "74HC574" H 3100 1050 50  0000 C CNN
 F 2 "Package_DIP:DIP-20_W7.62mm" H 3100 1300 50  0001 C CNN
@@
 	2700 2050 2700 2150
 $Comp
-L power:GND #PWR?
+L power:GND #PWR041
 U 1 1 632E6C13
 P 2700 2250
-F 0 "#PWR?" H 2700 2000 50  0001 C CNN
+F 0 "#PWR041" H 2700 2000 50  0001 C CNN
 F 1 "GND" H 2705 2077 50  0000 C CNN
 F 2 "" H 2700 2250 50  0001 C CNN
@@
 C3
 $Comp
-L 74IEC:74HC574 U?
+L 74IEC:74HC574 U34
 U 1 1 6330BD21
 P 2200 6600
-F 0 "U?" H 2200 7150 50  0000 C CNN
+F 0 "U34" H 2200 7150 50  0000 C CNN
 F 1 "74HC574" H 2200 6050 50  0000 C CNN
 F 2 "Package_DIP:DIP-20_W7.62mm" H 2200 6300 50  0001 C CNN
@@
 P 3250 6650
 AR Path="/6332DE4B" Ref="U?"  Part="1"
-AR Path="/62FD43AB/6332DE4B" Ref="U?"  Part="1"
-F 0 "U?" H 3250 7350 50  0000 C CNN
+AR Path="/62FD43AB/6332DE4B" Ref="U35"  Part="1"
+F 0 "U35" H 3250 7350 50  0000 C CNN
 F 1 "74HC166" H 3250 5950 50  0000 C CNN
 F 2 "Package_DIP:DIP-16_W7.62mm" H 3250 6050 50  0001 C CNN
@@
 	2700 7050 2900 7050
 $Comp
-L power:GND #PWR?
+L power:GND #PWR046
 U 1 1 63470A69
 P 1900 7150
-F 0 "#PWR?" H 1900 6900 50  0001 C CNN
+F 0 "#PWR046" H 1900 6900 50  0001 C CNN
 F 1 "GND" H 1905 6977 50  0000 C CNN
 F 2 "" H 1900 7150 50  0001 C CNN
@@
 $EndComp
 $Comp
-L 74IEC:74XX153 U?
+L 74IEC:74XX153 U31
 U 1 1 63481D4A
 P 5350 1700
-F 0 "U?" H 5350 2350 50  0000 C CNN
+F 0 "U31" H 5350 2350 50  0000 C CNN
 F 1 "74XX153" H 5350 1050 50  0000 C CNN
 F 2 "Package_DIP:DIP-16_W7.62mm" H 5350 1750 50  0001 C CNN
@@
 $EndComp
 $Comp
-L 74IEC:74XX153 U?
+L 74IEC:74XX153 U32
 U 1 1 63485DD9
 P 5350 3500
-F 0 "U?" H 5350 4150 50  0000 C CNN
+F 0 "U32" H 5350 4150 50  0000 C CNN
 F 1 "74XX153" H 5350 2850 50  0000 C CNN
 F 2 "Package_DIP:DIP-16_W7.62mm" H 5350 3550 50  0001 C CNN
@@
 P 4500 6550
 AR Path="/62A08194/638D500F" Ref="SWIO?"  Part="1"
-AR Path="/62FD43AB/638D500F" Ref="SWIO?"  Part="1"
-F 0 "SWIO?" H 4500 6950 50  0000 C CNN
+AR Path="/62FD43AB/638D500F" Ref="SWIO1"  Part="1"
+F 0 "SWIO1" H 4500 6950 50  0000 C CNN
 F 1 "SW_Push_DPDT" H 4500 6944 50  0001 C CNN
 F 2 "Button_Switch_THT:SW_E-Switch_EG2219_DPDT_Angled" H 4500 6750 50  0001 C CNN
@@
 	4850 6650 4700 6650
 $Comp
-L power:GND #PWR?
+L power:GND #PWR045
 U 1 1 6397C066
 P 4850 6950
-F 0 "#PWR?" H 4850 6700 50  0001 C CNN
+F 0 "#PWR045" H 4850 6700 50  0001 C CNN
 F 1 "GND" H 4855 6777 50  0000 C CNN
 F 2 "" H 4850 6950 50  0001 C CNN
@@
 Connection ~ 4850 6650
 $Comp
-L Device:R RVF?
+L Device:R RVF1
 U 1 1 639A492B
 P 4200 6050
-F 0 "RVF?" H 3900 6150 50  0000 L CNN
+F 0 "RVF1" H 3900 6150 50  0000 L CNN
 F 1 "4.7kOm" H 3850 5900 50  0000 L CNN
 F 2 "Resistor_SMD:R_0805_2012Metric_Pad1.20x1.40mm_HandSolder" V 4130 6050 50  0001 C CNN
@@
 $EndComp
 $Comp
-L power:VCC #PWR?
+L power:VCC #PWR044
 U 1 1 639BDFE6
 P 4200 5700
-F 0 "#PWR?" H 4200 5550 50  0001 C CNN
+F 0 "#PWR044" H 4200 5550 50  0001 C CNN
 F 1 "VCC" H 4215 5873 50  0000 C CNN
 F 2 "" H 4200 5700 50  0001 C CNN
@@
 128K/512K
 $Comp
-L 74IEC:74HC86 U?
+L 74IEC:74HC86 U20
 U 4 1 63A0E5BA
 P 5400 5400
-F 0 "U?" H 5400 5550 50  0000 C CNN
+F 0 "U20" H 5400 5550 50  0000 C CNN
 F 1 "74HC86" H 5400 5250 50  0000 C CNN
 F 2 "Package_DIP:DIP-14_W7.62mm" H 5400 5100 50  0001 C CNN
@@
 512KMOD
 $Comp
-L power:GND #PWR?
+L power:GND #PWR047
 U 1 1 6334F3AB
 P 2800 7350
-F 0 "#PWR?" H 2800 7100 50  0001 C CNN
+F 0 "#PWR047" H 2800 7100 50  0001 C CNN
 F 1 "GND" H 2805 7177 50  0000 C CNN
 F 2 "" H 2800 7350 50  0001 C CNN
@@
 Connection ~ 4900 3850
 $Comp
-L power:GND #PWR?
+L power:GND #PWR043
 U 1 1 635A9564
 P 4900 4950
-F 0 "#PWR?" H 4900 4700 50  0001 C CNN
+F 0 "#PWR043" H 4900 4700 50  0001 C CNN
 F 1 "GND" H 4905 4777 50  0000 C CNN
 F 2 "" H 4900 4950 50  0001 C CNN
@@
 	2750 4050 2750 3100
 $Comp
-L Gal:GAL16V8 U?
+L Gal:GAL16V8 U33
 U 1 1 637AE6C9
 P 3300 4300
-F 0 "U?" H 3300 4850 50  0000 C CNN
+F 0 "U33" H 3300 4850 50  0000 C CNN
 F 1 "GAL16V8" H 3300 3750 50  0000 C CNN
 F 2 "Package_DIP:DIP-20_W7.62mm" H 3300 4850 50  0001 C CNN
@@
 512KMOD
 $Comp
-L power:VCC #PWR?
+L power:VCC #PWR042
 U 1 1 64647478
 P 2650 4750
-F 0 "#PWR?" H 2650 4600 50  0001 C CNN
+F 0 "#PWR042" H 2650 4600 50  0001 C CNN
 F 1 "VCC" H 2665 4923 50  0000 C CNN
 F 2 "" H 2650 4750 50  0001 C CNN

Commit message: some change
Parts:
- U31, U32: value 74XX153 -> 74HC153
Changed lines of the file:
@@
 P 5350 1700
 F 0 "U31" H 5350 2350 50  0000 C CNN
-F 1 "74XX153" H 5350 1050 50  0000 C CNN
+F 1 "74HC153" H 5350 1050 50  0000 C CNN
 F 2 "Package_DIP:DIP-16_W7.62mm" H 5350 1750 50  0001 C CNN
 F 3 "https://www.ti.com/lit/ug/scyd013b/scyd013b.pdf" H 5350 1750 50  0001 C CNN
@@
 P 5350 3500
 F 0 "U32" H 5350 4150 50  0000 C CNN
-F 1 "74XX153" H 5350 2850 50  0000 C CNN
+F 1 "74HC153" H 5350 2850 50  0000 C CNN
 F 2 "Package_DIP:DIP-16_W7.62mm" H 5350 3550 50  0001 C CNN
 F 3 "https://www.ti.com/lit/ug/scyd013b/scyd013b.pdf" H 5350 3550 50  0001 C CNN

Commit message: reset annotate and update CPU for new symbol
Parts:
- renumbered RVF1 to RVF?, SWIO1 to SWIO?, U29 to U?, U30 to U?, U34 to U?, U35 to U?, U31 to U?, U32 to U?, U33 to U?, U20 to U?
Changed lines of the file:
@@
 	1400 1700 1500 1600
 $Comp
-L 74IEC:74HC574 U29
+L 74IEC:74HC574 U?
 U 1 1 632C89BD
 P 2200 1500
-F 0 "U29" H 2200 2050 50  0000 C CNN
+F 0 "U?" H 2200 2050 50  0000 C CNN
 F 1 "74HC574" H 2200 950 50  0000 C CNN
 F 2 "Package_DIP:DIP-20_W7.62mm" H 2200 1200 50  0001 C CNN
@@
 $EndComp
 $Comp
-L 74IEC:74HC574 U30
+L 74IEC:74HC574 U?
 U 1 1 632CEC67
 P 3100 1600
-F 0 "U30" H 3100 2150 50  0000 C CNN
+F 0 "U?" H 3100 2150 50  0000 C CNN
 F 1 "74HC574" H 3100 1050 50  0000 C CNN
 F 2 "Package_DIP:DIP-20_W7.62mm" H 3100 1300 50  0001 C CNN
@@
 	2700 2050 2700 2150
 $Comp
-L power:GND #PWR041
+L power:GND #PWR?
 U 1 1 632E6C13
 P 2700 2250
-F 0 "#PWR041" H 2700 2000 50  0001 C CNN
+F 0 "#PWR?" H 2700 2000 50  0001 C CNN
 F 1 "GND" H 2705 2077 50  0000 C CNN
 F 2 "" H 2700 2250 50  0001 C CNN
@@
 C3
 $Comp
-L 74IEC:74HC574 U34
+L 74IEC:74HC574 U?
 U 1 1 6330BD21
 P 2200 6600
-F 0 "U34" H 2200 7150 50  0000 C CNN
+F 0 "U?" H 2200 7150 50  0000 C CNN
 F 1 "74HC574" H 2200 6050 50  0000 C CNN
 F 2 "Package_DIP:DIP-20_W7.62mm" H 2200 6300 50  0001 C CNN
@@
 P 3250 6650
 AR Path="/6332DE4B" Ref="U?"  Part="1"
-AR Path="/62FD43AB/6332DE4B" Ref="U35"  Part="1"
-F 0 "U35" H 3250 7350 50  0000 C CNN
+AR Path="/62FD43AB/6332DE4B" Ref="U?"  Part="1"
+F 0 "U?" H 3250 7350 50  0000 C CNN
 F 1 "74HC166" H 3250 5950 50  0000 C CNN
 F 2 "Package_DIP:DIP-16_W7.62mm" H 3250 6050 50  0001 C CNN
@@
 	2700 7050 2900 7050
 $Comp
-L power:GND #PWR046
+L power:GND #PWR?
 U 1 1 63470A69
 P 1900 7150
-F 0 "#PWR046" H 1900 6900 50  0001 C CNN
+F 0 "#PWR?" H 1900 6900 50  0001 C CNN
 F 1 "GND" H 1905 6977 50  0000 C CNN
 F 2 "" H 1900 7150 50  0001 C CNN
@@
 $EndComp
 $Comp
-L 74IEC:74XX153 U31
+L 74IEC:74XX153 U?
 U 1 1 63481D4A
 P 5350 1700
-F 0 "U31" H 5350 2350 50  0000 C CNN
+F 0 "U?" H 5350 2350 50  0000 C CNN
 F 1 "74HC153" H 5350 1050 50  0000 C CNN
 F 2 "Package_DIP:DIP-16_W7.62mm" H 5350 1750 50  0001 C CNN
@@
 $EndComp
 $Comp
-L 74IEC:74XX153 U32
+L 74IEC:74XX153 U?
 U 1 1 63485DD9
 P 5350 3500
-F 0 "U32" H 5350 4150 50  0000 C CNN
+F 0 "U?" H 5350 4150 50  0000 C CNN
 F 1 "74HC153" H 5350 2850 50  0000 C CNN
 F 2 "Package_DIP:DIP-16_W7.62mm" H 5350 3550 50  0001 C CNN
@@
 P 4500 6550
 AR Path="/62A08194/638D500F" Ref="SWIO?"  Part="1"
-AR Path="/62FD43AB/638D500F" Ref="SWIO1"  Part="1"
-F 0 "SWIO1" H 4500 6950 50  0000 C CNN
+AR Path="/62FD43AB/638D500F" Ref="SWIO?"  Part="1"
+F 0 "SWIO?" H 4500 6950 50  0000 C CNN
 F 1 "SW_Push_DPDT" H 4500 6944 50  0001 C CNN
 F 2 "Button_Switch_THT:SW_E-Switch_EG2219_DPDT_Angled" H 4500 6750 50  0001 C CNN
@@
 	4850 6650 4700 6650
 $Comp
-L power:GND #PWR045
+L power:GND #PWR?
 U 1 1 6397C066
 P 4850 6950
-F 0 "#PWR045" H 4850 6700 50  0001 C CNN
+F 0 "#PWR?" H 4850 6700 50  0001 C CNN
 F 1 "GND" H 4855 6777 50  0000 C CNN
 F 2 "" H 4850 6950 50  0001 C CNN
@@
 Connection ~ 4850 6650
 $Comp
-L Device:R RVF1
+L Device:R RVF?
 U 1 1 639A492B
 P 4200 6050
-F 0 "RVF1" H 3900 6150 50  0000 L CNN
+F 0 "RVF?" H 3900 6150 50  0000 L CNN
 F 1 "4.7kOm" H 3850 5900 50  0000 L CNN
 F 2 "Resistor_SMD:R_0805_2012Metric_Pad1.20x1.40mm_HandSolder" V 4130 6050 50  0001 C CNN
@@
 $EndComp
 $Comp
-L power:VCC #PWR044
+L power:VCC #PWR?
 U 1 1 639BDFE6
 P 4200 5700
-F 0 "#PWR044" H 4200 5550 50  0001 C CNN
+F 0 "#PWR?" H 4200 5550 50  0001 C CNN
 F 1 "VCC" H 4215 5873 50  0000 C CNN
 F 2 "" H 4200 5700 50  0001 C CNN
@@
 128K/512K
 $Comp
-L 74IEC:74HC86 U20
+L 74IEC:74HC86 U?
 U 4 1 63A0E5BA
 P 5400 5400
-F 0 "U20" H 5400 5550 50  0000 C CNN
+F 0 "U?" H 5400 5550 50  0000 C CNN
 F 1 "74HC86" H 5400 5250 50  0000 C CNN
 F 2 "Package_DIP:DIP-14_W7.62mm" H 5400 5100 50  0001 C CNN
@@
 512KMOD
 $Comp
-L power:GND #PWR047
+L power:GND #PWR?
 U 1 1 6334F3AB
 P 2800 7350
-F 0 "#PWR047" H 2800 7100 50  0001 C CNN
+F 0 "#PWR?" H 2800 7100 50  0001 C CNN
 F 1 "GND" H 2805 7177 50  0000 C CNN
 F 2 "" H 2800 7350 50  0001 C CNN
@@
 Connection ~ 4900 3850
 $Comp
-L power:GND #PWR043
+L power:GND #PWR?
 U 1 1 635A9564
 P 4900 4950
-F 0 "#PWR043" H 4900 4700 50  0001 C CNN
+F 0 "#PWR?" H 4900 4700 50  0001 C CNN
 F 1 "GND" H 4905 4777 50  0000 C CNN
 F 2 "" H 4900 4950 50  0001 C CNN
@@
 	2750 4050 2750 3100
 $Comp
-L Gal:GAL16V8 U33
+L Gal:GAL16V8 U?
 U 1 1 637AE6C9
 P 3300 4300
-F 0 "U33" H 3300 4850 50  0000 C CNN
+F 0 "U?" H 3300 4850 50  0000 C CNN
 F 1 "GAL16V8" H 3300 3750 50  0000 C CNN
 F 2 "Package_DIP:DIP-20_W7.62mm" H 3300 4850 50  0001 C CNN
@@
 512KMOD
 $Comp
-L power:VCC #PWR042
+L power:VCC #PWR?
 U 1 1 64647478
 P 2650 4750
-F 0 "#PWR042" H 2650 4600 50  0001 C CNN
+F 0 "#PWR?" H 2650 4600 50  0001 C CNN
 F 1 "VCC" H 2665 4923 50  0000 C CNN
 F 2 "" H 2650 4750 50  0001 C CNN

Commit message: fix erc
Parts:
- gave numbers to parts that had none: 10
Changed lines of the file:
@@
 Wire Wire Line
 	1400 1700 950  1700
-Text GLabel 950  1700 0    50   Input ~ 10
+Text HLabel 950  1700 0    50   Input ~ 10
 MD0
-Text GLabel 950  1800 0    50   Input ~ 10
+Text HLabel 950  1800 0    50   Input ~ 10
 MD1
-Text GLabel 950  1900 0    50   Input ~ 10
+Text HLabel 950  1900 0    50   Input ~ 10
 MD2
-Text GLabel 950  2000 0    50   Input ~ 10
+Text HLabel 950  2000 0    50   Input ~ 10
 MD3
-Text GLabel 950  2100 0    50   Input ~ 10
+Text HLabel 950  2100 0    50   Input ~ 10
 MD4
-Text GLabel 950  2200 0    50   Input ~ 10
+Text HLabel 950  2200 0    50   Input ~ 10
 MD5
-Text GLabel 950  2300 0    50   Input ~ 10
+Text HLabel 950  2300 0    50   Input ~ 10
 MD6
-Text GLabel 950  2400 0    50   Input ~ 10
+Text HLabel 950  2400 0    50   Input ~ 10
 MD7
 Entry Wire Line
@@
 	1400 1700 1500 1600
 $Comp
-L 74IEC:74HC574 U?
+L 74IEC:74HC574 U29
 U 1 1 632C89BD
 P 2200 1500
-F 0 "U?" H 2200 2050 50  0000 C CNN
+F 0 "U29" H 2200 2050 50  0000 C CNN
 F 1 "74HC574" H 2200 950 50  0000 C CNN
 F 2 "Package_DIP:DIP-20_W7.62mm" H 2200 1200 50  0001 C CNN
@@
 $EndComp
 $Comp
-L 74IEC:74HC574 U?
+L 74IEC:74HC574 U30
 U 1 1 632CEC67
 P 3100 1600
-F 0 "U?" H 3100 2150 50  0000 C CNN
+F 0 "U30" H 3100 2150 50  0000 C CNN
 F 1 "74HC574" H 3100 1050 50  0000 C CNN
 F 2 "Package_DIP:DIP-20_W7.62mm" H 3100 1300 50  0001 C CNN
@@
 	2700 2050 2700 2150
 $Comp
-L power:GND #PWR?
+L power:GND #PWR0141
 U 1 1 632E6C13
 P 2700 2250
-F 0 "#PWR?" H 2700 2000 50  0001 C CNN
+F 0 "#PWR0141" H 2700 2000 50  0001 C CNN
 F 1 "GND" H 2705 2077 50  0000 C CNN
 F 2 "" H 2700 2250 50  0001 C CNN
@@
 C3
 $Comp
-L 74IEC:74HC574 U?
+L 74IEC:74HC574 U34
 U 1 1 6330BD21
 P 2200 6600
-F 0 "U?" H 2200 7150 50  0000 C CNN
+F 0 "U34" H 2200 7150 50  0000 C CNN
 F 1 "74HC574" H 2200 6050 50  0000 C CNN
 F 2 "Package_DIP:DIP-20_W7.62mm" H 2200 6300 50  0001 C CNN
@@
 P 3250 6650
 AR Path="/6332DE4B" Ref="U?"  Part="1"
-AR Path="/62FD43AB/6332DE4B" Ref="U?"  Part="1"
-F 0 "U?" H 3250 7350 50  0000 C CNN
+AR Path="/62FD43AB/6332DE4B" Ref="U35"  Part="1"
+F 0 "U35" H 3250 7350 50  0000 C CNN
 F 1 "74HC166" H 3250 5950 50  0000 C CNN
 F 2 "Package_DIP:DIP-16_W7.62mm" H 3250 6050 50  0001 C CNN
@@
 	2700 7050 2900 7050
 $Comp
-L power:GND #PWR?
+L power:GND #PWR0142
 U 1 1 63470A69
 P 1900 7150
-F 0 "#PWR?" H 1900 6900 50  0001 C CNN
+F 0 "#PWR0142" H 1900 6900 50  0001 C CNN
 F 1 "GND" H 1905 6977 50  0000 C CNN
 F 2 "" H 1900 7150 50  0001 C CNN
@@
 $EndComp
 $Comp
-L 74IEC:74XX153 U?
+L 74IEC:74XX153 U31
 U 1 1 63481D4A
 P 5350 1700
-F 0 "U?" H 5350 2350 50  0000 C CNN
+F 0 "U31" H 5350 2350 50  0000 C CNN
 F 1 "74HC153" H 5350 1050 50  0000 C CNN
 F 2 "Package_DIP:DIP-16_W7.62mm" H 5350 1750 50  0001 C CNN
@@
 $EndComp
 $Comp
-L 74IEC:74XX153 U?
+L 74IEC:74XX153 U32
 U 1 1 63485DD9
 P 5350 3500
-F 0 "U?" H 5350 4150 50  0000 C CNN
+F 0 "U32" H 5350 4150 50  0000 C CNN
 F 1 "74HC153" H 5350 2850 50  0000 C CNN
 F 2 "Package_DIP:DIP-16_W7.62mm" H 5350 3550 50  0001 C CNN
@@
 P 4500 6550
 AR Path="/62A08194/638D500F" Ref="SWIO?"  Part="1"
-AR Path="/62FD43AB/638D500F" Ref="SWIO?"  Part="1"
-F 0 "SWIO?" H 4500 6950 50  0000 C CNN
+AR Path="/62FD43AB/638D500F" Ref="SWIO1"  Part="1"
+F 0 "SWIO1" H 4500 6950 50  0000 C CNN
 F 1 "SW_Push_DPDT" H 4500 6944 50  0001 C CNN
 F 2 "Button_Switch_THT:SW_E-Switch_EG2219_DPDT_Angled" H 4500 6750 50  0001 C CNN
@@
 	4850 6650 4700 6650
 $Comp
-L power:GND #PWR?
+L power:GND #PWR0143
 U 1 1 6397C066
 P 4850 6950
-F 0 "#PWR?" H 4850 6700 50  0001 C CNN
+F 0 "#PWR0143" H 4850 6700 50  0001 C CNN
 F 1 "GND" H 4855 6777 50  0000 C CNN
 F 2 "" H 4850 6950 50  0001 C CNN
@@
 Connection ~ 4850 6650
 $Comp
-L Device:R RVF?
+L Device:R RVF1
 U 1 1 639A492B
 P 4200 6050
-F 0 "RVF?" H 3900 6150 50  0000 L CNN
+F 0 "RVF1" H 3900 6150 50  0000 L CNN
 F 1 "4.7kOm" H 3850 5900 50  0000 L CNN
 F 2 "Resistor_SMD:R_0805_2012Metric_Pad1.20x1.40mm_HandSolder" V 4130 6050 50  0001 C CNN
@@
 $EndComp
 $Comp
-L power:VCC #PWR?
+L power:VCC #PWR0144
 U 1 1 639BDFE6
 P 4200 5700
-F 0 "#PWR?" H 4200 5550 50  0001 C CNN
+F 0 "#PWR0144" H 4200 5550 50  0001 C CNN
 F 1 "VCC" H 4215 5873 50  0000 C CNN
 F 2 "" H 4200 5700 50  0001 C CNN
@@
 128K/512K
 $Comp
-L 74IEC:74HC86 U?
+L 74IEC:74HC86 U20
 U 4 1 63A0E5BA
 P 5400 5400
-F 0 "U?" H 5400 5550 50  0000 C CNN
+F 0 "U20" H 5400 5550 50  0000 C CNN
 F 1 "74HC86" H 5400 5250 50  0000 C CNN
 F 2 "Package_DIP:DIP-14_W7.62mm" H 5400 5100 50  0001 C CNN
@@
 Text Label 1400 4000 2    50   ~ 0
 BL
-Text GLabel 1000 2550 0    50   Input ~ 10
+Text HLabel 1000 2550 0    50   Input ~ 10
 F25Hz
-Text GLabel 1000 2650 0    50   Input ~ 10
+Text HLabel 1000 2650 0    50   Input ~ 10
 CBRDB
-Text GLabel 1000 2750 0    50   Input ~ 10
+Text HLabel 1000 2750 0    50   Input ~ 10
 CBRDR
-Text GLabel 1000 2850 0    50   Input ~ 10
+Text HLabel 1000 2850 0    50   Input ~ 10
 CBRDG
-Text GLabel 1000 2950 0    50   Input ~ 10
+Text HLabel 1000 2950 0    50   Input ~ 10
 PA6
-Text GLabel 1000 3050 0    50   Input ~ 10
+Text HLabel 1000 3050 0    50   Input ~ 10
 PA7
-Text GLabel 1000 3200 0    50   Input ~ 10
+Text HLabel 1000 3200 0    50   Input ~ 10
 ~C1
-Text GLabel 1000 3350 0    50   Input ~ 10
+Text HLabel 1000 3350 0    50   Input ~ 10
 ~C2
-Text GLabel 1000 3500 0    50   Input ~ 10
+Text HLabel 1000 3500 0    50   Input ~ 10
 C3
-Text GLabel 1000 3600 0    50   Input ~ 10
+Text HLabel 1000 3600 0    50   Input ~ 10
 C5
-Text GLabel 1000 3700 0    50   Input ~ 10
+Text HLabel 1000 3700 0    50   Input ~ 10
 FSYNC
-Text GLabel 1000 3800 0    50   Input ~ 10
+Text HLabel 1000 3800 0    50   Input ~ 10
 C17
-Text GLabel 1000 3900 0    50   Input ~ 10
+Text HLabel 1000 3900 0    50   Input ~ 10
 C18
-Text GLabel 1000 4000 0    50   Input ~ 10
+Text HLabel 1000 4000 0    50   Input ~ 10
 BL
 Wire Wire Line
@@
 512KMOD
 $Comp
-L power:GND #PWR?
+L power:GND #PWR0145
 U 1 1 6334F3AB
 P 2800 7350
-F 0 "#PWR?" H 2800 7100 50  0001 C CNN
+F 0 "#PWR0145" H 2800 7100 50  0001 C CNN
 F 1 "GND" H 2805 7177 50  0000 C CNN
 F 2 "" H 2800 7350 50  0001 C CNN
@@
 Connection ~ 4900 3850
 $Comp
-L power:GND #PWR?
+L power:GND #PWR0146
 U 1 1 635A9564
 P 4900 4950
-F 0 "#PWR?" H 4900 4700 50  0001 C CNN
+F 0 "#PWR0146" H 4900 4700 50  0001 C CNN
 F 1 "GND" H 4905 4777 50  0000 C CNN
 F 2 "" H 4900 4950 50  0001 C CNN
@@
 	2750 4050 2750 3100
 $Comp
-L Gal:GAL16V8 U?
+L Gal:GAL16V8 U33
 U 1 1 637AE6C9
 P 3300 4300
-F 0 "U?" H 3300 4850 50  0000 C CNN
+F 0 "U33" H 3300 4850 50  0000 C CNN
 F 1 "GAL16V8" H 3300 3750 50  0000 C CNN
 F 2 "Package_DIP:DIP-20_W7.62mm" H 3300 4850 50  0001 C CNN
@@
 512KMOD
 $Comp
-L power:VCC #PWR?
+L power:VCC #PWR0147
 U 1 1 64647478
 P 2650 4750
-F 0 "#PWR?" H 2650 4600 50  0001 C CNN
+F 0 "#PWR0147" H 2650 4600 50  0001 C CNN
 F 1 "VCC" H 2665 4923 50  0000 C CNN
 F 2 "" H 2650 4750 50  0001 C CNN
@@
 	4700 4450 4700 3950
 Connection ~ 4700 3950
-Text GLabel 6000 4650 2    50   Output ~ 10
+Text HLabel 6000 4650 2    50   Output ~ 10
 GPA6
-Text GLabel 6000 4550 2    50   Output ~ 10
+Text HLabel 6000 4550 2    50   Output ~ 10
 GPA7
-Text GLabel 6000 5400 2    50   Output ~ 10
+Text HLabel 6000 5400 2    50   Output ~ 10
 TTLSYNC
-Text GLabel 6000 3800 2    50   Output ~ 10
+Text HLabel 6000 3800 2    50   Output ~ 10
 TTLY
-Text GLabel 6000 3200 2    50   Output ~ 10
+Text HLabel 6000 3200 2    50   Output ~ 10
 TTLG
-Text GLabel 6000 2000 2    50   Output ~ 10
+Text HLabel 6000 2000 2    50   Output ~ 10
 TTLR
-Text GLabel 6000 1400 2    50   Output ~ 10
+Text HLabel 6000 1400 2    50   Output ~ 10
 TTLB
 NoConn ~ 4700 6450
@@
 	5000 4050 4800 4050
 Wire Bus Line
-	1500 950  1500 7500
+	1500 950  1500 7350
 $EndSCHEMATC
