File: ZX-Spectrum-Pentagon/VideoFormating.sch (KiCad schematic (older format))
At the start: 10 parts, among them U20 74HC86, U29 74HC574, U30 74HC574, U31 74HC153, U32 74HC153, U33 GAL16V8, U34 74HC574, U35 74HC166

Commit message: move from globag label to hierarchical label. fix all warning
Connections:
- wire segments 185 -> 186
Changed lines of the file:
@@
 Comment4 ""
 $EndDescr
-Text Label 1400 2400 2    50   ~ 0
-MD7
-Text Label 1400 2300 2    50   ~ 0
-MD6
-Text Label 1400 2200 2    50   ~ 0
-MD5
-Text Label 1400 2100 2    50   ~ 0
-MD4
-Text Label 1400 2000 2    50   ~ 0
-MD3
-Text Label 1400 1900 2    50   ~ 0
-MD2
-Text Label 1400 1800 2    50   ~ 0
-MD1
-Text Label 1400 1700 2    50   ~ 0
-MD0
-Wire Wire Line
-	1400 2400 950  2400
-Wire Wire Line
-	1400 2300 950  2300
-Wire Wire Line
-	1400 2200 950  2200
-Wire Wire Line
-	1400 2100 950  2100
-Wire Wire Line
-	1400 2000 950  2000
-Wire Wire Line
-	1400 1900 950  1900
-Wire Wire Line
-	1400 1800 950  1800
-Wire Wire Line
-	1400 1700 950  1700
-Text HLabel 950  1700 0    50   Input ~ 10
-MD0
-Text HLabel 950  1800 0    50   Input ~ 10
-MD1
-Text HLabel 950  1900 0    50   Input ~ 10
-MD2
-Text HLabel 950  2000 0    50   Input ~ 10
-MD3
-Text HLabel 950  2100 0    50   Input ~ 10
-MD4
-Text HLabel 950  2200 0    50   Input ~ 10
-MD5
-Text HLabel 950  2300 0    50   Input ~ 10
-MD6
-Text HLabel 950  2400 0    50   Input ~ 10
-MD7
-Entry Wire Line
-	1400 2400 1500 2300
-Entry Wire Line
-	1400 2300 1500 2200
-Entry Wire Line
-	1400 2200 1500 2100
-Entry Wire Line
-	1400 2100 1500 2000
-Entry Wire Line
-	1400 2000 1500 1900
-Entry Wire Line
-	1400 1900 1500 1800
-Entry Wire Line
-	1400 1800 1500 1700
-Entry Wire Line
-	1400 1700 1500 1600
 $Comp
 L 74IEC:74HC574 U29
@@
 	2700 2050 2700 2150
 $Comp
-L power:GND #PWR0141
+L power:GND #PWR041
 U 1 1 632E6C13
 P 2700 2250
-F 0 "#PWR0141" H 2700 2000 50  0001 C CNN
+F 0 "#PWR041" H 2700 2000 50  0001 C CNN
 F 1 "GND" H 2705 2077 50  0000 C CNN
 F 2 "" H 2700 2250 50  0001 C CNN
@@
 Text Label 1600 1250 0    50   ~ 0
 MD2
-Text Label 1600 1150 0    50   ~ 0
-MD1
 Text Label 1600 1050 0    50   ~ 0
 MD0
@@
 	1600 1250 1900 1250
 Wire Wire Line
-	1600 1150 1900 1150
-Wire Wire Line
 	1600 1050 1900 1050
 Entry Wire Line
@@
 Entry Wire Line
 	1600 1250 1500 1150
-Entry Wire Line
-	1600 1150 1500 1050
 Entry Wire Line
 	1600 1050 1500 950
@@
 Text Label 1600 6650 0    50   ~ 0
 MD5
-Text Label 1600 6550 0    50   ~ 0
-MD4
-Text Label 1600 6450 0    50   ~ 0
-MD3
 Text Label 1600 6350 0    50   ~ 0
 MD2
-Text Label 1600 6250 0    50   ~ 0
-MD1
 Text Label 1600 6150 0    50   ~ 0
 MD0
@@
 	1600 6650 1900 6650
 Wire Wire Line
-	1600 6550 1900 6550
-Wire Wire Line
-	1600 6450 1900 6450
-Wire Wire Line
 	1600 6350 1900 6350
 Wire Wire Line
-	1600 6250 1900 6250
-Wire Wire Line
 	1600 6150 1900 6150
 Entry Wire Line
@@
 	1600 6650 1500 6550
 Entry Wire Line
-	1600 6550 1500 6450
-Entry Wire Line
-	1600 6450 1500 6350
-Entry Wire Line
 	1600 6350 1500 6250
-Entry Wire Line
-	1600 6250 1500 6150
 Entry Wire Line
 	1600 6150 1500 6050
@@
 Connection ~ 2800 7250
 Wire Wire Line
-	1900 7050 1900 7150
-Wire Wire Line
 	2900 7150 2650 7150
 Wire Wire Line
@@
 	2700 7050 2900 7050
 $Comp
-L power:GND #PWR0142
+L power:GND #PWR046
 U 1 1 63470A69
-P 1900 7150
-F 0 "#PWR0142" H 1900 6900 50  0001 C CNN
-F 1 "GND" H 1905 6977 50  0000 C CNN
-F 2 "" H 1900 7150 50  0001 C CNN
-F 3 "" H 1900 7150 50  0001 C CNN
-	1    1900 7150
+P 1800 7150
+F 0 "#PWR046" H 1800 6900 50  0001 C CNN
+F 1 "GND" H 1805 6977 50  0000 C CNN
+F 2 "" H 1800 7150 50  0001 C CNN
+F 3 "" H 1800 7150 50  0001 C CNN
+	1    1800 7150
 	1    0    0    -1
 $EndComp
@@
 	4850 6650 4700 6650
 $Comp
-L power:GND #PWR0143
+L power:GND #PWR045
 U 1 1 6397C066
 P 4850 6950
-F 0 "#PWR0143" H 4850 6700 50  0001 C CNN
+F 0 "#PWR045" H 4850 6700 50  0001 C CNN
 F 1 "GND" H 4855 6777 50  0000 C CNN
 F 2 "" H 4850 6950 50  0001 C CNN
@@
 $EndComp
 $Comp
-L power:VCC #PWR0144
+L power:VCC #PWR044
 U 1 1 639BDFE6
 P 4200 5700
-F 0 "#PWR0144" H 4200 5550 50  0001 C CNN
+F 0 "#PWR044" H 4200 5550 50  0001 C CNN
 F 1 "VCC" H 4215 5873 50  0000 C CNN
 F 2 "" H 4200 5700 50  0001 C CNN
@@
 512KMOD
 $Comp
-L power:GND #PWR0145
+L power:GND #PWR047
 U 1 1 6334F3AB
 P 2800 7350
-F 0 "#PWR0145" H 2800 7100 50  0001 C CNN
+F 0 "#PWR047" H 2800 7100 50  0001 C CNN
 F 1 "GND" H 2805 7177 50  0000 C CNN
 F 2 "" H 2800 7350 50  0001 C CNN
@@
 Connection ~ 4900 3850
 $Comp
-L power:GND #PWR0146
+L power:GND #PWR043
 U 1 1 635A9564
 P 4900 4950
-F 0 "#PWR0146" H 4900 4700 50  0001 C CNN
+F 0 "#PWR043" H 4900 4700 50  0001 C CNN
 F 1 "GND" H 4905 4777 50  0000 C CNN
 F 2 "" H 4900 4950 50  0001 C CNN
@@
 512KMOD
 $Comp
-L power:VCC #PWR0147
+L power:VCC #PWR042
 U 1 1 64647478
 P 2650 4750
-F 0 "#PWR0147" H 2650 4600 50  0001 C CNN
+F 0 "#PWR042" H 2650 4600 50  0001 C CNN
 F 1 "VCC" H 2665 4923 50  0000 C CNN
 F 2 "" H 2650 4750 50  0001 C CNN
@@
 Wire Wire Line
 	5000 4050 4800 4050
+Wire Wire Line
+	1900 7050 1800 7050
+Wire Wire Line
+	1800 7050 1800 7150
+Entry Wire Line
+	1500 1050 1600 1150
+Wire Wire Line
+	1600 1150 1900 1150
+Text Label 1600 1150 0    50   ~ 0
+MD1
+Entry Wire Line
+	1500 6150 1600 6250
+Entry Wire Line
+	1500 6350 1600 6450
+Entry Wire Line
+	1500 6450 1600 6550
+Wire Wire Line
+	1600 6250 1900 6250
+Wire Wire Line
+	1600 6450 1900 6450
+Wire Wire Line
+	1600 6550 1900 6550
+Text Label 1600 6250 0    50   ~ 0
+MD1
+Text Label 1600 6450 0    50   ~ 0
+MD3
+Text Label 1600 6550 0    50   ~ 0
+MD4
+Text HLabel 1000 1050 0    50   Input ~ 0
+MD0
+Text HLabel 1000 1150 0    50   Input ~ 0
+MD1
+Text HLabel 1000 1250 0    50   Input ~ 0
+MD2
+Text HLabel 1000 1350 0    50   Input ~ 0
+MD3
+Text HLabel 1000 1450 0    50   Input ~ 0
+MD4
+Text HLabel 1000 1550 0    50   Input ~ 0
+MD5
+Text HLabel 1000 1650 0    50   Input ~ 0
+MD6
+Text HLabel 1000 1750 0    50   Input ~ 0
+MD7
+Entry Wire Line
+	1400 1050 1500 950
+Entry Wire Line
+	1400 1150 1500 1050
+Entry Wire Line
+	1400 1250 1500 1150
+Entry Wire Line
+	1400 1350 1500 1250
+Entry Wire Line
+	1400 1450 1500 1350
+Entry Wire Line
+	1400 1550 1500 1450
+Entry Wire Line
+	1400 1650 1500 1550
+Entry Wire Line
+	1400 1750 1500 1650
+Wire Wire Line
+	1000 1750 1400 1750
+Wire Wire Line
+	1000 1650 1400 1650
+Wire Wire Line
+	1000 1550 1400 1550
+Wire Wire Line
+	1000 1450 1400 1450
+Wire Wire Line
+	1000 1350 1400 1350
+Wire Wire Line
+	1000 1250 1400 1250
+Wire Wire Line
+	1000 1150 1400 1150
+Wire Wire Line
+	1000 1050 1400 1050
 Wire Bus Line
 	1500 950  1500 7350
+Text Label 1400 1050 2    50   ~ 0
+MD0
+Text Label 1400 1150 2    50   ~ 0
+MD1
+Text Label 1400 1250 2    50   ~ 0
+MD2
+Text Label 1400 1350 2    50   ~ 0
+MD3
+Text Label 1400 1450 2    50   ~ 0
+MD4
+Text Label 1400 1550 2    50   ~ 0
+MD5
+Text Label 1400 1650 2    50   ~ 0
+MD6
+Text Label 1400 1750 2    50   ~ 0
+MD7
 $EndSCHEMATC

Commit message: clear annotation
Parts:
- renumbered RVF1 to RVF?, SWIO1 to SWIO?, U29 to U?, U30 to U?, U34 to U?, U35 to U?, U31 to U?, U32 to U?, U33 to U?, U20 to U?
Changed lines of the file:
@@
 $EndDescr
 $Comp
-L 74IEC:74HC574 U29
+L 74IEC:74HC574 U?
 U 1 1 632C89BD
 P 2200 1500
-F 0 "U29" H 2200 2050 50  0000 C CNN
+F 0 "U?" H 2200 2050 50  0000 C CNN
 F 1 "74HC574" H 2200 950 50  0000 C CNN
 F 2 "Package_DIP:DIP-20_W7.62mm" H 2200 1200 50  0001 C CNN
@@
 $EndComp
 $Comp
-L 74IEC:74HC574 U30
+L 74IEC:74HC574 U?
 U 1 1 632CEC67
 P 3100 1600
-F 0 "U30" H 3100 2150 50  0000 C CNN
+F 0 "U?" H 3100 2150 50  0000 C CNN
 F 1 "74HC574" H 3100 1050 50  0000 C CNN
 F 2 "Package_DIP:DIP-20_W7.62mm" H 3100 1300 50  0001 C CNN
@@
 	2700 2050 2700 2150
 $Comp
-L power:GND #PWR041
+L power:GND #PWR?
 U 1 1 632E6C13
 P 2700 2250
-F 0 "#PWR041" H 2700 2000 50  0001 C CNN
+F 0 "#PWR?" H 2700 2000 50  0001 C CNN
 F 1 "GND" H 2705 2077 50  0000 C CNN
 F 2 "" H 2700 2250 50  0001 C CNN
@@
 C3
 $Comp
-L 74IEC:74HC574 U34
+L 74IEC:74HC574 U?
 U 1 1 6330BD21
 P 2200 6600
-F 0 "U34" H 2200 7150 50  0000 C CNN
+F 0 "U?" H 2200 7150 50  0000 C CNN
 F 1 "74HC574" H 2200 6050 50  0000 C CNN
 F 2 "Package_DIP:DIP-20_W7.62mm" H 2200 6300 50  0001 C CNN
@@
 P 3250 6650
 AR Path="/6332DE4B" Ref="U?"  Part="1"
-AR Path="/62FD43AB/6332DE4B" Ref="U35"  Part="1"
-F 0 "U35" H 3250 7350 50  0000 C CNN
+AR Path="/62FD43AB/6332DE4B" Ref="U?"  Part="1"
+F 0 "U?" H 3250 7350 50  0000 C CNN
 F 1 "74HC166" H 3250 5950 50  0000 C CNN
 F 2 "Package_DIP:DIP-16_W7.62mm" H 3250 6050 50  0001 C CNN
@@
 	2700 7050 2900 7050
 $Comp
-L power:GND #PWR046
+L power:GND #PWR?
 U 1 1 63470A69
 P 1800 7150
-F 0 "#PWR046" H 1800 6900 50  0001 C CNN
+F 0 "#PWR?" H 1800 6900 50  0001 C CNN
 F 1 "GND" H 1805 6977 50  0000 C CNN
 F 2 "" H 1800 7150 50  0001 C CNN
@@
 $EndComp
 $Comp
-L 74IEC:74XX153 U31
+L 74IEC:74XX153 U?
 U 1 1 63481D4A
 P 5350 1700
-F 0 "U31" H 5350 2350 50  0000 C CNN
+F 0 "U?" H 5350 2350 50  0000 C CNN
 F 1 "74HC153" H 5350 1050 50  0000 C CNN
 F 2 "Package_DIP:DIP-16_W7.62mm" H 5350 1750 50  0001 C CNN
@@
 $EndComp
 $Comp
-L 74IEC:74XX153 U32
+L 74IEC:74XX153 U?
 U 1 1 63485DD9
 P 5350 3500
-F 0 "U32" H 5350 4150 50  0000 C CNN
+F 0 "U?" H 5350 4150 50  0000 C CNN
 F 1 "74HC153" H 5350 2850 50  0000 C CNN
 F 2 "Package_DIP:DIP-16_W7.62mm" H 5350 3550 50  0001 C CNN
@@
 P 4500 6550
 AR Path="/62A08194/638D500F" Ref="SWIO?"  Part="1"
-AR Path="/62FD43AB/638D500F" Ref="SWIO1"  Part="1"
-F 0 "SWIO1" H 4500 6950 50  0000 C CNN
+AR Path="/62FD43AB/638D500F" Ref="SWIO?"  Part="1"
+F 0 "SWIO?" H 4500 6950 50  0000 C CNN
 F 1 "SW_Push_DPDT" H 4500 6944 50  0001 C CNN
 F 2 "Button_Switch_THT:SW_E-Switch_EG2219_DPDT_Angled" H 4500 6750 50  0001 C CNN
@@
 	4850 6650 4700 6650
 $Comp
-L power:GND #PWR045
+L power:GND #PWR?
 U 1 1 6397C066
 P 4850 6950
-F 0 "#PWR045" H 4850 6700 50  0001 C CNN
+F 0 "#PWR?" H 4850 6700 50  0001 C CNN
 F 1 "GND" H 4855 6777 50  0000 C CNN
 F 2 "" H 4850 6950 50  0001 C CNN
@@
 Connection ~ 4850 6650
 $Comp
-L Device:R RVF1
+L Device:R RVF?
 U 1 1 639A492B
 P 4200 6050
-F 0 "RVF1" H 3900 6150 50  0000 L CNN
+F 0 "RVF?" H 3900 6150 50  0000 L CNN
 F 1 "4.7kOm" H 3850 5900 50  0000 L CNN
 F 2 "Resistor_SMD:R_0805_2012Metric_Pad1.20x1.40mm_HandSolder" V 4130 6050 50  0001 C CNN
@@
 $EndComp
 $Comp
-L power:VCC #PWR044
+L power:VCC #PWR?
 U 1 1 639BDFE6
 P 4200 5700
-F 0 "#PWR044" H 4200 5550 50  0001 C CNN
+F 0 "#PWR?" H 4200 5550 50  0001 C CNN
 F 1 "VCC" H 4215 5873 50  0000 C CNN
 F 2 "" H 4200 5700 50  0001 C CNN
@@
 128K/512K
 $Comp
-L 74IEC:74HC86 U20
+L 74IEC:74HC86 U?
 U 4 1 63A0E5BA
 P 5400 5400
-F 0 "U20" H 5400 5550 50  0000 C CNN
+F 0 "U?" H 5400 5550 50  0000 C CNN
 F 1 "74HC86" H 5400 5250 50  0000 C CNN
 F 2 "Package_DIP:DIP-14_W7.62mm" H 5400 5100 50  0001 C CNN
@@
 512KMOD
 $Comp
-L power:GND #PWR047
+L power:GND #PWR?
 U 1 1 6334F3AB
 P 2800 7350
-F 0 "#PWR047" H 2800 7100 50  0001 C CNN
+F 0 "#PWR?" H 2800 7100 50  0001 C CNN
 F 1 "GND" H 2805 7177 50  0000 C CNN
 F 2 "" H 2800 7350 50  0001 C CNN
@@
 Connection ~ 4900 3850
 $Comp
-L power:GND #PWR043
+L power:GND #PWR?
 U 1 1 635A9564
 P 4900 4950
-F 0 "#PWR043" H 4900 4700 50  0001 C CNN
+F 0 "#PWR?" H 4900 4700 50  0001 C CNN
 F 1 "GND" H 4905 4777 50  0000 C CNN
 F 2 "" H 4900 4950 50  0001 C CNN
@@
 	2750 4050 2750 3100
 $Comp
-L Gal:GAL16V8 U33
+L Gal:GAL16V8 U?
 U 1 1 637AE6C9
 P 3300 4300
-F 0 "U33" H 3300 4850 50  0000 C CNN
+F 0 "U?" H 3300 4850 50  0000 C CNN
 F 1 "GAL16V8" H 3300 3750 50  0000 C CNN
 F 2 "Package_DIP:DIP-20_W7.62mm" H 3300 4850 50  0001 C CNN
@@
 512KMOD
 $Comp
-L power:VCC #PWR042
+L power:VCC #PWR?
 U 1 1 64647478
 P 2650 4750
-F 0 "#PWR042" H 2650 4600 50  0001 C CNN
+F 0 "#PWR?" H 2650 4600 50  0001 C CNN
 F 1 "VCC" H 2665 4923 50  0000 C CNN
 F 2 "" H 2650 4750 50  0001 C CNN

Commit message: use bold for MD0-MD8 on VideoFormating
Changed lines of the file:
@@
 Text Label 1600 6550 0    50   ~ 0
 MD4
-Text HLabel 1000 1050 0    50   Input ~ 0
+Text HLabel 1000 1050 0    50   Input ~ 10
 MD0
-Text HLabel 1000 1150 0    50   Input ~ 0
+Text HLabel 1000 1150 0    50   Input ~ 10
 MD1
-Text HLabel 1000 1250 0    50   Input ~ 0
+Text HLabel 1000 1250 0    50   Input ~ 10
 MD2
-Text HLabel 1000 1350 0    50   Input ~ 0
+Text HLabel 1000 1350 0    50   Input ~ 10
 MD3
-Text HLabel 1000 1450 0    50   Input ~ 0
+Text HLabel 1000 1450 0    50   Input ~ 10
 MD4
-Text HLabel 1000 1550 0    50   Input ~ 0
+Text HLabel 1000 1550 0    50   Input ~ 10
 MD5
-Text HLabel 1000 1650 0    50   Input ~ 0
+Text HLabel 1000 1650 0    50   Input ~ 10
 MD6
-Text HLabel 1000 1750 0    50   Input ~ 0
+Text HLabel 1000 1750 0    50   Input ~ 10
 MD7
 Entry Wire Line
@@
 Wire Wire Line
 	1000 1050 1400 1050
-Wire Bus Line
-	1500 950  1500 7350
 Text Label 1400 1050 2    50   ~ 0
 MD0
@@
 Text Label 1400 1750 2    50   ~ 0
 MD7
+Wire Bus Line
+	1500 950  1500 7350
 $EndSCHEMATC
