File: ZX-Spectrum-Pentagon/ZX-Spectrum-Keyboard_Switch.kicad_pcb (KiCad board)
At the start: 2 copper layers, 283.2 x 111.1 mm, 8 parts

Commit message: restore ZX-Spectrum-Keyboard_Switch.kicad_sch
Parts:
- H1, H2, H3, H4, H5, H6, H7, H8: footprint MountingHole:MountingHole_2.7mm_M2.5_Pad_Via -> MountingHole:MountingHole_2.2mm_M2_Pad_Via
- moved H8 0.43 mm to (305.0, 133.3)
