File: ZX-Spectrum-Pentagon/ZX-Spectrum-HDMI.kicad_sch (KiCad schematic)
At the start: 0 parts

Commit message: add HDMI adapter
Parts:
- added U?: ADV7513BSWZ, Package_QFP:LQFP-64-1EP_10x10mm_P0.5mm_EP5x5mm, symbol adv7513:ADV7513BSWZ
Connections:
- new net: U?.1 (DVDD), U?.11 (DVDD), U?.31 (DVDD), U?.51 (DVDD)
- new net: U?.15 (AVDD), U?.19 (AVDD), U?.25 (AVDD)
