File: mdconnectors/mdconnector.kicad_sch (KiCad schematic)
At the start: 7 parts

Commit message: improve libraty
Parts:
- CN1: renamed from CN?; footprint (none) -> MD-XXSM:CUI_MD-30SM
- CN2: renamed from CN?; footprint (none) -> MD-XXSM:CUI_MD-40SM
- CN3: renamed from CN?; footprint (none) -> MD-XXSM:CUI_MD-50SM
- CN4: renamed from CN?; footprint (none) -> MD-XXSM:CUI_MD-60SM
- CN5: renamed from CN?; footprint (none) -> MD-XXSM:CUI_MD-70SM
- CN6: renamed from CN?; footprint (none) -> MD-XXSM:CUI_MD-80SM
- CN7: renamed from CN?; footprint (none) -> MD-XXSM:CUI_MD-90SM
Changed lines of the file:
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@@
   (symbol (lib_id "mdconnector:MD-50") (at 168.91 53.34 0) (unit 1)
     (in_bom yes) (on_board yes) (fields_autoplaced)
-    (property "Reference" "CN?" (id 0) (at 168.91 40.64 0))
+    (property "Reference" "CN3" (id 0) (at 168.91 40.64 0))
     (property "Value" "MD-50" (id 1) (at 168.91 43.18 0))
-    (property "Footprint" "" (id 2) (at 168.91 53.34 0)
+    (property "Footprint" "MD-XXSM:CUI_MD-50SM" (id 2) (at 168.91 53.34 0)
       (effects (font (size 1.27 1.27)) hide)
     )
-    (property "Datasheet" "" (id 3) (at 168.91 53.34 0)
+    (property "Datasheet" "https://eu.mouser.com/datasheet/2/670/md_sm_series-1778126.pdf" (id 3) (at 168.91 53.34 0)
       (effects (font (size 1.27 1.27)) hide)
     )
     (pin "1")
-    (pin "10")
-    (pin "11")
-    (pin "12")
     (pin "2")
     (pin "3")
     (pin "4")
     (pin "5")
+    (pin "S1")
+    (pin "S2")
+    (pin "S3")
   )
   (symbol (lib_id "mdconnector:MD-40") (at 140.97 53.34 0) (unit 1)
     (in_bom yes) (on_board yes) (fields_autoplaced)
-    (property "Reference" "CN?" (id 0) (at 140.97 40.64 0))
+    (property "Reference" "CN2" (id 0) (at 140.97 40.64 0))
     (property "Value" "MD-40" (id 1) (at 140.97 43.18 0))
-    (property "Footprint" "" (id 2) (at 140.97 53.34 0)
+    (property "Footprint" "MD-XXSM:CUI_MD-40SM" (id 2) (at 140.97 53.34 0)
       (effects (font (size 1.27 1.27)) hide)
     )
-    (property "Datasheet" "" (id 3) (at 140.97 53.34 0)
+    (property "Datasheet" "https://eu.mouser.com/datasheet/2/670/md_sm_series-1778126.pdf" (id 3) (at 140.97 53.34 0)
       (effects (font (size 1.27 1.27)) hide)
     )
     (pin "1")
-    (pin "10")
-    (pin "11")
-    (pin "12")
     (pin "2")
     (pin "3")
     (pin "4")
+    (pin "S1")
+    (pin "S2")
+    (pin "S3")
   )
   (symbol (lib_id "mdconnector:MD-30") (at 113.03 53.34 0) (unit 1)
     (in_bom yes) (on_board yes) (fields_autoplaced)
-    (property "Reference" "CN?" (id 0) (at 113.03 40.64 0))
+    (property "Reference" "CN1" (id 0) (at 113.03 40.64 0))
     (property "Value" "MD-30" (id 1) (at 113.03 43.18 0))
-    (property "Footprint" "" (id 2) (at 113.03 53.34 0)
+    (property "Footprint" "MD-XXSM:CUI_MD-30SM" (id 2) (at 113.03 53.34 0)
       (effects (font (size 1.27 1.27)) hide)
     )
-    (property "Datasheet" "" (id 3) (at 113.03 53.34 0)
+    (property "Datasheet" "https://eu.mouser.com/datasheet/2/670/md_sm_series-1778126.pdf" (id 3) (at 113.03 53.34 0)
       (effects (font (size 1.27 1.27)) hide)
     )
     (pin "1")
-    (pin "10")
-    (pin "11")
-    (pin "12")
     (pin "2")
     (pin "3")
+    (pin "S1")
+    (pin "S2")
+    (pin "S3")
   )
   (symbol (lib_id "mdconnector:MD-90") (at 167.64 85.09 0) (unit 1)
     (in_bom yes) (on_board yes) (fields_autoplaced)
-    (property "Reference" "CN?" (id 0) (at 167.64 71.12 0))
+    (property "Reference" "CN7" (id 0) (at 167.64 71.12 0))
     (property "Value" "MD-90" (id 1) (at 167.64 73.66 0))
-    (property "Footprint" "" (id 2) (at 167.64 85.09 0)
+    (property "Footprint" "MD-XXSM:CUI_MD-90SM" (id 2) (at 167.64 85.09 0)
       (effects (font (size 1.27 1.27)) hide)
     )
-    (property "Datasheet" "" (id 3) (at 167.64 85.09 0)
+    (property "Datasheet" "https://eu.mouser.com/datasheet/2/670/md_sm_series-1778126.pdf" (id 3) (at 167.64 85.09 0)
       (effects (font (size 1.27 1.27)) hide)
     )
     (pin "1")
-    (pin "10")
-    (pin "11")
-    (pin "12")
     (pin "2")
     (pin "3")
@@
     (pin "8")
     (pin "9")
+    (pin "S1")
+    (pin "S2")
+    (pin "S3")
   )
   (symbol (lib_id "mdconnector:MD-70") (at 113.03 85.09 0) (unit 1)
     (in_bom yes) (on_board yes) (fields_autoplaced)
-    (property "Reference" "CN?" (id 0) (at 113.03 71.12 0))
+    (property "Reference" "CN5" (id 0) (at 113.03 71.12 0))
     (property "Value" "MD-70" (id 1) (at 113.03 73.66 0))
-    (property "Footprint" "" (id 2) (at 113.03 85.09 0)
+    (property "Footprint" "MD-XXSM:CUI_MD-70SM" (id 2) (at 113.03 85.09 0)
       (effects (font (size 1.27 1.27)) hide)
     )
-    (property "Datasheet" "" (id 3) (at 113.03 85.09 0)
+    (property "Datasheet" "https://eu.mouser.com/datasheet/2/670/md_sm_series-1778126.pdf" (id 3) (at 113.03 85.09 0)
       (effects (font (size 1.27 1.27)) hide)
     )
     (pin "1")
-    (pin "10")
-    (pin "11")
-    (pin "12")
     (pin "2")
     (pin "3")
@@
     (pin "6")
     (pin "7")
+    (pin "S1")
+    (pin "S2")
+    (pin "S3")
   )
   (symbol (lib_id "mdconnector:MD-80") (at 140.97 85.09 0) (unit 1)
     (in_bom yes) (on_board yes) (fields_autoplaced)
-    (property "Reference" "CN?" (id 0) (at 140.6525 71.12 0))
+    (property "Reference" "CN6" (id 0) (at 140.6525 71.12 0))
     (property "Value" "MD-80" (id 1) (at 140.6525 73.66 0))
-    (property "Footprint" "" (id 2) (at 140.97 85.09 0)
+    (property "Footprint" "MD-XXSM:CUI_MD-80SM" (id 2) (at 140.97 85.09 0)
       (effects (font (size 1.27 1.27)) hide)
     )
-    (property "Datasheet" "" (id 3) (at 140.97 85.09 0)
+    (property "Datasheet" "https://eu.mouser.com/datasheet/2/670/md_sm_series-1778126.pdf" (id 3) (at 140.97 85.09 0)
       (effects (font (size 1.27 1.27)) hide)
     )
     (pin "1")
-    (pin "10")
-    (pin "11")
-    (pin "12")
     (pin "2")
     (pin "3")
@@
     (pin "7")
     (pin "8")
+    (pin "S1")
+    (pin "S2")
+    (pin "S3")
   )
   (symbol (lib_id "mdconnector:MD-60") (at 196.85 53.34 0) (unit 1)
     (in_bom yes) (on_board yes) (fields_autoplaced)
-    (property "Reference" "CN?" (id 0) (at 196.85 40.64 0))
+    (property "Reference" "CN4" (id 0) (at 196.85 40.64 0))
     (property "Value" "MD-60" (id 1) (at 196.85 43.18 0))
-    (property "Footprint" "" (id 2) (at 196.85 53.34 0)
+    (property "Footprint" "MD-XXSM:CUI_MD-60SM" (id 2) (at 196.85 53.34 0)
       (effects (font (size 1.27 1.27)) hide)
     )
-    (property "Datasheet" "" (id 3) (at 196.85 53.34 0)
+    (property "Datasheet" "https://eu.mouser.com/datasheet/2/670/md_sm_series-1778126.pdf" (id 3) (at 196.85 53.34 0)
       (effects (font (size 1.27 1.27)) hide)
     )
     (pin "1")
-    (pin "10")
-    (pin "11")
-    (pin "12")
     (pin "2")
     (pin "3")
@@
     (pin "5")
     (pin "6")
+    (pin "S1")
+    (pin "S2")
+    (pin "S3")
   )
   (sheet_instances
@@
   )
   (symbol_instances
-    (path "/0a45186a-4d19-41e8-ba59-9c616b1eb67a"
-      (reference "CN?") (unit 1) (value "MD-50") (footprint "")
+    (path "/6a5b8b35-cd7a-4a5f-9466-a7f580af64f4"
+      (reference "CN1") (unit 1) (value "MD-30") (footprint "MD-XXSM:CUI_MD-30SM")
     )
     (path "/3cc7e3e4-5b55-4a09-8e5e-4cfa4465ee7f"
-      (reference "CN?") (unit 1) (value "MD-40") (footprint "")
+      (reference "CN2") (unit 1) (value "MD-40") (footprint "MD-XXSM:CUI_MD-40SM")
     )
-    (path "/6a5b8b35-cd7a-4a5f-9466-a7f580af64f4"
-      (reference "CN?") (unit 1) (value "MD-30") (footprint "")
+    (path "/0a45186a-4d19-41e8-ba59-9c616b1eb67a"
+      (reference "CN3") (unit 1) (value "MD-50") (footprint "MD-XXSM:CUI_MD-50SM")
+    )
+    (path "/ff7f7fcf-1d3d-4a69-82ac-d2e88a7490ae"
+      (reference "CN4") (unit 1) (value "MD-60") (footprint "MD-XXSM:CUI_MD-60SM")
+    )
+    (path "/b8de7d05-4670-47c9-bd98-21786752c184"
+      (reference "CN5") (unit 1) (value "MD-70") (footprint "MD-XXSM:CUI_MD-70SM")
+    )
+    (path "/e7849295-e96a-4fb4-9b79-de43230a78e1"
+      (reference "CN6") (unit 1) (value "MD-80") (footprint "MD-XXSM:CUI_MD-80SM")
     )
     (path "/8154a1c7-b289-4e70-8e4a-846b3baf74ef"
-      (reference "CN?") (unit 1) (value "MD-90") (footprint "")
-    )
-    (path "/b8de7d05-4670-47c9-bd98-21786752c184"
-      (reference "CN?") (unit 1) (value "MD-70") (footprint "")
-    )
-    (path "/e7849295-e96a-4fb4-9b79-de43230a78e1"
-      (reference "CN?") (unit 1) (value "MD-80") (footprint "")
-    )
-    (path "/ff7f7fcf-1d3d-4a69-82ac-d2e88a7490ae"
-      (reference "CN?") (unit 1) (value "MD-60") (footprint "")
+      (reference "CN7") (unit 1) (value "MD-90") (footprint "MD-XXSM:CUI_MD-90SM")
     )
   )
