File: stlinkv2/stlinkv2.kicad_pcb (KiCad board)
At the start: 2 copper layers, 80 x 45.7 mm, 82 parts, among them J1 STLSWD, J2 JTAG, J3 SWD, J4 CLONE, J5 DBG_UART, J6 STM8, J7 POWER, J8 POWER, J9 USB_B_Mini, SW1 EXRERNAL POWER, U1 STM32F103CBTx, U2 74LVCC3245, U3 LD3985M33R_SOT23, U4 USBLC6-2, U5 ADUM3160, Y1 8MHz

Commit message: update schematic and pcb
Parts:
- added H1: MH, MountingHole:MountingHole_2.2mm_M2_ISO14580_Pad, F.Cu at (27.9, 27.9)
- added H2: MH, MountingHole:MountingHole_2.2mm_M2_ISO14580_Pad, F.Cu at (102.9, 27.9)
- added H3: MH, MountingHole:MountingHole_2.2mm_M2_ISO14580_Pad, F.Cu at (102.9, 68.6)
- added H4: MH, MountingHole:MountingHole_2.2mm_M2_ISO14580_Pad, F.Cu at (27.9, 68.6)
- moved C10 35.6 mm to (43.2, 33.0)
- moved R8 9.25 mm to (57.1, 30.5), turned to 180 degrees
- moved R6 7.73 mm to (66.0, 39.4), turned to 180 degrees
- moved R11 6.89 mm to (93.2, 30.5), turned to 90 degrees
- moved C5 6.63 mm to (71.1, 66.0)
- moved J5 5.25 mm to (85.1, 30.5)
- moved R21 5.08 mm to (81.3, 38.1)
- moved JP2 5.08 mm to (57.1, 27.9)
- moved D5 3.84 mm to (48.3, 27.9)
- moved D6 3.84 mm to (48.3, 30.5), turned to 0 degrees
- moved R36 3.84 mm to (52.1, 27.9)
- moved R37 3.84 mm to (52.1, 30.5)
- moved J6 3.81 mm to (100.3, 35.6)
- moved J3 3.81 mm to (96.5, 30.5)
- moved SW1 3.48 mm to (36.8, 28.6)
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Connections:
- D1 pad 1: SWMA -> RST
- D1 pad 6: RST -> SWMA
- JP1 pad 1: BOOT0 -> +3V3
- JP1 pad 2: +3V3 -> BOOT0
- U2 pad 16: DBG_TX -> T_JTDI
- U2 pad 18: T_JTDI -> DBG_TX
- U2 pad 6: T_JTDO -> DBG_TXB
- U2 pad 8: DBG_TXB -> T_JTDO
Routing:
- net RST: track 4.23 -> 54.4 mm, vias 0 -> 3
- net V_BUF: track 9.15 -> 57.0 mm, vias 0 -> 3
- net SWMA: track 15.5 -> 52.1 mm, vias 2 -> 6
- net RSTB: track 0.00 -> 25.3 mm, vias 0 -> 2
- net T_JTMS: track 23.5 -> 47.5 mm, vias 2 -> 5
- net BOOT1: track 2.17 -> 25.3 mm, vias 0 -> 2
- net T_JTDI: track 18.9 -> 41.4 mm, vias 2 -> 6
- net T_SWO: track 0.00 -> 21.2 mm, vias 0 -> 2
- net T_SWDIO_IN: track 0.00 -> 16.8 mm, vias 0 -> 2
- net T_JTDO: track 5.02 -> 20.9 mm, vias 0 -> 2
- net DBG_TX: track 0.00 -> 13.6 mm, vias 0 -> 1
- net T_JRST: track 3.43 -> 15.5 mm
- net SWM_IN: track 13.3 -> 24.9 mm, vias 2 -> 3
- net +3V3: track 42.4 -> 53.5 mm, vias 9 -> 13
- net DBG_TXB: track 0.00 -> 8.79 mm, vias 0 -> 2
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Other:
- outline, holes or cut-outs redrawn

Commit message: update schema and pcb
Parts:
- turned D3 to 180 degrees
Routing:
- net USB5V: track 28.1 -> 30.7 mm
- net Net-(J6-Pad2): track 19.2 -> 21.7 mm
- net STM_JTMS: track 18.2 -> 20.5 mm
- net RST: track 54.4 -> 52.3 mm
- net V_TGT: track 33.6 -> 35.4 mm
- net STM_JTCK: track 26.8 -> 25.5 mm
- net Net-(C12-Pad1): track 17.4 -> 16.4 mm
- net Net-(J6-Pad4): track 22.7 -> 21.7 mm
- net LED: track 27.1 -> 28.0 mm
- net +3V3: track 53.5 -> 52.7 mm

Commit message: some update
Parts:
- moved R36 16.1 mm to (36.8, 33.0)
- moved D5 16.1 mm to (33.0, 33.0)
- moved R37 15.2 mm to (36.8, 30.5)
- moved D6 15.2 mm to (33.0, 30.5)
- moved C10 8.52 mm to (50.8, 29.2), turned to 90 degrees
- moved SW1 7.65 mm to (44.5, 29.2)
Connections:
- J1 pad 5: unconnected-(J1-Pad5) -> T_SWO
- J1 pad 6: unconnected-(J1-Pad6) -> LED
- U2 pad 2: GND -> BOOT0
- U2 pad 22: GND -> BOOT0
Routing:
- net BOOT0: track 25.4 -> 59.4 mm, vias 2 -> 5
- net LED: track 28.0 -> 52.7 mm, vias 2 -> 3
- net T_SWO: track 21.0 -> 28.8 mm
- net V_BUF: track 57.0 -> 50.8 mm
- net +3V3: track 52.7 -> 53.8 mm
- net T_SWDIO_IN: track 16.9 -> 16.1 mm
Other:
- outline, holes or cut-outs redrawn
- board text added: "BOOT_RX"
- board text added: "BOOT_TX"

Commit message: update schematic and pcb
Parts:
- turned JP2 to 0 degrees
Connections:
- JP2 pad 1: BOOT1 -> +3V3
- JP2 pad 2: +3V3 -> BOOT1
Changed lines of the file:
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@@
   )
   (footprint "Jumper:SolderJumper-2_P1.3mm_Open_TrianglePad1.0x1.5mm" (layer "F.Cu")
-    (at 57.15 27.94 180)
+    (at 57.15 27.94)
     (descr "SMD Solder Jumper, 1x1.5mm Triangular Pads, 0.3mm gap, open")
     (tags "solder jumper open")
@@
     (property "Sheetname" "")
     (attr exclude_from_pos_files)
-    (fp_text reference "JP2" (at 2.286 0 90) (layer "F.SilkS")
+    (fp_text reference "JP2" (at -2.032 0 90) (layer "F.SilkS")
       (effects (font (size 0.8 0.8) (thickness 0.15)))
     )
@@
       (effects (font (size 0.8 0.8) (thickness 0.15)))
     )
-    (fp_text user "${VALUE}" (at 0 0 180 unlocked) (layer "Dwgs.User") hide
+    (fp_text user "${VALUE}" (at 0 0 unlocked) (layer "Dwgs.User") hide
       (effects (font (size 0.8 0.8) (thickness 0.15)))
     )
@@
     (fp_line (start -1.65 -1.25) (end -1.65 1.25) (layer "F.CrtYd") (width 0.05))
     (fp_line (start 1.65 1.25) (end 1.65 -1.25) (layer "F.CrtYd") (width 0.05))
-    (pad "1" smd custom (at -0.725 0 180) (size 0.3 0.3) (layers "F.Cu" "F.Mask")
-      (net 47 "BOOT1") (pinfunction "A") (pintype "passive") (zone_connect 2)
+    (pad "1" smd custom (at -0.725 0) (size 0.3 0.3) (layers "F.Cu" "F.Mask")
+      (net 5 "+3V3") (pinfunction "A") (pintype "passive") (zone_connect 2)
       (options (clearance outline) (anchor rect))
       (primitives
@@
           ) (width 0) (fill yes))
       ))
-    (pad "2" smd custom (at 0.725 0 180) (size 0.3 0.3) (layers "F.Cu" "F.Mask")
-      (net 5 "+3V3") (pinfunction "B") (pintype "passive") (zone_connect 2)
+    (pad "2" smd custom (at 0.725 0) (size 0.3 0.3) (layers "F.Cu" "F.Mask")
+      (net 47 "BOOT1") (pinfunction "B") (pintype "passive") (zone_connect 2)
       (options (clearance outline) (anchor rect))
       (primitives
@@
   )
   (gr_line (start 62.457064 58.166) (end 63.754 58.42) (layer "F.SilkS") (width 0.15))
+  (gr_circle locked (center 73.9775 51.1175) (end 74.2315 51.1175) (layer "F.SilkS") (width 0.15) (fill solid))
   (gr_arc locked (start 102.87 25.4) (mid 104.666051 26.143949) (end 105.41 27.94) (layer "Dwgs.User") (width 0.5))
   (gr_line locked (start 102.87 25.4) (end 27.94 25.4) (layer "Dwgs.User") (width 0.5))
@@
   (gr_arc locked (start 105.41 68.58) (mid 104.666051 70.376051) (end 102.87 71.12) (layer "Dwgs.User") (width 0.5))
   (gr_line locked (start 105.41 68.58) (end 105.41 27.94) (layer "Dwgs.User") (width 0.5))
-  (gr_line locked (start 25.4 48.26) (end 105.41 48.26) (layer "Dwgs.User") (width 0.01))
   (gr_arc locked (start 27.94 71.12) (mid 26.143949 70.376051) (end 25.4 68.58) (layer "Dwgs.User") (width 0.5))
+  (gr_line locked (start 25.4 48.26) (end 105.41 48.26) (layer "Cmts.User") (width 0.01))
   (gr_line locked (start 46.5455 34.925) (end 50.9905 34.925) (layer "Edge.Cuts") (width 0.1))
   (gr_line locked (start 33.8455 55.245) (end 38.2905 55.245) (layer "Edge.Cuts") (width 0.1))
@@
     (effects (font (size 0.8 0.8) (thickness 0.15)))
   )
-  (dimension (type orthogonal) (layer "Dwgs.User")
+  (dimension (type orthogonal) (layer "Cmts.User")
     (pts (xy 27.94 68.58) (xy 102.87 68.58))
     (height 7.62)
     (orientation 0)
-    (gr_text "74,9300 mm" (at 65.405 75.25) (layer "Dwgs.User")
+    (gr_text "74,9300 mm" (at 65.405 75.25) (layer "Cmts.User")
       (effects (font (size 0.8 0.8) (thickness 0.15)))
     )
@@
     (style (thickness 0.15) (arrow_length 1.27) (text_position_mode 0) (extension_height 0.58642) (extension_offset 0.5) keep_text_aligned)
   )
-  (dimension (type orthogonal) (layer "Dwgs.User")
+  (dimension (type orthogonal) (layer "Cmts.User")
     (pts (xy 25.4 68.58) (xy 105.41 68.58))
     (height 12.7)
     (orientation 0)
-    (gr_text "80,0100 mm" (at 65.405 80.13) (layer "Dwgs.User")
+    (gr_text "80,0100 mm" (at 65.405 80.13) (layer "Cmts.User")
       (effects (font (size 1 1) (thickness 0.15)))
     )
@@
     (style (thickness 0.1) (arrow_length 1.27) (text_position_mode 0) (extension_height 0.58642) (extension_offset 0.5) keep_text_aligned)
   )
-  (dimension (type orthogonal) (layer "Dwgs.User")
+  (dimension (type orthogonal) (layer "Cmts.User")
     (pts (xy 27.94 71.12) (xy 27.94 25.4))
     (height -12.7)
     (orientation 1)
-    (gr_text "45,72 mm" (at 14.29 48.26 90) (layer "Dwgs.User")
+    (gr_text "45,72 mm" (at 14.29 48.26 90) (layer "Cmts.User")
       (effects (font (size 0.8 0.8) (thickness 0.15)))
     )
@@
     (style (thickness 0.15) (arrow_length 1.27) (text_position_mode 0) (extension_height 0.58642) (extension_offset 0.5) keep_text_aligned)
   )
-  (dimension (type orthogonal) (layer "Dwgs.User")
+  (dimension (type orthogonal) (layer "Cmts.User")
     (pts (xy 27.94 27.94) (xy 27.94 68.58))
     (height -7.62)
     (orientation 1)
-    (gr_text "40,64 mm" (at 19.05 48.26 90) (layer "Dwgs.User")
+    (gr_text "40,64 mm" (at 19.05 48.26 90) (layer "Cmts.User")
       (effects (font (size 1 1) (thickness 0.15)))
     )
@@
   (segment (start 60.235 64.995) (end 60.01 64.77) (width 0.5) (layer "F.Cu") (net 5))
   (segment (start 66.99 36.83) (end 69.4925 36.83) (width 0.5) (layer "F.Cu") (net 5))
-  (segment (start 56.425 27.94) (end 54.61 27.94) (width 0.5) (layer "F.Cu") (net 5))
   (segment (start 74.815685 45.74) (end 74.0125 45.74) (width 0.25) (layer "F.Cu") (net 5))
   (segment (start 65.305 52.39) (end 65.6875 52.0075) (width 0.25) (layer "F.Cu") (net 5))
   (segment (start 60.96 60.96) (end 61.28 61.28) (width 0.5) (layer "F.Cu") (net 5))
+  (segment (start 56.425 27.94) (end 54.61 27.94) (width 0.5) (layer "F.Cu") (net 5))
   (segment (start 64.77 41.275) (end 65.5475 41.275) (width 0.25) (layer "F.Cu") (net 5))
   (segment (start 61.28 61.28) (end 61.28 62.23) (width 0.5) (layer "F.Cu") (net 5))
@@
   (via (at 71.12 68.58) (size 0.8) (drill 0.4) (layers "F.Cu" "B.Cu") (net 5))
   (via (at 75.565 46.2595) (size 0.8) (drill 0.4) (layers "F.Cu" "B.Cu") (free) (net 5))
-  (via (at 54.61 27.94) (size 0.8) (drill 0.4) (layers "F.Cu" "B.Cu") (net 5))
   (via (at 65.6875 51.1525) (size 0.8) (drill 0.4) (layers "F.Cu" "B.Cu") (net 5))
   (via (at 57.785 67.31) (size 0.8) (drill 0.4) (layers "F.Cu" "B.Cu") (net 5))
+  (via (at 54.61 27.94) (size 0.8) (drill 0.4) (layers "F.Cu" "B.Cu") (net 5))
   (via (at 64.77 41.275) (size 0.8) (drill 0.4) (layers "F.Cu" "B.Cu") (net 5))
   (via (at 67.945 35.56) (size 0.8) (drill 0.4) (layers "F.Cu" "B.Cu") (net 5))
@@
   (via (at 68.707 28.575) (size 0.8) (drill 0.4) (layers "F.Cu" "B.Cu") (net 7))
   (via (at 82.3205 29.25507) (size 0.8) (drill 0.4) (layers "F.Cu" "B.Cu") (net 7))
+  (segment (start 54.2925 31.115) (end 52.07 31.115) (width 0.25) (layer "B.Cu") (net 7))
   (segment (start 82.3205 29.25507) (end 80.802635 27.737205) (width 0.25) (layer "B.Cu") (net 7))
-  (segment (start 52.07 31.115) (end 54.2925 31.115) (width 0.25) (layer "B.Cu") (net 7))
-  (segment (start 56.8325 28.575) (end 68.707 28.575) (width 0.25) (layer "B.Cu") (net 7))
+  (segment (start 68.707 28.575) (end 60.96 28.575) (width 0.25) (layer "B.Cu") (net 7))
+  (segment (start 55.08625 30.32125) (end 54.2925 31.115) (width 0.25) (layer "B.Cu") (net 7))
+  (segment (start 59.21375 30.32125) (end 55.08625 30.32125) (width 0.25) (layer "B.Cu") (net 7))
   (segment (start 69.544795 27.737205) (end 68.707 28.575) (width 0.25) (layer "B.Cu") (net 7))
+  (segment (start 60.96 28.575) (end 59.21375 30.32125) (width 0.25) (layer "B.Cu") (net 7))
   (segment (start 80.802635 27.737205) (end 69.544795 27.737205) (width 0.25) (layer "B.Cu") (net 7))
-  (segment (start 54.2925 31.115) (end 56.8325 28.575) (width 0.25) (layer "B.Cu") (net 7))
   (segment (start 55.65 42.14) (end 55.65 53.975) (width 0.5) (layer "F.Cu") (net 8))
   (segment (start 55.65 53.975) (end 55.65 56.11) (width 0.5) (layer "F.Cu") (net 8))
@@
   (segment (start 65.695 40.449524) (end 65.695 42.320342) (width 0.25) (layer "B.Cu") (net 46))
   (segment (start 68.384792 37.561716) (end 66.33 39.616508) (width 0.25) (layer "B.Cu") (net 46))
-  (segment (start 57.875 27.94) (end 58.0625 28.1275) (width 0.25) (layer "F.Cu") (net 47))
   (segment (start 58.0625 28.1275) (end 58.0625 30.48) (width 0.25) (layer "F.Cu") (net 47))
   (segment (start 68.58 40.64) (end 69.1 41.16) (width 0.25) (layer "F.Cu") (net 47))
   (segment (start 69.1 41.16) (end 69.1 42.8275) (width 0.25) (layer "F.Cu") (net 47))
   (segment (start 66.04 40.311586) (end 66.368414 40.64) (width 0.25) (layer "F.Cu") (net 47))
+  (segment (start 57.875 27.94) (end 58.0625 28.1275) (width 0.25) (layer "F.Cu") (net 47))
   (segment (start 58.42 30.8375) (end 58.0625 30.48) (width 0.25) (layer "F.Cu") (net 47))
   (segment (start 66.04 34.925) (end 66.04 40.311586) (width 0.25) (layer "F.Cu") (net 47))

Commit message: some update
Routing:
- net V_TGT: track 35.4 -> 33.4 mm
Changed lines of the file:
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@@
   (segment (start 62.68 47.819293) (end 62.68 35.13) (width 0.25) (layer "B.Cu") (net 34))
   (segment (start 84.789695 36.285) (end 83.045 34.540305) (width 0.25) (layer "F.Cu") (net 35))
-  (segment (start 86.9945 36.285) (end 84.789695 36.285) (width 0.25) (layer "F.Cu") (net 35))
-  (segment (start 87.63 35.6495) (end 86.9945 36.285) (width 0.25) (layer "F.Cu") (net 35))
-  (segment (start 87.63 38.1) (end 90.17 38.1) (width 0.25) (layer "F.Cu") (net 35))
   (segment (start 83.045 28.7925) (end 82.1925 27.94) (width 0.25) (layer "F.Cu") (net 35))
   (segment (start 83.045 34.540305) (end 83.045 28.7925) (width 0.25) (layer "F.Cu") (net 35))
-  (via (at 87.63 35.6495) (size 0.8) (drill 0.4) (layers "F.Cu" "B.Cu") (net 35))
+  (segment (start 87.63 38.1) (end 90.17 38.1) (width 0.25) (layer "F.Cu") (net 35))
+  (segment (start 86.36 36.83) (end 85.815 36.285) (width 0.25) (layer "F.Cu") (net 35))
+  (segment (start 85.815 36.285) (end 84.789695 36.285) (width 0.25) (layer "F.Cu") (net 35))
+  (via (at 86.36 36.83) (size 0.8) (drill 0.4) (layers "F.Cu" "B.Cu") (net 35))
   (segment (start 96.52 30.48) (end 100.33 34.29) (width 0.25) (layer "B.Cu") (net 35))
   (segment (start 93.98 38.1) (end 95.25 36.83) (width 0.25) (layer "B.Cu") (net 35))
@@
   (segment (start 90.17 38.1) (end 93.98 38.1) (width 0.25) (layer "B.Cu") (net 35))
   (segment (start 100.33 34.29) (end 100.33 35.57) (width 0.25) (layer "B.Cu") (net 35))
-  (segment (start 87.63 35.6495) (end 87.63 38.1) (width 0.25) (layer "B.Cu") (net 35))
+  (segment (start 86.36 36.83) (end 87.63 38.1) (width 0.25) (layer "B.Cu") (net 35))
   (segment (start 83.82 38.1) (end 82.1925 38.1) (width 0.25) (layer "F.Cu") (net 36))
   (via (at 83.82 38.1) (size 0.8) (drill 0.4) (layers "F.Cu" "B.Cu") (net 36))

Commit message: update schematic and pcb
Parts:
- C8: value 20pF -> 100nF
- moved C12 1.27 mm to (57.1, 57.1), turned to 180 degrees
Connections:
- QC1 pad 3: USB5V -> +3V3
Routing:
- net USB5V: track 30.7 -> 32.6 mm, vias 0 -> 1
- net +3V3: track 53.8 -> 54.6 mm, vias 13 -> 16
- net V_BUF: track 50.8 -> 50.0 mm
- net BOOT1: track 24.9 -> 25.6 mm
- net SWMA: track 52.0 -> 52.6 mm
- net LED: track 52.7 -> 52.2 mm

Commit message: fix schematic and pcb
Parts:
- added D5: BAT60JFILM, Diode_SMD:D_SOD-323_HandSoldering, F.Cu at (52.1, 63.5)
- moved R1 16.9 mm to (81.3, 58.4)
- moved R20 2.54 mm to (81.3, 55.9)
- moved R23 2.54 mm to (81.3, 53.3)
- moved C13 1.80 mm to (52.1, 66.0)
- moved R7 1.80 mm to (66.0, 66.0), turned to -90 degrees
- moved R5 1.27 mm to (69.8, 36.8), turned to 0 degrees
- moved C16 1.27 mm to (62.2, 64.8)
- moved JP1 1.27 mm to (62.2, 67.3)
- turned C12 to 0 degrees
- turned C14 to 180 degrees
- turned U3 to 0 degrees
- renumbered D5 to D6, D6 to D7
Connections:
- net RST renamed SWIM_RST
- net RSTB renamed SWIM_RST_IN
- net SWM_IN renamed SWIM_IN
- D1 pad 4: T_JTDO -> T_JRST
- D1 pad 5: T_JRST -> T_JTDO_SWO
- J1 pad 2: GND -> STM_JTCK
- J1 pad 3: STM_JTCK -> GND
- J1 pad 4: +3V3 -> PRG_5V
- J2 pad 13: T_JTDI_ -> T_JTDO_SWO_
- J2 pad 5: T_JTDO_ -> T_JTDI_
- J3 pad 6: T_JTDI_ -> T_JTDO_SWO_
- R1 pad 2: T_JTDO_ -> T_JTDI_
- R16 pad 1: T_JTDO -> T_JTDO_SWO
- R16 pad 2: T_JTDO_ -> T_JTDO_SWO_
- U2 pad 16: T_JTDI -> DBG_TX
- U2 pad 17: T_JTDI -> T_JTDO_SWO
- U2 pad 18: DBG_TX -> T_JTDO_SWO
- U2 pad 6: DBG_TXB -> T_SWO
- U2 pad 7: T_SWO -> T_JTDO
- U2 pad 8: T_JTDO -> DBG_TXB
Routing:
- net PRG_5V: track 0.00 -> 47.6 mm, vias 0 -> 1
- net T_JTDO_SWO_: track 0.00 -> 28.7 mm, vias 0 -> 2
- net T_JTDO_SWO: track 0.00 -> 22.0 mm, vias 0 -> 2
- net T_JTDI: track 41.7 -> 21.0 mm, vias 6 -> 2
- net T_JTDO_: track 11.6 -> 0.00 mm, vias 2 -> 0
- net T_JTDO: track 20.4 -> 10.3 mm
- net SWIM_RST: track 52.2 -> 43.3 mm
- net BOOT1: track 25.6 -> 31.9 mm
- net LED: track 52.2 -> 56.5 mm
- net AIN1: track 14.4 -> 18.4 mm
- net STM_JTCK: track 25.5 -> 29.4 mm
- net T_NRST_: track 33.0 -> 36.4 mm
- net SWMA: track 52.6 -> 49.3 mm
- net EXTERN_5V: track 73.5 -> 76.8 mm
- net T_NRST: track 23.8 -> 21.3 mm
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
Commit message: update schema and pcb
Parts:
- added JP3: SolderJumper_3_Open, Jumper:SolderJumper-3_P1.3mm_Open_RoundedPad1.0x1.5mm, F.Cu at (57.1, 55.2)
- added R35: 1.5k, Resistor_SMD:R_0805_2012Metric, F.Cu at (57.1, 52.7)
- moved R24 5.08 mm to (81.3, 58.4)
- moved C12 4.45 mm to (57.1, 61.6)
- moved QC1 4.45 mm to (57.1, 58.4)
- moved U3 3.81 mm to (57.1, 64.8)
- moved C14 3.19 mm to (57.1, 68.0)
- moved D5 2.54 mm to (52.0, 61.0)
- moved D4 2.54 mm to (52.1, 63.5)
- moved R1 2.54 mm to (81.3, 55.9)
- moved R22 2.54 mm to (81.3, 53.3)
- renumbered C18 to C17, C19 to C18, C17 to C19, R25 to R10, R9 to R11, R10 to R12, R11 to R13, R12 to R14, R13 to R15, R14 to R16, R15 to R17, R16 to R18, R17 to R19, R18 to R20, R19 to R21, R20 to R22, R21 to R23, R23 to R24, R24 to R25, R33 to R31, R34 to R32, R32 to R33, R31 to R34, R35 to R36, R36 to R37, R37 to R38, R22 to R6, R6 to R7, R7 to R8, R8 to R9
Connections:
- net /DI+ renamed Net-(R26-Pad2)
- net /DI- renamed Net-(R29-Pad2)
- net USB_D+ renamed DD+
- net USB_D- renamed DD-
- C19 pad 1: Net-(C17-Pad1) -> +3V3
- U5 pad 12: Net-(C17-Pad1) -> Net-(U5-Pad12)
- U5 pad 13: Net-(C17-Pad1) -> +3V3
- U5 pad 14: Net-(C17-Pad1) -> +3V3
- U5 pad 16: USB5V -> +3V3
Routing:
- net +3V3: track 53.1 -> 65.5 mm, vias 15 -> 17
- net Net-(U5-Pad12): track 0.00 -> 10.8 mm
- net Net-(C17-Pad1): track 9.16 -> 0.00 mm
- net Net-(R36-Pad1): track 3.06 -> 9.39 mm
- net T_NRST: track 21.3 -> 26.4 mm
- net EXTERN_5V: track 76.8 -> 72.0 mm
- net T_JTDI_: track 35.3 -> 31.1 mm
- net PRG_5V: track 47.6 -> 44.0 mm
- net USB5V: track 33.3 -> 29.8 mm
- net PINCTRL: track 0.00 -> 2.70 mm
- net T_JTDI: track 21.0 -> 18.7 mm
- net T_JTMS_: track 44.2 -> 42.8 mm, vias 2 -> 3
- net T_JTCK_: track 50.5 -> 49.3 mm
- net LED: track 56.5 -> 55.4 mm, vias 3 -> 2
- net Net-(C12-Pad1): track 17.0 -> 16.2 mm
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