File: stlinkv2/stlinkv2.kicad_sch (KiCad schematic)
At the start: 82 parts, among them J1 STLSWD, J2 JTAG, J3 SWD, J4 CLONE, J5 DBG_UART, J6 STM8, J7 POWER, J8 POWER, J9 USB_B_Mini, SW1 EXRERNAL POWER, U1 STM32F103CBTx, U2 74LVCC3245, U3 LD3985M33R_SOT23, U4 USBLC6-2, U5 ADUM3160, Y1 8MHz

Commit message: update schematic and pcb
Parts:
- added H1, H2, H3, H4: MH, MountingHole:MountingHole_2.2mm_M2_ISO14580_Pad, symbol Mechanical:MountingHole_Pad
Connections:
- net +3V3: now also JP1.1 (A); no longer JP1.2 (B)
- net BOOT0: now also JP1.2 (B); no longer JP1.1 (A)
- net DBG_TX: now also U2.18 (B3); no longer U2.16 (B5)
- net DBG_TXB: now also U2.6 (A3); no longer U2.8 (A5)
- net GND: now also H1.1, H2.1, H3.1, H4.1
- net RST: now also D1.1 (K); no longer D1.6 (K)
- net SWMA: now also D1.6 (K); no longer D1.1 (K)
- net T_JTDI: now also U2.16 (B5); no longer U2.18 (B3)
- net T_JTDO: now also U2.8 (A5); no longer U2.6 (A3)
Other:
- moved on the sheet: JP1

Commit message: update schema and pcb
Changed lines of the file:
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@@
     )
   )
-  (global_label "T_SWO" (shape input) (at 132.08 86.36 180) (fields_autoplaced)
-    (effects (font (size 1.27 1.27)) (justify right))
-    (property "Intersheet References" "${INTERSHEET_REFS}" (id 0) (at 123.7402 86.2806 0)
-      (effects (font (size 1.27 1.27)) (justify right) hide)
+  (global_label "T_SWO" (shape input) (at 132.08 86.36 0) (fields_autoplaced)
+    (effects (font (size 1.27 1.27)) (justify left))
+    (property "Intersheet References" "${INTERSHEET_REFS}" (id 0) (at 140.4198 86.2806 0)
+      (effects (font (size 1.27 1.27)) (justify left) hide)
     )
   )

Commit message: some update
Connections:
- net BOOT0: now also U2.2 (A/~{B}), U2.22 (~{OE})
- net GND: no longer U2.2 (A/~{B}), U2.22 (~{OE})
- net LED: now also J1.6 (Pin_6)
- net T_SWO: now also J1.5 (Pin_5)
- no-connect marks 16 -> 14
Other:
- note added: "BOOT_RX"
- note added: "BOOT_TX"
Changed lines of the file:
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@@
   (junction (at 160.02 21.59) (diameter 0) (color 0 0 0 0)
   )
+  (junction (at 190.5 77.47) (diameter 0) (color 0 0 0 0)
+  )
   (junction (at 59.69 186.69) (diameter 0) (color 0 0 0 0)
   )
@@
   (junction (at 229.87 140.97) (diameter 0) (color 0 0 0 0)
   )
-  (junction (at 190.5 80.01) (diameter 0) (color 0 0 0 0)
-  )
   (junction (at 59.69 138.43) (diameter 0) (color 0 0 0 0)
   )
@@
   (no_connect (at 96.52 99.06))
   (no_connect (at 260.35 49.53))
-  (no_connect (at 85.09 25.4))
-  (no_connect (at 72.39 25.4))
   (no_connect (at 129.54 71.12))
   (no_connect (at 96.52 71.12))
@@
     (stroke (width 0) (type default) (color 0 0 0 0))
   )
-  (wire (pts (xy 190.5 80.01) (xy 190.5 82.55))
-    (stroke (width 0) (type default) (color 0 0 0 0))
-  )
   (wire (pts (xy 58.42 50.8) (xy 58.42 53.34))
     (stroke (width 0) (type default) (color 0 0 0 0))
@@
     (stroke (width 0) (type default) (color 0 0 0 0))
   )
+  (wire (pts (xy 187.96 77.47) (xy 190.5 77.47))
+    (stroke (width 0) (type default) (color 0 0 0 0))
+  )
   (wire (pts (xy 247.65 19.05) (xy 252.73 19.05))
     (stroke (width 0) (type default) (color 0 0 0 0))
@@
     (stroke (width 0) (type default) (color 0 0 0 0))
   )
+  (wire (pts (xy 85.09 25.4) (xy 87.63 25.4))
+    (stroke (width 0) (type default) (color 0 0 0 0))
+  )
   (wire (pts (xy 139.7 191.77) (xy 137.16 191.77))
     (stroke (width 0) (type default) (color 0 0 0 0))
@@
     (stroke (width 0) (type default) (color 0 0 0 0))
   )
+  (wire (pts (xy 69.85 25.4) (xy 72.39 25.4))
+    (stroke (width 0) (type default) (color 0 0 0 0))
+  )
   (wire (pts (xy 72.39 156.21) (xy 72.39 157.48))
     (stroke (width 0) (type default) (color 0 0 0 0))
@@
     (stroke (width 0) (type default) (color 0 0 0 0))
   )
+  (text "BOOT_RX" (at 93.98 26.67 0)
+    (effects (font (size 1.27 1.27)) (justify left bottom))
+  )
   (text "ISOLATED" (at 13.97 124.46 0)
     (effects (font (size 1.27 1.27) (thickness 0.254) bold) (justify left bottom))
   )
+  (text "BOOT_TX" (at 52.07 26.67 0)
+    (effects (font (size 1.27 1.27)) (justify left bottom))
+  )
   (label "D+" (at 29.21 153.67 0)
     (effects (font (size 1.27 1.27)) (justify left bottom))
@@
     )
   )
+  (global_label "LED" (shape output) (at 87.63 25.4 0) (fields_autoplaced)
+    (effects (font (size 1.27 1.27)) (justify left))
+    (property "Intersheet References" "${INTERSHEET_REFS}" (id 0) (at 93.4902 25.3206 0)
+      (effects (font (size 1.27 1.27)) (justify left) hide)
+    )
+  )
   (global_label "T_JTMS_" (shape bidirectional) (at 260.35 71.12 180) (fields_autoplaced)
     (effects (font (size 1.27 1.27)) (justify right))
@@
     )
   )
+  (global_label "T_SWO" (shape input) (at 69.85 25.4 180) (fields_autoplaced)
+    (effects (font (size 1.27 1.27)) (justify right))
+    (property "Intersheet References" "${INTERSHEET_REFS}" (id 0) (at 61.5102 25.3206 0)
+      (effects (font (size 1.27 1.27)) (justify right) hide)
+    )
+  )
   (global_label "T_JRST_" (shape output) (at 204.47 109.22 0) (fields_autoplaced)
     (effects (font (size 1.27 1.27)) (justify left))
@@
     )
   )
+  (global_label "BOOT0" (shape passive) (at 187.96 77.47 180) (fields_autoplaced)
+    (effects (font (size 1.27 1.27)) (justify right))
+    (property "Intersheet References" "${INTERSHEET_REFS}" (id 0) (at 179.4388 77.3906 0)
+      (effects (font (size 1.27 1.27)) (justify right) hide)
+    )
+  )
   (global_label "T_SWDIO_IN" (shape input) (at 93.98 91.44 180) (fields_autoplaced)
     (effects (font (size 1.27 1.27)) (justify right))
@@
     (pin "2")
   )
-  (symbol (lib_id "power:GND") (at 190.5 82.55 0) (unit 1)
-    (in_bom yes) (on_board yes)
-    (property "Reference" "#PWR024" (id 0) (at 190.5 88.9 0)
-      (effects (font (size 1.27 1.27)) hide)
-    )
-    (property "Value" "GND" (id 1) (at 190.5 86.36 0))
-    (property "Footprint" "" (id 2) (at 190.5 82.55 0)
-      (effects (font (size 1.27 1.27)) hide)
-    )
-    (property "Datasheet" "" (id 3) (at 190.5 82.55 0)
-      (effects (font (size 1.27 1.27)) hide)
-    )
-    (pin "1")
-  )
   (symbol (lib_id "power:GND") (at 95.25 189.23 0) (unit 1)
     (in_bom yes) (on_board yes)
@@
       (reference "#PWR023") (unit 1) (value "GND") (footprint "")
     )
-    (path "/de4af085-19f1-4fe4-a87d-f4c124501151"
-      (reference "#PWR024") (unit 1) (value "GND") (footprint "")
-    )
     (path "/2b42be67-bf3b-4be0-80b1-3043ccbfa647"

Commit message: update schematic and pcb
Connections:
- net +3V3: now also JP2.1 (A); no longer JP2.2 (B)
- net BOOT1: now also JP2.2 (B); no longer JP2.1 (A)
Other:
- moved on the sheet: JP2
Changed lines of the file:
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@@
     (pin "1")
   )
-  (symbol (lib_id "Jumper:SolderJumper_2_Open") (at 58.42 57.15 90) (unit 1)
+  (symbol (lib_id "Jumper:SolderJumper_2_Open") (at 58.42 57.15 270) (unit 1)
     (in_bom yes) (on_board yes)
     (property "Reference" "JP2" (id 0) (at 60.96 54.61 90))

Commit message: upddate capacitor values
Parts:
- C8: value 20pF -> 100nF
Changed lines of the file:
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@@
     (in_bom yes) (on_board yes)
     (property "Reference" "C8" (id 0) (at 21.59 67.31 0))
-    (property "Value" "20pF" (id 1) (at 22.86 72.39 0))
+    (property "Value" "100nF" (id 1) (at 22.86 72.39 0))
     (property "Footprint" "Capacitor_SMD:C_0805_2012Metric" (id 2) (at 20.0152 73.66 0)
       (effects (font (size 1.27 1.27)) hide)
@@
     )
     (path "/961cf994-e7e5-46b8-b479-3b05b33fef15"
-      (reference "C8") (unit 1) (value "20pF") (footprint "Capacitor_SMD:C_0805_2012Metric")
+      (reference "C8") (unit 1) (value "100nF") (footprint "Capacitor_SMD:C_0805_2012Metric")
     )
     (path "/ac5403d6-ed5e-478b-ab19-82f141eba405"

Commit message: update schematic and pcb
Connections:
- net +3V3: now also QC1.3 (C)
- net USB5V: no longer QC1.3 (C)
Changed lines of the file:
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@@
     (stroke (width 0) (type default) (color 0 0 0 0))
   )
-  (wire (pts (xy 161.29 185.42) (xy 161.29 191.77))
-    (stroke (width 0) (type default) (color 0 0 0 0))
-  )
   (wire (pts (xy 85.09 20.32) (xy 87.63 20.32))
     (stroke (width 0) (type default) (color 0 0 0 0))
@@
     (stroke (width 0) (type default) (color 0 0 0 0))
   )
-  (wire (pts (xy 157.48 191.77) (xy 161.29 191.77))
+  (wire (pts (xy 163.83 189.23) (xy 161.29 189.23))
     (stroke (width 0) (type default) (color 0 0 0 0))
   )
@@
     (stroke (width 0) (type default) (color 0 0 0 0))
   )
+  (wire (pts (xy 161.29 185.42) (xy 161.29 189.23))
+    (stroke (width 0) (type default) (color 0 0 0 0))
+  )
   (wire (pts (xy 157.48 81.28) (xy 157.48 83.82))
     (stroke (width 0) (type default) (color 0 0 0 0))
@@
     )
   )
-  (global_label "USB5V" (shape passive) (at 161.29 162.56 90) (fields_autoplaced)
-    (effects (font (size 1.27 1.27)) (justify left))
-    (property "Intersheet References" "${INTERSHEET_REFS}" (id 0) (at 161.3694 154.0388 90)
-      (effects (font (size 1.27 1.27)) (justify left) hide)
-    )
-  )
   (global_label "SWMA" (shape bidirectional) (at 195.58 24.13 90) (fields_autoplaced)
     (effects (font (size 1.27 1.27)) (justify left))
@@
     )
   )
-  (global_label "USB_D+" (shape bidirectional) (at 157.48 191.77 180) (fields_autoplaced)
-    (effects (font (size 1.27 1.27)) (justify right))
-    (property "Intersheet References" "${INTERSHEET_REFS}" (id 0) (at 147.4469 191.6906 0)
-      (effects (font (size 1.27 1.27)) (justify right) hide)
+  (global_label "USB_D+" (shape bidirectional) (at 163.83 189.23 0) (fields_autoplaced)
+    (effects (font (size 1.27 1.27)) (justify left))
+    (property "Intersheet References" "${INTERSHEET_REFS}" (id 0) (at 173.8631 189.1506 0)
+      (effects (font (size 1.27 1.27)) (justify left) hide)
     )
   )
@@
     (pin "1")
   )
+  (symbol (lib_id "power:+3V3") (at 161.29 162.56 0) (unit 1)
+    (in_bom yes) (on_board yes)
+    (property "Reference" "#PWR0101" (id 0) (at 161.29 166.37 0)
+      (effects (font (size 1.27 1.27)) hide)
+    )
+    (property "Value" "+3V3" (id 1) (at 158.75 158.75 0)
+      (effects (font (size 1.27 1.27)) (justify left))
+    )
+    (property "Footprint" "" (id 2) (at 161.29 162.56 0)
+      (effects (font (size 1.27 1.27)) hide)
+    )
+    (property "Datasheet" "" (id 3) (at 161.29 162.56 0)
+      (effects (font (size 1.27 1.27)) hide)
+    )
+    (pin "1")
+  )
   (symbol (lib_id "Device:C") (at 19.05 69.85 0) (unit 1)
     (in_bom yes) (on_board yes)
@@
       (reference "#PWR048") (unit 1) (value "+3V3") (footprint "")
     )
+    (path "/9581b63f-eedc-4fe4-8b30-cace49b9d9f7"
+      (reference "#PWR0101") (unit 1) (value "+3V3") (footprint "")
+    )
     (path "/01a5503d-60cf-497a-bd00-91e022c2b184"

Commit message: fix schematic and pcb
Parts:
- added D5: BAT60JFILM, Diode_SMD:D_SOD-323_HandSoldering, symbol Device:D
- renumbered D5 to D6, D6 to D7
Connections:
- net +3V3: no longer J1.4 (Pin_4)
- net DBG_TX: now also U2.16 (B5); no longer U2.18 (B3)
- net DBG_TXB: now also U2.8 (A5); no longer U2.6 (A3)
- net GND: now also J1.3 (Pin_3); no longer J1.2 (Pin_2)
- net STM_JTCK: now also J1.2 (Pin_2); no longer J1.3 (Pin_3)
- net T_JRST: now also D1.4 (K); no longer D1.5 (K)
- net T_JTDI: no longer U2.16 (B5), U2.17 (B4)
- net T_JTDI_: now also J2.5 (Pin_5), R1.2; no longer J2.13 (Pin_13), J3.6 (Pin_6)
- net T_JTDO: now also U2.7 (A4); no longer D1.4 (K), R16.1, U2.8 (A5)
- net T_SWO: now also U2.6 (A3); no longer U2.7 (A4)
- net at C12.1, C13.1, D3.1 (K)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: now also D5.1 (K)
- net RST renamed SWIM_RST
- net RSTB renamed SWIM_RST_IN
- net SWM_IN renamed SWIM_IN
- removed net T_JTDO_: J2.5 (Pin_5), R1.2, R16.2
- new net PRG_5V: D5.2 (A), J1.4 (Pin_4)
- new net T_JTDO_SWO: D1.5 (K), R16.1, U2.17 (B4), U2.18 (B3)
- new net T_JTDO_SWO_: J2.13 (Pin_13), J3.6 (Pin_6), R16.2
Other:
- note added: "GND"
- note added: "NRST"
- note added: "SWCLK"
- note added: "SWDIO"
- note added: "SWO"
- moved on the sheet: D1, D2, R31, R32

Commit message: update schema and pcb
Parts:
- added JP3: SolderJumper_3_Open, Jumper:SolderJumper-3_P1.3mm_Open_RoundedPad1.0x1.5mm, symbol Jumper:SolderJumper_3_Open
- added R35: 1.5k, Resistor_SMD:R_0805_2012Metric, symbol Device:R
- renumbered C18 to C17, C19 to C18, C17 to C19, R25 to R10, R9 to R11, R10 to R12, R11 to R13, R12 to R14, R13 to R15, R14 to R16, R15 to R17, R16 to R18, R17 to R19, R18 to R20, R19 to R21, R20 to R22, R21 to R23, R23 to R24, R24 to R25, R33 to R31, R34 to R32, R32 to R33, R31 to R34, R35 to R36, R36 to R37, R37 to R38, R22 to R6, R6 to R7, R7 to R8, R8 to R9
Connections:
- net +3V3: now also C19.1, U5.13 (SPD), U5.14 (VDD2), U5.16 (VBUS2), JP3.1 (A)
- net USB5V: no longer U5.16 (VBUS2)
- net at QC1.2 (E), R36.1: now also R35.1
- net DI+: no longer names the net of R26.2, U4.4
- net DI-: no longer names the net of R29.2, U4.6
- net USB_D+ renamed DD+
- net USB_D- renamed DD-
- new net: JP3.2 (C), U5.12 (PIN)
- new net PINCTRL: JP3.3 (B), R35.2
Other:
- moved on the sheet: C10, C11, C17, C19, C8, D6, D7, J9, JP1, JP2, PS1, R10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
