File: ZX-Spectrum-Pentagon/ZX-Spectrum-Pentagon/VideoEncoder.kicad_sch (KiCad schematic)
At the start: 46 parts, among them U49 AD724

Commit message: Fix RGB
Connections:
- net GREEN: now also RVE9.2; no longer RVE15.2
- net RED: now also RVE15.2; no longer RVE9.2
- net TTLG: now also RVE7.2; no longer RVE10.2
- net TTLR: now also RVE10.2; no longer RVE7.2
- net ENGREEN: now reaches U49.7 (GIN)
- net ENGREEN: now also CVE6.2; no longer CVE3.2
- net ENRED: now reaches U49.6 (RIN)
- net ENRED: now also CVE3.2; no longer CVE6.2
- net ENBLUE: now reaches CVE8.2, U49.8 (BIN)
Changed lines of the file:
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@@
+	(wire
+		(pts
+			(xy 123.19 121.92) (xy 143.51 121.92)
+		)
+		(stroke
+			(width 0)
+			(type default)
+		)
+	)
 	(wire
 		(pts
@@
 	(wire
 		(pts
-			(xy 123.19 119.38) (xy 123.19 124.46)
+			(xy 123.19 119.38) (xy 123.19 121.92)
 		)
 		(stroke
@@
 	(wire
 		(pts
-			(xy 125.73 121.92) (xy 125.73 134.62)
+			(xy 125.73 124.46) (xy 125.73 134.62)
 		)
 		(stroke
@@
 	(wire
 		(pts
-			(xy 123.19 124.46) (xy 143.51 124.46)
-		)
-		(stroke
-			(width 0)
-			(type default)
-		)
-	)
-	(wire
-		(pts
 			(xy 241.3 104.14) (xy 243.84 104.14)
 		)
@@
 	(wire
 		(pts
-			(xy 125.73 121.92) (xy 143.51 121.92)
+			(xy 125.73 124.46) (xy 143.51 124.46)
 		)
 		(stroke
@@
 		)
 	)
-	(label "TTLR"
+	(label "TTLG"
 		(at 40.64 82.55 0)
 		(fields_autoplaced yes)
@@
 		)
 	)
+	(label "ENGREEN"
+		(at 137.16 124.46 180)
+		(fields_autoplaced yes)
+		(effects
+			(font
+				(size 1.27 1.27)
+			)
+			(justify right bottom)
+		)
+	)
+	(label "ENBLUE"
+		(at 137.16 127 180)
+		(fields_autoplaced yes)
+		(effects
+			(font
+				(size 1.27 1.27)
+			)
+			(justify right bottom)
+		)
+	)
 	(label "HSYNC"
 		(at 40.64 147.32 0)
@@
 		)
 	)
-	(label "TTLG"
+	(label "TTLR"
 		(at 40.64 95.25 0)
 		(fields_autoplaced yes)
@@
 	)
 	(label "GREEN"
-		(at 130.81 101.6 180)
+		(at 130.81 88.9 180)
 		(fields_autoplaced yes)
 		(effects
@@
 		)
 	)
+	(label "ENRED"
+		(at 137.16 121.92 180)
+		(fields_autoplaced yes)
+		(effects
+			(font
+				(size 1.27 1.27)
+			)
+			(justify right bottom)
+		)
+	)
 	(label "+12V"
 		(at 35.56 29.21 180)
@@
 	)
 	(label "RED"
-		(at 130.81 88.9 180)
-		(fields_autoplaced yes)
-		(effects
+		(at 130.81 101.6 180)
+		(fields_autoplaced yes)
+		(effects
