File: ZX_Keyboard/Connectors.kicad_sch (KiCad schematic)
At the start: 17 parts

Commit message: new annotation
Parts:
- renumbered CC2 to CC1, CC1 to CC2, JC2 to JC1, JC3 to JC2, JC4 to JC3, JC1 to JC4, LEDC2 to LEDC1, LEDC1 to LEDC2, RC6 to RC1, RC3 to RC2, RC2 to RC3, RC1 to RC6
Changed lines of the file:
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@@
 		(dnp no)
 		(fields_autoplaced yes)
-		(property "Reference" "#PWR036"
+		(property "Reference" "#PWR037"
 			(at 116.84 50.8 0)
 			(effects
@@
 			(project "ZX_Keyboard"
 				(path "/f89ca003-fbba-4e13-be9e-35859400364e/12b760a5-c3eb-4ef4-950b-cc3bc2438e7f"
-					(reference "#PWR036")
+					(reference "#PWR037")
 					(unit 1)
 				)
@@
 		(dnp no)
 		(fields_autoplaced yes)
-		(property "Reference" "RC3"
+		(property "Reference" "RC2"
 			(at 152.4 45.7199 0)
 			(effects
@@
 			(project "ZX_Keyboard"
 				(path "/f89ca003-fbba-4e13-be9e-35859400364e/12b760a5-c3eb-4ef4-950b-cc3bc2438e7f"
-					(reference "RC3")
+					(reference "RC2")
 					(unit 1)
 				)
@@
 		(on_board yes)
 		(dnp no)
-		(property "Reference" "JC4"
+		(property "Reference" "JC3"
 			(at 129.54 135.89 0)
 			(effects
@@
 			(project ""
 				(path "/f89ca003-fbba-4e13-be9e-35859400364e/12b760a5-c3eb-4ef4-950b-cc3bc2438e7f"
-					(reference "JC4")
+					(reference "JC3")
 					(unit 1)
 				)
@@
 		(dnp no)
 		(fields_autoplaced yes)
-		(property "Reference" "LEDC1"
+		(property "Reference" "LEDC2"
 			(at 234.95 39.6874 90)
 			(effects
@@
 			(project "ZX_Keyboard"
 				(path "/f89ca003-fbba-4e13-be9e-35859400364e/12b760a5-c3eb-4ef4-950b-cc3bc2438e7f"
-					(reference "LEDC1")
+					(reference "LEDC2")
 					(unit 1)
 				)
@@
 		(on_board yes)
 		(dnp no)
-		(property "Reference" "JC2"
+		(property "Reference" "JC1"
 			(at 45.72 135.89 0)
 			(effects
@@
 			(project "ZX_Keyboard"
 				(path "/f89ca003-fbba-4e13-be9e-35859400364e/12b760a5-c3eb-4ef4-950b-cc3bc2438e7f"
-					(reference "JC2")
+					(reference "JC1")
 					(unit 1)
 				)
@@
 		(dnp no)
 		(fields_autoplaced yes)
-		(property "Reference" "JC1"
+		(property "Reference" "JC4"
 			(at 266.7 88.8999 0)
 			(effects
@@
 			(project "ZX_Keyboard"
 				(path "/f89ca003-fbba-4e13-be9e-35859400364e/12b760a5-c3eb-4ef4-950b-cc3bc2438e7f"
-					(reference "JC1")
+					(reference "JC4")
 					(unit 1)
 				)
@@
 		(on_board yes)
 		(dnp no)
-		(property "Reference" "#PWR035"
+		(property "Reference" "#PWR036"
 			(at 106.68 43.18 0)
 			(effects
@@
 			(project "ZX_Keyboard"
 				(path "/f89ca003-fbba-4e13-be9e-35859400364e/12b760a5-c3eb-4ef4-950b-cc3bc2438e7f"
-					(reference "#PWR035")
+					(reference "#PWR036")
 					(unit 1)
 				)
@@
 		(dnp no)
 		(fields_autoplaced yes)
-		(property "Reference" "#PWR042"
+		(property "Reference" "#PWR045"
 			(at 260.35 111.76 0)
 			(effects
@@
 			(project "ZX_Keyboard"
 				(path "/f89ca003-fbba-4e13-be9e-35859400364e/12b760a5-c3eb-4ef4-950b-cc3bc2438e7f"
-					(reference "#PWR042")
+					(reference "#PWR045")
 					(unit 1)
 				)
@@
 		(dnp no)
 		(fields_autoplaced yes)
-		(property "Reference" "CC1"
+		(property "Reference" "CC2"
 			(at 191.135 67.6909 0)
 			(effects
@@
 			(project "ZX_Keyboard"
 				(path "/f89ca003-fbba-4e13-be9e-35859400364e/12b760a5-c3eb-4ef4-950b-cc3bc2438e7f"
-					(reference "CC1")
+					(reference "CC2")
 					(unit 1)
 				)
@@
 		(on_board yes)
 		(dnp no)
-		(property "Reference" "JC3"
+		(property "Reference" "JC2"
 			(at 88.9 135.89 0)
 			(effects
@@
 			(project "ZX_Keyboard"
 				(path "/f89ca003-fbba-4e13-be9e-35859400364e/12b760a5-c3eb-4ef4-950b-cc3bc2438e7f"
-					(reference "JC3")
+					(reference "JC2")
 					(unit 1)
 				)
@@
 		(on_board yes)
 		(dnp no)
-		(property "Reference" "#PWR066"
+		(property "Reference" "#PWR034"
 			(at 88.9 175.26 0)
 			(effects
@@
 			(project "ZX_Keyboard"
 				(path "/f89ca003-fbba-4e13-be9e-35859400364e/12b760a5-c3eb-4ef4-950b-cc3bc2438e7f"
-					(reference "#PWR066")
+					(reference "#PWR034")
 					(unit 1)
 				)
@@
 		(dnp no)
 		(fields_autoplaced yes)
-		(property "Reference" "LEDC2"
+		(property "Reference" "LEDC1"
 			(at 165.1 52.3874 90)
 			(effects
@@
 			(project "ZX_Keyboard"
 				(path "/f89ca003-fbba-4e13-be9e-35859400364e/12b760a5-c3eb-4ef4-950b-cc3bc2438e7f"
-					(reference "LEDC2")
+					(reference "LEDC1")
 					(unit 1)
 				)
@@
 		(dnp no)
 		(fields_autoplaced yes)
-		(property "Reference" "#PWR041"
+		(property "Reference" "#PWR040"
 			(at 149.86 101.6 0)
 			(effects
@@
 			(project "ZX_Keyboard"
 				(path "/f89ca003-fbba-4e13-be9e-35859400364e/12b760a5-c3eb-4ef4-950b-cc3bc2438e7f"
-					(reference "#PWR041")
+					(reference "#PWR040")
 					(unit 1)
 				)
@@
 		(on_board yes)
 		(dnp no)
-		(property "Reference" "#PWR039"
+		(property "Reference" "#PWR038"
 			(at 124.46 82.55 0)
 			(effects
@@
 			(project "ZX_Keyboard"
 				(path "/f89ca003-fbba-4e13-be9e-35859400364e/12b760a5-c3eb-4ef4-950b-cc3bc2438e7f"
-					(reference "#PWR039")
+					(reference "#PWR038")
 					(unit 1)
 				)
@@
 		(dnp no)
 		(fields_autoplaced yes)
-		(property "Reference" "RC2"
+		(property "Reference" "RC3"
 			(at 163.83 40.6399 0)
 			(effects
@@
 			(project "ZX_Keyboard"
 				(path "/f89ca003-fbba-4e13-be9e-35859400364e/12b760a5-c3eb-4ef4-950b-cc3bc2438e7f"
-					(reference "RC2")
+					(reference "RC3")
 					(unit 1)
 				)
@@
 		(on_board yes)
 		(dnp no)
-		(property "Reference" "#PWR044"
+		(property "Reference" "#PWR033"
 			(at 45.72 176.53 0)
 			(effects
@@
 			(project "ZX_Keyboard"
 				(path "/f89ca003-fbba-4e13-be9e-35859400364e/12b760a5-c3eb-4ef4-950b-cc3bc2438e7f"
-					(reference "#PWR044")
+					(reference "#PWR033")
 					(unit 1)
 				)
@@
 		(dnp no)
 		(fields_autoplaced yes)
-		(property "Reference" "#PWR033"
+		(property "Reference" "#PWR043"
 			(at 231.14 26.67 0)
 			(effects
@@
 			(project "ZX_Keyboard"
 				(path "/f89ca003-fbba-4e13-be9e-35859400364e/12b760a5-c3eb-4ef4-950b-cc3bc2438e7f"
-					(reference "#PWR033")
+					(reference "#PWR043")
 					(unit 1)
 				)
@@
 		(on_board yes)
 		(dnp no)
-		(property "Reference" "#PWR043"
+		(property "Reference" "#PWR039"
 			(at 129.54 175.26 0)
 			(effects
@@
 			(project "ZX_Keyboard"
 				(path "/f89ca003-fbba-4e13-be9e-35859400364e/12b760a5-c3eb-4ef4-950b-cc3bc2438e7f"
-					(reference "#PWR043")
+					(reference "#PWR039")
 					(unit 1)
 				)
@@
 		(on_board yes)
 		(dnp no)
-		(property "Reference" "#PWR034"
+		(property "Reference" "#PWR035"
 			(at 116.84 35.56 0)
 			(effects
@@
 			(project "ZX_Keyboard"
 				(path "/f89ca003-fbba-4e13-be9e-35859400364e/12b760a5-c3eb-4ef4-950b-cc3bc2438e7f"
-					(reference "#PWR034")
+					(reference "#PWR035")
 					(unit 1)
 				)
@@
 		(on_board yes)
 		(dnp no)
-		(property "Reference" "RC1"
+		(property "Reference" "RC6"
 			(at 234.95 27.94 0)
 			(effects
@@
 			(project "ZX_Keyboard"
 				(path "/f89ca003-fbba-4e13-be9e-35859400364e/12b760a5-c3eb-4ef4-950b-cc3bc2438e7f"
-					(reference "RC1")
+					(reference "RC6")
 					(unit 1)
 				)
@@
 		(dnp no)
 		(fields_autoplaced yes)
-		(property "Reference" "#PWR040"
+		(property "Reference" "#PWR041"
 			(at 187.325 82.55 0)
 			(effects
@@
 			(project "ZX_Keyboard"
 				(path "/f89ca003-fbba-4e13-be9e-35859400364e/12b760a5-c3eb-4ef4-950b-cc3bc2438e7f"
-					(reference "#PWR040")
+					(reference "#PWR041")
 					(unit 1)
 				)
@@
 		(on_board yes)
 		(dnp no)
-		(property "Reference" "#PWR037"
+		(property "Reference" "#PWR042"
 			(at 220.98 69.85 0)
 			(effects
@@
 			(project "ZX_Keyboard"
 				(path "/f89ca003-fbba-4e13-be9e-35859400364e/12b760a5-c3eb-4ef4-950b-cc3bc2438e7f"
-					(reference "#PWR037")
+					(reference "#PWR042")
 					(unit 1)
 				)
@@
 		(dnp no)
 		(fields_autoplaced yes)
-		(property "Reference" "RC6"
+		(property "Reference" "RC1"
 			(at 127 68.5799 0)
 			(effects
@@
 			(project "ZX_Keyboard"
 				(path "/f89ca003-fbba-4e13-be9e-35859400364e/12b760a5-c3eb-4ef4-950b-cc3bc2438e7f"
-					(reference "RC6")
+					(reference "RC1")
 					(unit 1)
 				)
@@
 		(dnp no)
 		(fields_autoplaced yes)
-		(property "Reference" "CC2"
+		(property "Reference" "CC1"
 			(at 163.83 72.39 90)
 			(effects
@@
 			(project "ZX_Keyboard"
 				(path "/f89ca003-fbba-4e13-be9e-35859400364e/12b760a5-c3eb-4ef4-950b-cc3bc2438e7f"
-					(reference "CC2")
+					(reference "CC1")
 					(unit 1)
 				)
@@
 		(on_board yes)
 		(dnp no)
-		(property "Reference" "#PWR038"
+		(property "Reference" "#PWR044"
 			(at 231.14 69.85 0)
 			(effects
@@
 			(project "ZX_Keyboard"
 				(path "/f89ca003-fbba-4e13-be9e-35859400364e/12b760a5-c3eb-4ef4-950b-cc3bc2438e7f"
-					(reference "#PWR038")
-					(unit 1)
-				)
+					(reference "#PWR044")
+					(unit 1)
+				)
