File: extension_mb1136/connection_mb1136.kicad_sch (KiCad schematic)
At the start: 6 parts

Commit message: non functional update
Parts:
- CN1, CN2: value (none) -> Conn_02x19_Odd_Even; footprint (none) -> Connector_PinHeader_2.54mm:PinHeader_2x19_P2.54mm_Vertical
- CN3, CN5: value (none) -> Conn_01x08; footprint (none) -> Connector_PinSocket_2.54mm:PinSocket_1x08_P2.54mm_Vertical
- CN4: value (none) -> Conn_01x06; footprint (none) -> Connector_PinSocket_2.54mm:PinSocket_1x06_P2.54mm_Vertical
- CN6: value (none) -> Conn_01x10; footprint (none) -> Connector_PinSocket_2.54mm:PinSocket_1x10_P2.54mm_Vertical
