File: extension_mb1136/usb_mb1136.kicad_sch (KiCad schematic)
At the start: 25 parts

Commit message: non functional update
Parts:
- C1: value (none) -> 4.7uF; footprint (none) -> Capacitor_SMD:C_1206_3216Metric_Pad1.33x1.80mm_HandSolder
- CNUSB_1: value (none) -> USB_OTG; footprint (none) -> Connector_USB:USB_Micro-B_Molex-105017-0001
- CNUSB_2: value (none) -> USB_A; footprint (none) -> Connector_USB:USB_A_Molex_67643_Horizontal
- CNUSB_3: value (none) -> USB_BP; footprint (none) -> Connector_USB:USB_B_OST_USB-B1HSxx_Horizontal
- D1: value (none) -> ESDALC6V1-1U2; footprint (none) -> Diode_SMD:D_0201_0603Metric
- D2, D3: value (none) -> 1N4001; footprint (none) -> Diode_SMD:D_SOD-323_HandSoldering
- J1, J2: value (none) -> Conn_01x03; footprint (none) -> Connector_PinHeader_2.54mm:PinHeader_1x03_P2.54mm_Vertical
- LD1: value (none) -> RED; footprint (none) -> Diode_SMD:D_0805_2012Metric
- LD2: value (none) -> GREEN; footprint (none) -> Diode_SMD:D_0805_2012Metric
- Q1: value (none) -> S9013; footprint (none) -> Package_TO_SOT_SMD:SOT-23
- R1: value (none) -> 620; footprint (none) -> Resistor_SMD:R_0805_2012Metric
- R2, R6: value (none) -> 47K; footprint (none) -> Resistor_SMD:R_0805_2012Metric
- R3: value (none) -> 10K; footprint (none) -> Resistor_SMD:R_0805_2012Metric
- R4: value (none) -> 330; footprint (none) -> Resistor_SMD:R_0805_2012Metric
- R5: value (none) -> 430K; footprint (none) -> Resistor_SMD:R_0805_2012Metric
- R7: value (none) -> 620K; footprint (none) -> Resistor_SMD:R_0805_2012Metric
- R8: value (none) -> 22K; footprint (none) -> Resistor_SMD:R_0805_2012Metric
- R9: value (none) -> 1K5; footprint (none) -> Resistor_SMD:R_0805_2012Metric
- SW1, SW2: value (none) -> USB_SEL; footprint (none) -> Connector_PinHeader_2.54mm:PinHeader_2x03_P2.54mm_Vertical
- U1: value (none) -> STMPS2151MTR; footprint (none) -> Package_SO:SO-8_3.9x4.9mm_P1.27mm
- U2: value (none) -> USBLC6-2; footprint (none) -> Package_TO_SOT_SMD:SOT-23-6_Handsoldering
