File: beomaster_5500/beomaster_5500.kicad_pcb (KiCad board)
At the start: 2 copper layers, 1 part, among them Q1 Q_PNP_Darlington_ECB

Commit message: improve schema
Parts:
- removed Q1: Q_PNP_Darlington_ECB, Package_TO_SOT_THT:TO-247-3_Vertical
- added C201: 100UFx50V, Capacitor_THT:CP_Radial_D10.0mm_P7.50mm, F.Cu at (79.3, 100.2)
- added C207: 10UFx16V, Capacitor_THT:CP_Radial_D8.0mm_P5.00mm, F.Cu at (109.4, 46.5)
- added C214: 100UFx10V, Capacitor_THT:CP_Radial_D8.0mm_P5.00mm, F.Cu at (109.4, 56.1)
- added C301: 100UFx50V, Capacitor_THT:CP_Radial_D10.0mm_P7.50mm, F.Cu at (145.6, 100.2)
- added C307: 10UFx16V, Capacitor_THT:CP_Radial_D8.0mm_P5.00mm, F.Cu at (175.8, 46.5)
- added C314: 100UFx10V, Capacitor_THT:CP_Radial_D8.0mm_P5.00mm, F.Cu at (175.8, 56.1)
- added D201: 1N4148, Diode_THT:D_DO-35_SOD27_P10.16mm_Horizontal, F.Cu at (95.2, 43.5)
- added D202: 1N4148, Diode_THT:D_DO-35_SOD27_P10.16mm_Horizontal, F.Cu at (95.2, 47.1)
- added D203: 1N4148, Diode_THT:D_DO-35_SOD27_P10.16mm_Horizontal, F.Cu at (95.2, 50.6)
- added D204: 1N4148, Diode_THT:D_DO-35_SOD27_P10.16mm_Horizontal, F.Cu at (95.2, 54.2)
- added D205: 1N4148, Diode_THT:D_DO-35_SOD27_P10.16mm_Horizontal, F.Cu at (95.2, 57.7)
- added D206: 1N4148, Diode_THT:D_DO-35_SOD27_P10.16mm_Horizontal, F.Cu at (95.2, 61.3)
- added D207: 12V, Diode_THT:D_DO-35_SOD27_P10.16mm_Horizontal, F.Cu at (95.2, 64.8)
- added D301: 1N4148, Diode_THT:D_DO-35_SOD27_P10.16mm_Horizontal, F.Cu at (161.6, 43.5)
- added D302: 1N4148, Diode_THT:D_DO-35_SOD27_P10.16mm_Horizontal, F.Cu at (161.6, 47.1)
- added D303: 1N4148, Diode_THT:D_DO-35_SOD27_P10.16mm_Horizontal, F.Cu at (161.6, 50.6)
- added D304: 1N4148, Diode_THT:D_DO-35_SOD27_P10.16mm_Horizontal, F.Cu at (161.6, 54.2)
- added D305: 1N4148, Diode_THT:D_DO-35_SOD27_P10.16mm_Horizontal, F.Cu at (161.6, 57.7)
- added D306: 1N4148, Diode_THT:D_DO-35_SOD27_P10.16mm_Horizontal, F.Cu at (161.6, 61.3)
- added D307: 12V, Diode_THT:D_DO-35_SOD27_P10.16mm_Horizontal, F.Cu at (161.6, 64.8)
- added L201: 0,5UH, Inductor_THT:L_Radial_L10.2mm_W10.2mm_Px7.62mm_Py7.62mm_Pulse_LP-30, F.Cu at (67.3, 104.0)
- added L301: 0,5UH, Inductor_THT:L_Radial_L10.2mm_W10.2mm_Px7.62mm_Py7.62mm_Pulse_LP-30, F.Cu at (133.7, 104.0)
- added Q201: BF423, Package_TO_SOT_THT:TO-92_Inline_Wide, F.Cu at (95.2, 69.8)
- added Q202: BF857, Package_TO_SOT_THT:TO-220-3_Vertical, F.Cu at (56.9, 98.3)
- added Q203: BDV65B, Package_TO_SOT_THT:TO-247-3_Vertical, F.Cu at (96.9, 87.1)
- added Q204: BC547B, Package_TO_SOT_THT:TO-92_Inline_Wide, F.Cu at (95.2, 75.6)
- added Q205: BF422, Package_TO_SOT_THT:TO-92_Inline_Wide, F.Cu at (95.2, 81.4)
- added Q206: BC547B, Package_TO_SOT_THT:TO-92_Inline_Wide, F.Cu at (103.3, 69.8)
- added Q207: BC547B, Package_TO_SOT_THT:TO-92_Inline_Wide, F.Cu at (103.3, 75.6)
- added Q208: BC557B, Package_TO_SOT_THT:TO-92_Inline_Wide, F.Cu at (103.3, 81.4)
- added Q209: BDV64B, Package_TO_SOT_THT:TO-247-3_Vertical, F.Cu at (96.9, 93.7)
- added Q210: BC547B, Package_TO_SOT_THT:TO-92_Inline_Wide, F.Cu at (111.5, 69.8)
- added Q211: BF857, Package_TO_SOT_THT:TO-220-3_Vertical, F.Cu at (56.9, 104.3)
- added Q212: MPSA13, Package_TO_SOT_THT:TO-92_Inline_Wide, F.Cu at (111.5, 75.6)
- added Q213: BC547B, Package_TO_SOT_THT:TO-92_Inline_Wide, F.Cu at (111.5, 81.4)
- added Q301: BF423, Package_TO_SOT_THT:TO-92_Inline_Wide, F.Cu at (161.6, 69.8)
- added Q302: BF857, Package_TO_SOT_THT:TO-220-3_Vertical, F.Cu at (123.3, 98.3)
- added Q303: BDV65B, Package_TO_SOT_THT:TO-247-3_Vertical, F.Cu at (163.3, 87.1)
- added Q304: BC547B, Package_TO_SOT_THT:TO-92_Inline_Wide, F.Cu at (161.6, 75.6)
- added Q305: BF422, Package_TO_SOT_THT:TO-92_Inline_Wide, F.Cu at (161.6, 81.4)
- added Q306: BC547B, Package_TO_SOT_THT:TO-92_Inline_Wide, F.Cu at (169.7, 69.8)
- added Q307: BC547B, Package_TO_SOT_THT:TO-92_Inline_Wide, F.Cu at (169.7, 75.6)
- added Q308: BC557B, Package_TO_SOT_THT:TO-92_Inline_Wide, F.Cu at (169.7, 81.4)
- added Q309: BDV64B, Package_TO_SOT_THT:TO-247-3_Vertical, F.Cu at (163.3, 93.7)
- added Q310: BC547B, Package_TO_SOT_THT:TO-92_Inline_Wide, F.Cu at (177.9, 69.8)
- added Q311: BF857, Package_TO_SOT_THT:TO-220-3_Vertical, F.Cu at (123.3, 104.3)
- added Q312: MPSA13, Package_TO_SOT_THT:TO-92_Inline_Wide, F.Cu at (177.9, 75.6)
- added Q313: BC547B, Package_TO_SOT_THT:TO-92_Inline_Wide, F.Cu at (177.9, 81.4)
- added R201: 150, Resistor_THT:R_Axial_DIN0207_L6.3mm_D2.5mm_P10.16mm_Horizontal, F.Cu at (55.3, 43.8)
- added R202: 560, Resistor_THT:R_Axial_DIN0207_L6.3mm_D2.5mm_P10.16mm_Horizontal, F.Cu at (55.3, 47.8)
- added R203: 560, Resistor_THT:R_Axial_DIN0207_L6.3mm_D2.5mm_P10.16mm_Horizontal, F.Cu at (55.3, 51.9)
- added R204: 68, Resistor_THT:R_Axial_DIN0207_L6.3mm_D2.5mm_P10.16mm_Horizontal, F.Cu at (55.3, 55.9)
- added R205: 220K, Resistor_THT:R_Axial_DIN0207_L6.3mm_D2.5mm_P10.16mm_Horizontal, F.Cu at (55.3, 60.0)
- added R206: 1K, Resistor_THT:R_Axial_DIN0207_L6.3mm_D2.5mm_P10.16mm_Horizontal, F.Cu at (55.3, 64.0)
- added R207: 27, Resistor_THT:R_Axial_DIN0207_L6.3mm_D2.5mm_P10.16mm_Horizontal, F.Cu at (55.3, 68.1)
- added R208: 2,2M, Resistor_THT:R_Axial_DIN0207_L6.3mm_D2.5mm_P10.16mm_Horizontal, F.Cu at (55.3, 72.1)
- added R209: 10K, Resistor_THT:R_Axial_DIN0207_L6.3mm_D2.5mm_P10.16mm_Horizontal, F.Cu at (55.3, 76.2)
- added R210: 2,2K, Resistor_THT:R_Axial_DIN0207_L6.3mm_D2.5mm_P10.16mm_Horizontal, F.Cu at (55.3, 80.2)
- added R211: 680, Resistor_THT:R_Axial_DIN0207_L6.3mm_D2.5mm_P10.16mm_Horizontal, F.Cu at (55.3, 84.3)
- added R212: 270, Resistor_THT:R_Axial_DIN0207_L6.3mm_D2.5mm_P10.16mm_Horizontal, F.Cu at (55.3, 88.3)
- added R213: 33K, Resistor_THT:R_Axial_DIN0207_L6.3mm_D2.5mm_P10.16mm_Horizontal, F.Cu at (55.3, 92.4)
- added R214: 10K, Resistor_THT:R_Axial_DIN0207_L6.3mm_D2.5mm_P10.16mm_Horizontal, F.Cu at (68.6, 43.8)
- added R215: 470, Resistor_THT:R_Axial_DIN0207_L6.3mm_D2.5mm_P10.16mm_Horizontal, F.Cu at (68.6, 47.8)
- added R216: 2,2K, Resistor_THT:R_Axial_DIN0207_L6.3mm_D2.5mm_P10.16mm_Horizontal, F.Cu at (68.6, 51.9)
- added R217: 390, Resistor_THT:R_Axial_DIN0207_L6.3mm_D2.5mm_P10.16mm_Horizontal, F.Cu at (68.6, 55.9)
- added R218: 0.22, Resistor_THT:R_Axial_DIN0207_L6.3mm_D2.5mm_P10.16mm_Horizontal, F.Cu at (68.6, 60.0)
- added R219: 10K, Resistor_THT:R_Axial_DIN0207_L6.3mm_D2.5mm_P10.16mm_Horizontal, F.Cu at (68.6, 64.0)
- added R220: 1K, Resistor_THT:R_Axial_DIN0207_L6.3mm_D2.5mm_P10.16mm_Horizontal, F.Cu at (68.6, 68.1)
- added R221: 1K, Resistor_THT:R_Axial_DIN0207_L6.3mm_D2.5mm_P10.16mm_Horizontal, F.Cu at (68.6, 72.1)
- added R222: 10K, Resistor_THT:R_Axial_DIN0207_L6.3mm_D2.5mm_P10.16mm_Horizontal, F.Cu at (68.6, 76.2)
- added R223: 10K, Resistor_THT:R_Axial_DIN0207_L6.3mm_D2.5mm_P10.16mm_Horizontal, F.Cu at (68.6, 80.2)
- added R224: 390, Resistor_THT:R_Axial_DIN0207_L6.3mm_D2.5mm_P10.16mm_Horizontal, F.Cu at (68.6, 84.3)
- added R225: 100, Potentiometer_THT:Potentiometer_Bourns_3296Y_Vertical, F.Cu at (101.8, 99.1)
- added R226: 0.22, Resistor_THT:R_Axial_DIN0207_L6.3mm_D2.5mm_P10.16mm_Horizontal, F.Cu at (68.6, 88.3)
- added R227: 10K, Resistor_THT:R_Axial_DIN0207_L6.3mm_D2.5mm_P10.16mm_Horizontal, F.Cu at (68.6, 92.4)
- added R228: 100, Resistor_THT:R_Axial_DIN0207_L6.3mm_D2.5mm_P10.16mm_Horizontal, F.Cu at (81.9, 43.8)
- added R229: 270, Resistor_THT:R_Axial_DIN0207_L6.3mm_D2.5mm_P10.16mm_Horizontal, F.Cu at (81.9, 47.8)
- added R230: 1K, Resistor_THT:R_Axial_DIN0207_L6.3mm_D2.5mm_P10.16mm_Horizontal, F.Cu at (81.9, 51.9)
- added R231: 100, Resistor_THT:R_Axial_DIN0207_L6.3mm_D2.5mm_P10.16mm_Horizontal, F.Cu at (81.9, 55.9)
- added R232: 15K, Resistor_THT:R_Axial_DIN0207_L6.3mm_D2.5mm_P10.16mm_Horizontal, F.Cu at (81.9, 60.0)
- added R233: 15K, Resistor_THT:R_Axial_DIN0207_L6.3mm_D2.5mm_P10.16mm_Horizontal, F.Cu at (81.9, 64.0)
- added R234: 3,3K, Resistor_THT:R_Axial_DIN0207_L6.3mm_D2.5mm_P10.16mm_Horizontal, F.Cu at (81.9, 68.1)
- added R235: 47, Resistor_THT:R_Axial_DIN0207_L6.3mm_D2.5mm_P10.16mm_Horizontal, F.Cu at (81.9, 72.1)
- added R236: 4,7, Resistor_THT:R_Axial_DIN0207_L6.3mm_D2.5mm_P10.16mm_Horizontal, F.Cu at (81.9, 76.2)
- added R237: 180, Resistor_THT:R_Axial_DIN0207_L6.3mm_D2.5mm_P10.16mm_Horizontal, F.Cu at (81.9, 80.2)
- added R238: 270, Resistor_THT:R_Axial_DIN0207_L6.3mm_D2.5mm_P10.16mm_Horizontal, F.Cu at (81.9, 84.3)
- added R239: 68, Resistor_THT:R_Axial_DIN0207_L6.3mm_D2.5mm_P10.16mm_Horizontal, F.Cu at (81.9, 88.3)
- added R301: 150, Resistor_THT:R_Axial_DIN0207_L6.3mm_D2.5mm_P10.16mm_Horizontal, F.Cu at (121.7, 43.8)
- added R302: 560, Resistor_THT:R_Axial_DIN0207_L6.3mm_D2.5mm_P10.16mm_Horizontal, F.Cu at (121.7, 47.8)
- added R303: 560, Resistor_THT:R_Axial_DIN0207_L6.3mm_D2.5mm_P10.16mm_Horizontal, F.Cu at (121.7, 51.9)
- added R304: 68, Resistor_THT:R_Axial_DIN0207_L6.3mm_D2.5mm_P10.16mm_Horizontal, F.Cu at (121.7, 55.9)
- added R305: 220K, Resistor_THT:R_Axial_DIN0207_L6.3mm_D2.5mm_P10.16mm_Horizontal, F.Cu at (121.7, 60.0)
- added R306: 1K, Resistor_THT:R_Axial_DIN0207_L6.3mm_D2.5mm_P10.16mm_Horizontal, F.Cu at (121.7, 64.0)
- added R307: 27, Resistor_THT:R_Axial_DIN0207_L6.3mm_D2.5mm_P10.16mm_Horizontal, F.Cu at (121.7, 68.1)
- added R308: 2,2M, Resistor_THT:R_Axial_DIN0207_L6.3mm_D2.5mm_P10.16mm_Horizontal, F.Cu at (121.7, 72.1)
- added R309: 10K, Resistor_THT:R_Axial_DIN0207_L6.3mm_D2.5mm_P10.16mm_Horizontal, F.Cu at (121.7, 76.2)
- added R310: 2,2K, Resistor_THT:R_Axial_DIN0207_L6.3mm_D2.5mm_P10.16mm_Horizontal, F.Cu at (121.7, 80.2)
- added R311: 680, Resistor_THT:R_Axial_DIN0207_L6.3mm_D2.5mm_P10.16mm_Horizontal, F.Cu at (121.7, 84.3)
- added R312: 270, Resistor_THT:R_Axial_DIN0207_L6.3mm_D2.5mm_P10.16mm_Horizontal, F.Cu at (121.7, 88.3)
- added R313: 33K, Resistor_THT:R_Axial_DIN0207_L6.3mm_D2.5mm_P10.16mm_Horizontal, F.Cu at (121.7, 92.4)
- added R314: 10K, Resistor_THT:R_Axial_DIN0207_L6.3mm_D2.5mm_P10.16mm_Horizontal, F.Cu at (135.0, 43.8)
- added R315: 470, Resistor_THT:R_Axial_DIN0207_L6.3mm_D2.5mm_P10.16mm_Horizontal, F.Cu at (135.0, 47.8)
- added R316: 2,2K, Resistor_THT:R_Axial_DIN0207_L6.3mm_D2.5mm_P10.16mm_Horizontal, F.Cu at (135.0, 51.9)
- added R317: 390, Resistor_THT:R_Axial_DIN0207_L6.3mm_D2.5mm_P10.16mm_Horizontal, F.Cu at (135.0, 55.9)
- added R318: 0.22, Resistor_THT:R_Axial_DIN0207_L6.3mm_D2.5mm_P10.16mm_Horizontal, F.Cu at (135.0, 60.0)
- added R319: 10K, Resistor_THT:R_Axial_DIN0207_L6.3mm_D2.5mm_P10.16mm_Horizontal, F.Cu at (135.0, 64.0)
- added R320: 1K, Resistor_THT:R_Axial_DIN0207_L6.3mm_D2.5mm_P10.16mm_Horizontal, F.Cu at (135.0, 68.1)
- added R321: 1K, Resistor_THT:R_Axial_DIN0207_L6.3mm_D2.5mm_P10.16mm_Horizontal, F.Cu at (135.0, 72.1)
- added R322: 10K, Resistor_THT:R_Axial_DIN0207_L6.3mm_D2.5mm_P10.16mm_Horizontal, F.Cu at (135.0, 76.2)
- added R323: 10K, Resistor_THT:R_Axial_DIN0207_L6.3mm_D2.5mm_P10.16mm_Horizontal, F.Cu at (135.0, 80.2)
- added R324: 390, Resistor_THT:R_Axial_DIN0207_L6.3mm_D2.5mm_P10.16mm_Horizontal, F.Cu at (135.0, 84.3)
- added R325: 100, Potentiometer_THT:Potentiometer_Bourns_3296Y_Vertical, F.Cu at (168.1, 99.1)
- added R326: 0.22, Resistor_THT:R_Axial_DIN0207_L6.3mm_D2.5mm_P10.16mm_Horizontal, F.Cu at (135.0, 88.3)
- added R327: 10K, Resistor_THT:R_Axial_DIN0207_L6.3mm_D2.5mm_P10.16mm_Horizontal, F.Cu at (135.0, 92.4)
- added R328: 100, Resistor_THT:R_Axial_DIN0207_L6.3mm_D2.5mm_P10.16mm_Horizontal, F.Cu at (148.3, 43.8)
- added R329: 270, Resistor_THT:R_Axial_DIN0207_L6.3mm_D2.5mm_P10.16mm_Horizontal, F.Cu at (148.3, 47.8)
- added R330: 1K, Resistor_THT:R_Axial_DIN0207_L6.3mm_D2.5mm_P10.16mm_Horizontal, F.Cu at (148.3, 51.9)
- added R331: 100, Resistor_THT:R_Axial_DIN0207_L6.3mm_D2.5mm_P10.16mm_Horizontal, F.Cu at (148.3, 55.9)
- added R332: 15K, Resistor_THT:R_Axial_DIN0207_L6.3mm_D2.5mm_P10.16mm_Horizontal, F.Cu at (148.3, 60.0)
- added R333: 15K, Resistor_THT:R_Axial_DIN0207_L6.3mm_D2.5mm_P10.16mm_Horizontal, F.Cu at (148.3, 64.0)
- added R334: 3,3K, Resistor_THT:R_Axial_DIN0207_L6.3mm_D2.5mm_P10.16mm_Horizontal, F.Cu at (148.3, 68.1)
- added R335: 47, Resistor_THT:R_Axial_DIN0207_L6.3mm_D2.5mm_P10.16mm_Horizontal, F.Cu at (148.3, 72.1)
- added R336: 4,7, Resistor_THT:R_Axial_DIN0207_L6.3mm_D2.5mm_P10.16mm_Horizontal, F.Cu at (148.3, 76.2)
- added R337: 180, Resistor_THT:R_Axial_DIN0207_L6.3mm_D2.5mm_P10.16mm_Horizontal, F.Cu at (148.3, 80.2)
- added R338: 270, Resistor_THT:R_Axial_DIN0207_L6.3mm_D2.5mm_P10.16mm_Horizontal, F.Cu at (148.3, 84.3)
- added R339: 68, Resistor_THT:R_Axial_DIN0207_L6.3mm_D2.5mm_P10.16mm_Horizontal, F.Cu at (148.3, 88.3)
