File: Lenovo/Lenovo.kicad_pcb (KiCad board)
At the start: 2 copper layers, 57.1 x 17.8 mm, 15 parts, among them J1 Input, J2 SELECTOR, J3 +19.5V, J4 ACDET, J5 GND

Commit message: Change footprint
Parts:
- J1: footprint Custom-Connector:TENSILITY_54-00127 -> Custom-Connector:BarrelJack_DC007B
- moved J1 3.81 mm to (97.2, 57.1), turned to 90 degrees
