File: Lenovo/Lenovo.kicad_sch (KiCad schematic)
At the start: 15 parts, among them J1 Input, J2 SELECTOR, J3 +19.5V, J4 ACDET, J5 GND

Commit message: Change footprint
Parts:
- J1: footprint Custom-Connector:TENSILITY_54-00127 -> Custom-Connector:BarrelJack_DC007B; symbol Custom-Connector:54-00127 -> Connector:Barrel_Jack_MountingPin
Connections:
- net GND: now also J1.2, J1.MP (MountPin); no longer J1.B, J1.SH1, J1.SH2
- net POWER: now also J1.1; no longer J1.A
- no-connect marks 1 -> 0
Changed lines of the file:
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@@
-	)
-	(junction
-		(at 46.99 99.06)
-		(diameter 0)
-		(color 0 0 0 0)
 	)
 	(junction
@@
 		(color 0 0 0 0)
 	)
-	(no_connect
-		(at 50.8 88.9)
-	)
 	(wire
 		(pts
@@
 	(wire
 		(pts
+			(xy 43.18 99.06) (xy 63.5 99.06)
+		)
+		(stroke
+			(width 0)
+			(type default)
+		)
+	)
+	(wire
+		(pts
 			(xy 91.44 88.9) (xy 93.98 88.9)
 		)
@@
 	(wire
 		(pts
-			(xy 46.99 99.06) (xy 63.5 99.06)
-		)
-		(stroke
-			(width 0)
-			(type default)
-		)
-	)
-	(wire
-		(pts
 			(xy 83.82 135.89) (xy 86.36 135.89)
 		)
@@
 	(wire
 		(pts
-			(xy 38.1 99.06) (xy 46.99 99.06)
-		)
-		(stroke
-			(width 0)
-			(type default)
-		)
-	)
-	(wire
-		(pts
-			(xy 46.99 96.52) (xy 46.99 99.06)
+			(xy 43.18 96.52) (xy 43.18 99.06)
 		)
 		(stroke
@@
 		(pts
 			(xy 99.06 135.89) (xy 114.3 135.89)
-		)
-		(stroke
-			(width 0)
-			(type default)
-		)
-	)
-	(wire
-		(pts
-			(xy 38.1 96.52) (xy 38.1 99.06)
 		)
 		(stroke
@@
 	)
 	(symbol
-		(lib_id "Custom-Connector:54-00127")
-		(at 45.72 88.9 0)
+		(lib_id "Connector:Barrel_Jack_MountingPin")
+		(at 43.18 88.9 0)
 		(unit 1)
 		(exclude_from_sim no)
@@
 		(dnp no)
 		(property "Reference" "J1"
-			(at 37.592 82.042 0)
+			(at 35.052 82.042 0)
 			(effects
 				(font
@@
 		)
 		(property "Value" "Input"
-			(at 47.752 82.042 0)
+			(at 45.212 82.042 0)
 			(effects
 				(font
@@
 			)
 		)
-		(property "Footprint" "Custom-Connector:TENSILITY_54-00127"
-			(at 45.72 88.9 0)
+		(property "Footprint" "Custom-Connector:BarrelJack_DC007B"
+			(at 44.45 89.916 0)
+			(effects
+				(font
+					(size 1.27 1.27)
+				)
+				(hide yes)
+			)
+		)
+		(property "Datasheet" "~"
+			(at 44.45 89.916 0)
+			(effects
+				(font
+					(size 1.27 1.27)
+				)
+				(hide yes)
+			)
+		)
+		(property "Description" "DC Barrel Jack with a mounting pin"
+			(at 43.18 88.9 0)
+			(effects
+				(font
+					(size 1.27 1.27)
+				)
+				(hide yes)
+			)
+		)
+		(property "MF" "Tensility International Corp"
+			(at 43.18 88.9 0)
 			(effects
 				(font
@@
 			)
 		)
-		(property "Datasheet" "~"
-			(at 45.72 88.9 0)
-			(effects
-				(font
-					(size 1.27 1.27)
-				)
-				(hide yes)
-			)
-		)
-		(property "Description" "DC Barrel Jack with a mounting pin"
-			(at 45.72 88.9 0)
-			(effects
-				(font
-					(size 1.27 1.27)
-				)
-				(hide yes)
-			)
-		)
-		(property "MF" "Tensility International Corp"
-			(at 45.72 88.9 0)
+		(property "MAXIMUM_PACKAGE_HEIGHT" "7.3mm"
+			(at 43.18 88.9 0)
 			(effects
 				(font
@@
 			)
 		)
-		(property "MAXIMUM_PACKAGE_HEIGHT" "7.3mm"
-			(at 45.72 88.9 0)
+		(property "Package" "None"
+			(at 43.18 88.9 0)
 			(effects
 				(font
@@
 			)
 		)
-		(property "Package" "None"
-			(at 45.72 88.9 0)
+		(property "Price" "None"
+			(at 43.18 88.9 0)
 			(effects
 				(font
@@
 			)
 		)
-		(property "Price" "None"
-			(at 45.72 88.9 0)
+		(property "Check_prices" "https://www.snapeda.com/parts/54-00127/Tensility/view-part/?ref=eda"
+			(at 43.18 88.9 0)
 			(effects
 				(font
@@
 			)
 		)
-		(property "Check_prices" "https://www.snapeda.com/parts/54-00127/Tensility/view-part/?ref=eda"
-			(at 45.72 88.9 0)
+		(property "STANDARD" "Manufacturer Recommendations"
+			(at 43.18 88.9 0)
 			(effects
 				(font
@@
 			)
 		)
-		(property "STANDARD" "Manufacturer Recommendations"
-			(at 45.72 88.9 0)
+		(property "PARTREV" "A"
+			(at 43.18 88.9 0)
 			(effects
 				(font
@@
 			)
 		)
-		(property "PARTREV" "A"
-			(at 45.72 88.9 0)
+		(property "SnapEDA_Link" "https://www.snapeda.com/parts/54-00127/Tensility/view-part/?ref=snap"
+			(at 43.18 88.9 0)
 			(effects
 				(font
@@
 			)
 		)
-		(property "SnapEDA_Link" "https://www.snapeda.com/parts/54-00127/Tensility/view-part/?ref=snap"
-			(at 45.72 88.9 0)
+		(property "MP" "54-00127"
+			(at 43.18 88.9 0)
 			(effects
 				(font
@@
 			)
 		)
-		(property "MP" "54-00127"
-			(at 45.72 88.9 0)
+		(property "Description_1" "Connector, dc jack 5.5x2.1 mm, PCB mount, 90 degrees, silver plated, thru hole"
+			(at 43.18 88.9 0)
 			(effects
 				(font
@@
 			)
 		)
-		(property "Description_1" "Connector, dc jack 5.5x2.1 mm, PCB mount, 90 degrees, silver plated, thru hole"
-			(at 45.72 88.9 0)
+		(property "MANUFACTURER" "TENSILITY"
+			(at 43.18 88.9 0)
 			(effects
 				(font
@@
 			)
 		)
-		(property "MANUFACTURER" "TENSILITY"
-			(at 45.72 88.9 0)
+		(property "Availability" "In Stock"
+			(at 43.18 88.9 0)
 			(effects
 				(font
@@
 			)
 		)
-		(property "Availability" "In Stock"
-			(at 45.72 88.9 0)
+		(property "SNAPEDA_PN" "54-00127"
+			(at 43.18 88.9 0)
 			(effects
 				(font
@@
 			)
 		)
-		(property "SNAPEDA_PN" "54-00127"
-			(at 45.72 88.9 0)
-			(effects
-				(font
-					(size 1.27 1.27)
-				)
-				(justify bottom)
-				(hide yes)
-			)
-		)
-		(pin "C"
-		)
-		(pin "B"
-		)
-		(pin "SH1"
-		)
-		(pin "A"
-		)
-		(pin "SH2"
+		(pin "1"
+		)
+		(pin "2"
+		)
+		(pin "MP"
 		)
 		(instances
